File: schematics/dATX_JC100.kicad_sch (KiCad schematic)
At the start: 21 parts

Commit message: clock
Other:
- added sheet Clock (dATX_Clock.kicad_sch)
Changed lines of the file:
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@@
+		)
+	)
+	(sheet
+		(at 95.25 132.08)
+		(size 12.7 10.16)
+		(exclude_from_sim no)
+		(in_bom yes)
+		(on_board yes)
+		(dnp no)
+		(fields_autoplaced yes)
+		(stroke
+			(width 0.1524)
+			(type solid)
+		)
+		(fill
+			(color 0 0 0 0.0000)
+		)
+		(property "Sheetname" "Clock"
+			(at 95.25 131.3684 0)
+			(effects
+				(font
+					(size 1.27 1.27)
+				)
+				(justify left bottom)
+			)
+		)
+		(property "Sheetfile" "dATX_Clock.kicad_sch"
+			(at 95.25 142.8246 0)
+			(effects
+				(font
+					(size 1.27 1.27)
+				)
+				(justify left top)
+			)
+		)
+		(pin "CLK" output
+			(at 107.95 135.89 0)
+			(effects
+				(font
+					(size 1.27 1.27)
+				)
+				(justify right)
+			)
+		)
+		(pin "CLK2" output
+			(at 107.95 138.43 0)
+			(effects
+				(font
+					(size 1.27 1.27)
+				)
+				(justify right)
+			)
+		)
+		(instances
+			(project "dATX_JC100"
+				(path "/06d7853b-ec0e-46e4-9a93-83dad81d944c"
+					(page "2")
+				)
+			)
 		)
 	)

Commit message: lots
Parts:
- added C1: 120pF, Capacitor_THT:C_Disc_D3.0mm_W1.6mm_P2.50mm, symbol Device:C
- added C10, C11, C12, C13, C14, C7, C8, C9: 1uF, Capacitor_THT:CP_Radial_D4.0mm_P1.50mm, symbol Device:C_Polarized
- added C2: 100nF, Capacitor_THT:C_Disc_D3.0mm_W1.6mm_P2.50mm, symbol Device:C
- added C3: 1nF, Capacitor_THT:C_Disc_D3.0mm_W1.6mm_P2.50mm, symbol Device:C
- added C4, C5, C6: 100nF, symbol Device:C
- added D1: RESET, LED_THT:LED_D5.0mm, symbol Device:LED
- added D10: L7, LED_THT:LED_D5.0mm, symbol Device:LED
- added D11: L6, LED_THT:LED_D5.0mm, symbol Device:LED
- added D12: L5, LED_THT:LED_D5.0mm, symbol Device:LED
- added D13: L4, LED_THT:LED_D5.0mm, symbol Device:LED
- added D14: L3, LED_THT:LED_D5.0mm, symbol Device:LED
- added D15: L2, LED_THT:LED_D5.0mm, symbol Device:LED
- added D16: L1, LED_THT:LED_D5.0mm, symbol Device:LED
- added D2: CLK, LED_THT:LED_D5.0mm, symbol Device:LED
- added D3: CLK2, LED_THT:LED_D5.0mm, symbol Device:LED
- added D4: +5V, LED_THT:LED_D5.0mm, symbol Device:LED
- added D5: +12V, LED_THT:LED_D5.0mm, symbol Device:LED
- added D6: -12V, LED_THT:LED_D5.0mm, symbol Device:LED
- added D7: 3.3V, LED_THT:LED_D5.0mm, symbol Device:LED
- added D8: -5V, LED_THT:LED_D5.0mm, symbol Device:LED
- added D9: L8, LED_THT:LED_D5.0mm, symbol Device:LED
- added JP1: XOSC_CLK, symbol Jumper:Jumper_2_Bridged
- added JP10: CLK_SIOA, Connector_PinHeader_2.54mm:PinHeader_1x02_P2.54mm_Vertical, symbol Jumper:Jumper_2_Open
- added JP11: CLK2_SIOA, symbol Jumper:Jumper_2_Bridged
- added JP12: CTC_SIOA, Connector_PinHeader_2.54mm:PinHeader_1x02_P2.54mm_Vertical, symbol Jumper:Jumper_2_Open
- added JP13: CLK_SIOB, Connector_PinHeader_2.54mm:PinHeader_1x02_P2.54mm_Vertical, symbol Jumper:Jumper_2_Open
- added JP14: CLK2_SIOB, Connector_PinHeader_2.54mm:PinHeader_1x02_P2.54mm_Vertical, symbol Jumper:Jumper_2_Open
- added JP15: CTC_SIOB, symbol Jumper:Jumper_2_Bridged
- added JP2: XRES_CLK2, symbol Jumper:Jumper_2_Open
- added JP3: CLK_CLK2, symbol Jumper:SolderJumper_2_Open
- added JP4: RESET, Connector_PinHeader_2.54mm:PinHeader_1x02_P2.54mm_Vertical, symbol Jumper:Jumper_2_Open
- added JP5: RAM_SELECT, Connector_PinHeader_2.54mm:PinHeader_1x03_P2.54mm_Vertical, symbol Jumper:Jumper_3_Bridged12
- added JP6: ROM_SELECT, Connector_PinHeader_2.54mm:PinHeader_1x03_P2.54mm_Vertical, symbol Jumper:Jumper_3_Bridged12
- added JP7: ROM_WRITE, Connector_PinHeader_2.54mm:PinHeader_1x03_P2.54mm_Vertical, symbol Jumper:Jumper_3_Bridged12
- added JP8: CLK_CTC, Connector_PinHeader_2.54mm:PinHeader_1x02_P2.54mm_Vertical, symbol Jumper:Jumper_2_Open
- added JP9: CLK2_CTC, symbol Jumper:Jumper_2_Bridged
- added R1, R2: 330R, symbol Device:R
- added R10, R11, R12, R13, R14, R7, R8, R9: R, Resistor_THT:R_Axial_DIN0207_L6.3mm_D2.5mm_P10.16mm_Horizontal, symbol Device:R
- added R15, R18: 4K7, Resistor_THT:R_Axial_DIN0207_L6.3mm_D2.5mm_P10.16mm_Horizontal, symbol Device:R
- added R16: 10K, Resistor_THT:R_Axial_DIN0207_L6.3mm_D2.5mm_P10.16mm_Horizontal, symbol Device:R
- added R17, R19, R20, R21, R22, R27, R28, R33, R34: 100K, Resistor_THT:R_Axial_DIN0207_L6.3mm_D2.5mm_P10.16mm_Horizontal, symbol Device:R
- added R23, R24, R25, R26, R29, R30, R31, R32: 2K2, Resistor_THT:R_Axial_DIN0207_L6.3mm_D2.5mm_P10.16mm_Horizontal, symbol Device:R
- added R3, R4, R5, R6: 10K, symbol Device:R
- added RAM_0: AS6C4008, Package_DIP:DIP-32_W15.24mm, symbol Memory_RAM:AS6C4008-55PCN
- added RAM_1: IDT6116, Package_DIP:DIP-24_W15.24mm, symbol Carboni_Library:IDT6116
- added RN1: 1K, Resistor_THT:R_Array_SIP9, symbol Device:R_Network08
- added ROM_0, ROM_1: W27C512, Package_DIP:DIP-28_W15.24mm, symbol 8bitChips:W27C512
- added SW1: RESET, Button_Switch_THT:SW_PUSH_6mm, symbol Switch:SW_Push
- added U1: 74LS04, symbol 74xx:74LS04
- added U10, U11: MAX232, Package_DIP:DIP-16_W7.62mm_Socket, symbol Interface_UART:MAX232
- added U2: DS1233, Package_TO_SOT_THT:TO-92L_Inline, symbol Carboni_Library:DS1233
- added U3: 74AHCT125, symbol 74xx:74AHCT125
- added U4: 74HCT139, symbol 74xx:74LS139
- added U5: 74HCT688, symbol 74xx:74HCT688
- added U6, U9: 74HCT273, symbol 74xx:74HCT273
- added U7: 74HCT157, symbol 74xx:74LS157
- added U8: 74HCT138, symbol 74xx:74HCT138
- added XTAL_OSC_0: Crystal Oscillator, Oscillator:Oscillator_DIP-8, symbol Device:Crystal_GND24
- added XTAL_RES_0: Crystal Resonator, Crystal:Resonator-2Pin_W6.0mm_H3.0mm, symbol Device:Crystal
- ATX_PWR_0: value Conn_02x12_Top_Bottom -> Power Supply
Connections:
- net RXA: now reaches SIO_0.12 (RXDA)
- net RXA: now also R31.1
- net at SIO_0.13 (~{RXCA}): now also SIO_0.14 (~{TXCA}), JP10.2 (B), JP11.2 (B), JP12.2 (B)
- net TXA: now reaches SIO_0.15 (TXDA)
- net TXA: now also R32.1
- net at SIO_0.17 (~{RTSA}): now also R25.1
- net at SIO_0.18 (~{CTSA}): now also R26.1
- net GND: now reaches SIO_0.19 (~{DCDA})
- net GND: now also ATX_PWR_0.15 (Pin_15), ATX_PWR_0.17 (Pin_17), ATX_PWR_0.18 (Pin_18), ATX_PWR_0.19 (Pin_19), ATX_PWR_0.24 (Pin_24), ATX_PWR_0.3 (Pin_3), ATX_PWR_0.5 (Pin_5), ATX_PWR_0.7 (Pin_7), CPU_0.29 (GND), CTC_0.5 (GND), DMA_0.30 (GND), FPU_0.1 (VSS), PIO_0.11 (GND), SERIAL_0.5, SERIAL_1.5, SIO_0.22 (~{DCDB}), SIO_0.31 (GND), C1.2, C10.1, C14.1, C3.2, C4.1, C5.1, C6.1, JP4.2 (B), R10.1, R11.1, R12.1, R13.1, R14.1, R27.2, R28.2, R8.1, R9.1, RAM_0.16 (VSS), RAM_1.12 (GND), RN1.1 (common), ROM_0.14 (GND), ROM_1.14 (GND), SW1.2, U1.7 (GND), U10.15 (GND), U11.15 (GND), U2.1 (GND), U3.1, U3.12, U3.4, U3.7 (GND), U4.13 (A1), U4.3 (A1), U4.8 (GND), U5.10 (GND), U5.18 (R7), U5.3 (R0), U5.5 (R1), U5.7 (R2), U6.10 (GND), U7.15 (E), U7.8 (GND), U8.8 (GND), U9.10 (GND), XTAL_OSC_0.2
- net CLK: now reaches SIO_0.20 (F)
- net CLK: now also CPU_0.6 (CLK), CTC_0.15 (CLK), DMA_0.7 (CLK), D2.2 (A), JP1.2 (B), JP10.1 (A), JP13.1 (A), JP3.2 (B), JP8.2 (B)
- net RESET: now reaches SIO_0.21 (~{RESET})
- net RESET: now also CPU_0.26 (RESET), CTC_0.17 (~{RESET}), R18.1, U3.11, U3.5, U6.1 (~{Mr}), U9.1 (~{Mr})
- net at SIO_0.23 (~{CTSB}): now also R24.1
- net at SIO_0.24 (~{RTSB}): now also R23.1
- net TXB: now reaches SIO_0.26 (TXDB)
- net TXB: now also R30.1
- net at SIO_0.27 (~{TXCB}): now also SIO_0.28 (~{RXCB}), JP13.2 (B), JP14.2 (B), JP15.2 (B)
- net RXB: now reaches SIO_0.29 (RXDB)
- net RXB: now also R29.1
- net RD: now reaches SIO_0.32 (~{RD})
- net RD: now also CPU_0.21 (RD), CTC_0.6 (~{RD}), DMA_0.9 (~{RD}), RAM_0.24 (OE#), RAM_1.20 (~{OE}), ROM_0.22 (~{OE/Vpp}), ROM_1.22 (~{OE/Vpp})
- net at SIO_0.33 (C/~{D}): now also U1.8
- net at SIO_0.34 (B/~{A}): now also CTC_0.19 (CS1)
- net at SIO_0.35 (~{CE}): now also U8.15 (~{Y0})
- net IORQ: now reaches SIO_0.36 (~{IORQ})
- net IORQ: now also CPU_0.20 (IORQ), CTC_0.10 (~{IORQ}), DMA_0.12 (~{MREQ}), U5.1 (G)
- net INT: now reaches SIO_0.5 (~{INT})
- net INT: now also CPU_0.16 (INT), CTC_0.12 (~{INT}), R5.2
- net IE_1: now reaches SIO_0.6 (IEI)
- net IE_1: now also CTC_0.11 (IEO)
- net IE_2: now reaches SIO_0.7 (IEO)
- net IE_2: now also PIO_0.24 (IEI)
- net M1: now reaches SIO_0.8 (~{M1})
- net M1: now also CPU_0.27 (M1), CTC_0.14 (~{M1}), DMA_0.26 (~{M1})
- net +5V: now reaches SIO_0.9 (+5V)
- net +5V: now also ATX_PWR_0.21 (Pin_21), ATX_PWR_0.22 (Pin_22), ATX_PWR_0.23 (Pin_23), ATX_PWR_0.4 (Pin_4), ATX_PWR_0.6 (Pin_6), CPU_0.11 (VCC), CTC_0.24 (+5V), DMA_0.11 (VCC), DMA_0.38 (IEI), PIO_0.26 (VCC), C13.2, C4.2, C5.2, C6.2, C9.2, D1.2 (A), D4.2 (A), R15.1, R18.2, R19.1, R20.2, R21.1, R22.1, R3.1, R33.1, R34.1, R4.1, R5.1, R6.1, RAM_0.32 (VCC), RAM_1.24 (VCC), ROM_0.28 (VCC), ROM_1.28 (VCC), U1.14 (VCC), U10.16 (VCC), U11.16 (VCC), U2.3 (+5V), U3.14 (VCC), U4.16 (VCC), U5.12 (R4), U5.14 (R5), U5.16 (R6), U5.20 (VCC), U5.9 (R3), U6.17 (D6), U6.18 (D7), U6.20 (VCC), U6.3 (D0), U7.10 (I1c), U7.13 (I1d), U7.16 (VCC), U7.3 (I1a), U7.6 (I1b), U8.16 (VCC), U9.20 (VCC), XTAL_OSC_0.1, XTAL_OSC_0.4
- net at SERIAL_1.2: now also U11.13 (R1I)
- net at SERIAL_1.3: now also U11.14 (T1O)
- net at SERIAL_1.7: now also U11.7 (T2O)
- net at SERIAL_1.8: now also U11.8 (R2I)
- net IE_3: now reaches PIO_0.22 (IEO)
- net IE_0: now reaches CTC_0.13 (IEI)
- net IE_0: now also DMA_0.36 (IEO)
- net at CTC_0.16 (~{CE}): now also U8.13 (~{Y2})
- net at CTC_0.18 (CS0): now also U1.9
- net at CTC_0.20 (CLK/TRG3): now also CTC_0.21 (CLK/TRG2), CTC_0.22 (CLK/TRG1), CTC_0.23 (CLK/TRG0), CTC_0.9 (ZC/TO2), JP8.1 (A), JP9.1 (A)
- net at CTC_0.7 (ZC/TO0): now also JP12.1 (A)
- net at CTC_0.8 (ZC/TO1): now also JP15.1 (A)
- net NMI: now reaches CPU_0.17 (NMI)
- net NMI: now also R4.2
- net HALT: now reaches CPU_0.18 (HALT)
- net MREQ: now reaches CPU_0.19 (MREQ)
- net MREQ: now also DMA_0.10 (~{IORQ}), U4.1 (E)
- net WR: now reaches CPU_0.22 (WR)
- net WR: now also DMA_0.8 (~{WR}), RAM_0.29 (WE#), RAM_1.21 (~{WE}), U3.9, U5.2 (P0)
- net BUSAK: now reaches CPU_0.23 (BUSAK)
- net WAIT: now reaches CPU_0.24 (WAIT)
- net WAIT: now also R6.2
- net BUSRQ: now reaches CPU_0.25 (BUSRQ)
- net BUSRQ: now also R3.2
- net RFSH: now reaches CPU_0.28 (RFSH)
- net at SERIAL_0.2: now also U10.13 (R1I)
- net at SERIAL_0.3: now also U10.14 (T1O)
- net at SERIAL_0.7: now also U10.7 (T2O)
- net at SERIAL_0.8: now also U10.8 (R2I)
- net +3.3V: now reaches ATX_PWR_0.1 (Pin_1)
- net +3.3V: now also ATX_PWR_0.12 (Pin_12), ATX_PWR_0.13 (Pin_13), ATX_PWR_0.2 (Pin_2), D7.2 (A)
- net +12V: now reaches ATX_PWR_0.10 (Pin_10)
- net +12V: now also ATX_PWR_0.11 (Pin_11), D5.2 (A)
- net -12V: now reaches ATX_PWR_0.14 (Pin_14)
- net -12V: now also D6.2 (A)
- net PS_ON: now reaches ATX_PWR_0.16 (Pin_16)
- net -5V: now reaches ATX_PWR_0.20 (Pin_20)
- net -5V: now also D8.2 (A)
- net PWR_OK: now reaches ATX_PWR_0.8 (Pin_8)
- net +5VSB: now reaches ATX_PWR_0.9 (Pin_9)
- new net: D6.1 (K), R12.2
- new net: JP6.1 (A), R22.2, ROM_0.20 (~{CE})
- new net: JP6.3 (B), R21.2, ROM_1.20 (~{CE})
- new net: D7.1 (K), R13.2
- new net: D4.1 (K), R10.2
- new net: R31.2, R34.2, U10.12 (R1O)
- new net: D16.1 (K), RN1.9 (R8)
- new net: D16.2 (A), U9.19 (Q7)
- new net: D8.1 (K), R14.2
- new net: R17.2, U3.13, U3.3
- new net: U3.10, U8.11 (~{Y4})
- new net: C11.1, U11.1 (C1+)
- new net: R23.2, U11.10 (T2I)
- new net: R30.2, U11.11 (T1I)
- new net: R29.2, R33.2, U11.12 (R1O)
- new net: C13.1, U11.2 (VS+)
- new net: C11.2, U11.3 (C1-)
- new net: C12.1, U11.4 (C2+)
- new net: C12.2, U11.5 (C2-)
- new net: C14.2, U11.6 (VS-)
- new net: R24.2, R27.1, U11.9 (R2O)
- new net: D10.1 (K), RN1.3 (R2)
- new net: D10.2 (A), U9.5 (Q1)
- new net: D9.1 (K), RN1.2 (R1)
- new net: D9.2 (A), U9.2 (Q0)
- new net: R7.2, U3.6
- new net: D5.1 (K), R11.2
- new net: C7.1, U10.1 (C1+)
- new net: C7.2, U10.3 (C1-)
- new net: C3.1, JP4.1 (A), R15.2, R16.1, SW1.1, U2.2 (RESET)
- new net: D2.1 (K), R8.2
- new net: JP1.1 (A), XTAL_OSC_0.3
- new net: D3.1 (K), R9.2
- new net: U3.8, U9.11 (Cp)
- new net: C9.1, U10.2 (VS+)
- new net: D12.1 (K), RN1.5 (R4)
- new net: D12.2 (A), U9.9 (Q3)
- new net: C1.1, R1.1, U1.1, XTAL_RES_0.1
- new net: R2.2, U1.4, U1.5, XTAL_RES_0.2
- new net: D15.1 (K), RN1.8 (R7)
- new net: D15.2 (A), U9.16 (Q6)
- new net: C2.1, R1.2, U1.2
- new net: JP2.1 (A), U1.6
- new net: R25.2, U10.10 (T2I)
- new net: R32.2, U10.11 (T1I)
- new net: C8.1, U10.4 (C2+)
- new net: C8.2, U10.5 (C2-)
- new net: C10.2, U10.6 (VS-)
- new net: R26.2, R28.1, U10.9 (R2O)
- new net: JP5.1 (A), R19.2, RAM_0.22 (CE#)
- new net: JP5.3 (B), R20.1, RAM_1.18 (~{CS})
- new net: R16.2, R17.1, U3.2
- new net: D14.1 (K), RN1.7 (R6)
- new net: D14.2 (A), U9.15 (Q5)
- new net: C2.2, R2.1, U1.3
- new net: U5.19 (P=R), U6.11 (Cp)
- new net: D11.1 (K), RN1.4 (R3)
- new net: D11.2 (A), U9.6 (Q2)
- new net: D13.1 (K), RN1.6 (R5)
- new net: U4.12 (O0), U4.2 (A0)
- new net: D1.1 (K), R7.1
- new net: U4.14 (A0), U6.15 (Q5)
- new net: D13.2 (A), U9.12 (Q4)
- new net: U6.12 (Q4), U7.14 (I0d)
- new net: U6.5 (Q1), U7.2 (I0a)
- new net: U6.6 (Q2), U7.5 (I0b)
- new net: U6.9 (Q3), U7.11 (I0c)
- new net CLK2: D3.2 (A), JP11.1 (A), JP14.1 (A), JP2.2 (B), JP3.1 (A), JP9.2 (B)
- new net MA15: RAM_0.31 (A15), ROM_0.1 (A15), ROM_1.1 (A15), U7.4 (Za)
- new net MA16: RAM_0.2 (A16), U7.7 (Zb)
- new net MA17: RAM_0.30 (A17), U7.9 (Zc)
- new net MA18: RAM_0.1 (A18), U7.12 (Zd)
- new net SEL_RAM: JP5.2 (C), U4.5 (O1)
- new net SEL_ROM: JP6.2 (C), U4.4 (O0)
- no-connect marks 0 -> 21
Other:
- removed sheet Clock
- note added: "-5V deprecated in ATX 2.0"
- note added: "A0"
- note added: "A1"
- note added: "A1-7"
- note added: "A15"
- note added: "A2-7"
- note added: "Bus Output LEDs"
- note added: "Clock Generator"
- note added: "D1-5"
- note added: "I/O write to 0x78 or 0x79 = 0111 100X"
- note added: "If SIO baud rate using CLK2: Must be less than half rate of CLK due to internal sync of CTC."
- note added: "Inverter for compatibility with RC2014 software."
- note added: "JP10-15 select clock source for SIO (A&B): CTC, CLK, or CLK2"
- note added: "JP8-9 select clock source for CTC: CLK or CLK2"
- note added: "LA15-18"
- note added: "LA19"
- note added: "MA19"
- note added: "Memory Management Unit"
- note added: "Power Decoupling"
- note added: "Power and Clock LEDs"
- note added: "RAM and ROM"
- note added: "RESET: Open collector, active low."
- note added: "RS-232 Serial"
- note added: "RS-232_0 (Port A)"
- note added: "RS-232_1 (Port B)"
- note added: "Recommended CLK: 1.00 - 8.00 MHz (safe). 100 kHz (min), 4.00 MHz (best*), 20.0 MHz (max). Recommended CLK2: 1.8432 MHz (safe), 7.3728 MHz (best**). *For speeds >4 MHz, Am9511 must divide clock. **Only use strictly if CLK is CLK2 (JP3 closed)."
- note added: "Reset and Voltage Supervisor"
- note added: "SEL Lo: Zx = I0x SEL Hi: Zx = I1x"
- note added: "SIO Port A clk"
- note added: "SIO Port B clk"
- note added: "Y0: /SIO = /IORQ 0x80 Y2: /CTC = /IORQ 0x88 Y4: /LIO = /IORQ 0x90"
- company: (none) -> Jules Carboni
- title: (none) -> Project Carbon Z80 Motherboard
- moved on the sheet: ATX_PWR_0, CPU_0, CTC_0, DMA_0, FLOPPY_0, FPU_0, JCBUS_0, JCBUS_1, JCBUS_2, JCBUS_3, JCBUS_4, JCBUS_5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

Commit message: heaps
Parts:
- removed JP7: ROM_WRITE, Connector_PinHeader_2.54mm:PinHeader_1x03_P2.54mm_Vertical, symbol Jumper:Jumper_3_Bridged12
- removed KEYBD_0, MOUSE_0: Mini-DIN-6, Carboni_Library:Mini_DIN_6, symbol Connector:Mini-DIN-6
- added C15, C18, C19: 100nF, symbol Device:C
- added C16, C17: 100nF, Capacitor_THT:C_Disc_D3.0mm_W1.6mm_P2.50mm, symbol Device:C
- added D17: BUSY, LED_THT:LED_D5.0mm, symbol Device:LED
- added JP16: TX1, Connector_PinHeader_2.54mm:PinHeader_1x03_P2.54mm_Vertical, symbol Jumper:Jumper_3_Open
- added JP17: RX1, Connector_PinHeader_2.54mm:PinHeader_1x03_P2.54mm_Vertical, symbol Jumper:Jumper_3_Open
- added JP18: TX2, Connector_PinHeader_2.54mm:PinHeader_1x03_P2.54mm_Vertical, symbol Jumper:Jumper_3_Open
- added JP19: RX2, Connector_PinHeader_2.54mm:PinHeader_1x03_P2.54mm_Vertical, symbol Jumper:Jumper_3_Open
- added R35: 100K, Resistor_THT:R_Axial_DIN0207_L6.3mm_D2.5mm_P10.16mm_Horizontal, symbol Device:R
- added R36: 1K, Resistor_THT:R_Axial_DIN0207_L6.3mm_D2.5mm_P10.16mm_Horizontal, symbol Device:R
- added R37: 10K, Resistor_THT:R_Axial_DIN0207_L6.3mm_D2.5mm_P10.16mm_Horizontal, symbol Device:R
- added R38, R39, R40, R41: 4K7, Resistor_THT:R_Axial_DIN0207_L6.3mm_D2.5mm_P10.16mm_Horizontal, symbol Device:R
- added SW2: RESET, Button_Switch_THT:SW_PUSH_6mm, symbol Switch:SW_Push
- added U12: 74LS00, symbol 74xx:74LS00
- added U13: 74HCT74, symbol 74xx:74HCT74
- added U14: 74LS32, symbol 74xx:74LS32
- added U15: 74HCT138, symbol 74xx:74HCT138
- FDD_0: renamed from FLOPPY_0; value Conn_02x17_Odd_Even -> Floppy_IBM
- IDE_0: renamed from PATA_0; value Conn_02x20_Odd_Even -> CompactFlash
- TS_0: renamed from TAPE_OUT_0; value AudioJack2 -> TAPE_IN
- TS_1: renamed from TAPE_IN_0; value AudioJack2 -> TAPE_OUT
Connections:
- net +5V: now also FPU_0.2 (VCC), IDE_0.20 (Pin_20), C15.2, C18.2, C19.2, D17.2 (A), R38.2, R39.2, R41.2, U12.14 (VCC), U13.10 (~{S}), U13.4 (~{S}), U13.7 (GND), U14.7 (GND), U15.16 (VCC); no longer C4.2, U1.14 (VCC)
- net +5VSB: now also C4.2, U1.14 (VCC), C17.1
- net CLK: now also PIO_0.25 (CLK), U13.11 (C), U13.3 (C), U14.10, U14.13
- net GND: now also IDE_0.19 (Pin_19), IDE_0.2 (Pin_2), IDE_0.22 (Pin_22), IDE_0.24 (Pin_24), IDE_0.26 (Pin_26), IDE_0.30 (Pin_30), IDE_0.40 (Pin_40), C15.1, C16.1, C18.1, C19.1, U12.7 (GND), U13.14 (VCC), U14.14 (VCC), U14.4, U15.8 (GND)
- net INT: now also PIO_0.23 (~{INT})
- net IORQ: now also PIO_0.36 (~{IORQ}), U13.13 (~{R})
- net M1: now also U12.2, U15.6 (E2)
- net PS_ON: now also U1.12, R37.1
- net RD: now also PIO_0.35 (~{RD}), U13.2 (D), U14.12
- net RESET: now also IDE_0.1 (Pin_1), U12.1
- net RXA: now also JP17.1 (A)
- net RXB: now also JP17.3 (B), JP19.1 (A)
- net TXA: now also JP16.1 (A)
- net TXB: now also JP16.3 (B), JP18.1 (A)
- net WR: now also U14.1
- net RTSA: now reaches R25.1, SIO_0.17 (~{RTSA})
- net RTSA: now also JP18.3 (B)
- net CTSA: now reaches R26.1, SIO_0.18 (~{CTSA})
- net CTSA: now also JP19.3 (B)
- net at U1.10: now also U1.13, R35.2
- net at U1.11: now also C17.2, R36.1
- net SEL_PIO: now reaches U8.9 (~{Y6})
- net SEL_PIO: now also PIO_0.4 (~{CE})
- net IRQ_IDE: now reaches PIO_0.10 (PA4)
- net IRQ_FDC: now reaches PIO_0.12 (PA3)
- net IRQ_TAPE: now reaches PIO_0.13 (PA2)
- net IRQ_FPU: now reaches PIO_0.14 (PA1)
- net IRQ_PS2: now reaches PIO_0.15 (PA0)
- net IRQ0: now reaches PIO_0.27 (PB0)
- net IRQ1: now reaches PIO_0.28 (PB1)
- net IRQ2: now reaches PIO_0.29 (PB2)
- net IRQ3: now reaches PIO_0.30 (PB3)
- net IRQ4: now reaches PIO_0.31 (PB4)
- net IRQ5: now reaches PIO_0.32 (PB5)
- net IRQ6: now reaches PIO_0.33 (PB6)
- net IRQ7: now reaches PIO_0.34 (PB7)
- net at PIO_0.37 (~{M1}): now also U12.6
- net IDER: now reaches IDE_0.23 (Pin_23)
- net IDER: now also U14.8
- net IDEW: now reaches IDE_0.25 (Pin_25)
- net IDEW: now also U14.6
- net at IDE_0.29 (Pin_29): now also R41.1
- net at IDE_0.34 (Pin_34): now also R38.1
- net at IDE_0.37 (Pin_37): now also U14.2, U15.15 (~{Y0})
- net at IDE_0.38 (Pin_38): now also R39.1
- net at IDE_0.39 (Pin_39): now also R40.1
- new net: U13.1 (~{R}), U14.11
- new net: U13.5 (Q), U14.9
- new net: R36.2, R37.2, SW2.1
- new net: U14.3, U14.5
- new net: D17.1 (K), R40.2
- new net: U13.9 (Q), U15.5 (~{E1})
- new net: C16.2, R35.1, SW2.2
- new net: U12.3, U12.4, U12.5
- new net RX: JP17.2 (C)
- new net RX2: JP19.2 (C)
- new net TX: JP16.2 (C)
- new net TX2: JP18.2 (C)
- no-connect marks 21 -> 49
Other:
- note added: "(20 = keypin)"
- note added: "-5V deprecated in ATX 1.3"
- note added: "2KB SRAM"
- note added: "512KB SRAM 55ns access time."
- note added: "64KB E/EPROM 45ns access time. No write enable."
- note added: "64KB E/EPROM Optional alternate ROM"
- note added: "A2"
- note added: "A3"
- note added: "A4"
- note added: "A5"
- note added: "A6"
- note added: "A7"
- note added: "ATX Power Switch"
- note added: "BUSY when IDE R/W."
- note added: "Chipset Device SEL Decode"
- note added: "DIO"
- note added: "PCB ideally has 2x IDT6116 for 4KB, selected by line A11 && SEL_RAM. W27C512 does not support erasure."
- note added: "PIO for Mode 2 interrupt routing from chipset and expansion devices."
- note added: "Project Carbon Z80 Microcomputer Jules Carboni August 2025"
- note added: "U1 requires +5VSB for POWER switch."
- note added: "Y0: /IDE = 0001 0xxx"
- note added: "Y0: /SIO = /IORQ 0x80 Y2: /CTC = /IORQ 0x88 Y4: /LIO = /IORQ 0x90 Y6: /PIO = /IORQ 0x98"
- note removed: "-5V deprecated in ATX 2.0"
- note removed: "A2-7"
- note removed: "Y0: /SIO = /IORQ 0x80 Y2: /CTC = /IORQ 0x88 Y4: /LIO = /IORQ 0x90"
- moved on the sheet: C3, D1, D2, D3, D4, D5, D6, D7, D8, FDD_0, FPU_0, IDE_0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

Commit message: yee
Parts:
- added C20, C23: 100nF, symbol Device:C
- added C21: 120pF, Capacitor_THT:C_Disc_D3.0mm_W1.6mm_P2.50mm, symbol Device:C
- added C22: 100nF, Capacitor_THT:C_Disc_D3.0mm_W1.6mm_P2.50mm, symbol Device:C
- added JP7: XRES_CLK2, symbol Jumper:Jumper_2_Open
- added R42, R43: 330R, symbol Device:R
- added U16: 74LS00, Package_DIP:DIP-14_W7.62mm, symbol 74xx:74LS00
- added U17: 74LS00, symbol 74xx:74LS00
- added U18: 74LS04, symbol 74xx:74LS04
- added XTAL_RES_1: Crystal Resonator, Crystal:Resonator-2Pin_W6.0mm_H3.0mm, symbol Device:Crystal
- JCBUS_0, JCBUS_1, JCBUS_2, JCBUS_3, JCBUS_4, JCBUS_5: value Conn_02x50_Row_Letter_First -> JC100
- U1, U12, U13, U14, U3: footprint (none) -> Package_DIP:DIP-14_W7.62mm
- U15, U4, U8: footprint (none) -> Package_DIP:DIP-16_W7.62mm
- U9: footprint (none) -> Package_DIP:DIP-20_W7.62mm
Connections:
- net IRQ_PS2 is gone; now on net IRQ_FPU: PIO_0.15 (PA0)
- net +5V: now also C4.2, U1.14 (VCC), C23.2, U18.7 (GND)
- net +5VSB: now also C20.2, U16.7 (GND); no longer C4.2, U1.14 (VCC)
- net GND: now also C20.1, C21.2, C23.1, U16.14 (VCC), U18.14 (VCC)
- net IORQ: now also U12.9
- net IRQ_FDC: now also PIO_0.13 (PA2); no longer PIO_0.12 (PA3)
- net IRQ_FPU: no longer PIO_0.14 (PA1)
- net IRQ_IDE: now also PIO_0.12 (PA3); no longer PIO_0.10 (PA4)
- net IRQ_TAPE: now also PIO_0.14 (PA1); no longer PIO_0.13 (PA2)
- net PS_ON: now also U16.6; no longer U1.12
- net at U1.10, U1.13: no longer R35.2
- net at C17.2, R36.1: now also U17.1, U17.2; no longer U1.11
- net at U8.5 (~{E1}): now also U12.11
- net at IDE_0.37 (Pin_37), U14.2: now also U15.9 (~{Y6}); no longer U15.15 (~{Y0})
- net SEL_FDC: now reaches U15.11 (~{Y4})
- net SEL_TAPE: now reaches U15.13 (~{Y2})
- net at U12.8: now also U12.12, U12.13
- new net: C21.1, R42.1, U18.1, XTAL_RES_1.1
- new net: C22.1, R42.2, U18.2
- new net: C22.2, R43.1, U18.3
- new net: R43.2, U18.4, U18.5, XTAL_RES_1.2
- new net: R35.2, U16.4, U16.5, U17.3
- new net: JP7.1 (A), U18.6
- new net SEL_FPU: U15.15 (~{Y0})
- no-connect marks 49 -> 46
Other:
- note added: "JP8-9 select clock source for CTC: CLK or CLK2 JP10-15 select clock source for SIO (A&B): CTC, CLK, or CLK2"
- note added: "SEL_IDE"
- note added: "U14 requires +5VSB for ATX POWER switch."
- note added: "Y0: /FPU = 0x80 Y2: /TAP = 0x88 Y4: /FDC = 0x90 Y6: /IDE = 0x98"
- note removed: "JP10-15 select clock source for SIO (A&B): CTC, CLK, or CLK2"
- note removed: "JP8-9 select clock source for CTC: CLK or CLK2"
- note removed: "U1 requires +5VSB for POWER switch."
- note removed: "Y0: /IDE = 0001 0xxx"
- moved on the sheet: C16, C17, FDD_0, FPU_0, JCBUS_0, JCBUS_1, JCBUS_2, JCBUS_3, JCBUS_4, JCBUS_5, R3, R35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

Commit message: yurr
Parts:
- removed C22: 100nF, Capacitor_THT:C_Disc_D3.0mm_W1.6mm_P2.50mm, symbol Device:C
- removed C23: 100nF, symbol Device:C
- removed JP7: XRES_CLK2, symbol Jumper:Jumper_2_Open
- removed U18: 74LS04, symbol 74xx:74LS04
- added C24, C27: 120pF, Capacitor_THT:C_Disc_D3.0mm_W1.6mm_P2.50mm, symbol Device:C
- added C25, C28: 100nF, Capacitor_THT:C_Disc_D3.0mm_W1.6mm_P2.50mm, symbol Device:C
- added C26: 100nF, symbol Device:C
- added FDC_0: GM82C765B, Package_DIP:DIP-40_W15.24mm_Socket, symbol Carboni_Library:GM82C765B
- added JP20: CLK_FDC_CLK, symbol Jumper:SolderJumper_2_Open
- added JP21: PWR_FDC_12, symbol Jumper:SolderJumper_2_Open
- added JP22: PWR_FDC_5, symbol Jumper:SolderJumper_2_Open
- added JP23: FDC_JP1, Connector_PinHeader_2.54mm:PinHeader_1x03_P2.54mm_Vertical, symbol Jumper:Jumper_3_Open
- added JP24: FDC_JP2, Connector_PinHeader_2.54mm:PinHeader_1x03_P2.54mm_Vertical, symbol Jumper:Jumper_3_Open
- added JP7: CLK_FDC_RES, symbol Jumper:SolderJumper_2_Open
- added R44: 10K, Resistor_THT:R_Axial_DIN0207_L6.3mm_D2.5mm_P10.16mm_Horizontal, symbol Device:R
- added R45, R46, R47, R48, R49: 330R, symbol Device:R
- added RN2: 10K, Resistor_THT:R_Array_SIP9, symbol Device:R_Network08
- added U18: 74AHCT125, symbol 74xx:74AHCT125
- added U19: 74LS04, Package_DIP:DIP-14_W7.62mm, symbol 74xx:74LS04
- added U20: 74HCT138, symbol 74xx:74HCT138
- added XTAL_RES_2: XTAL RES FDC 9.6MHz, Crystal:Resonator-2Pin_W6.0mm_H3.0mm, symbol Device:Crystal
- C21: value 120pF -> 100nF; footprint Capacitor_THT:C_Disc_D3.0mm_W1.6mm_P2.50mm -> (none)
- D17: value BUSY -> BUSY_IDE
- R42: value 330R -> 1K; footprint (none) -> Resistor_THT:R_Axial_DIN0207_L6.3mm_D2.5mm_P10.16mm_Horizontal
- XTAL_RES_1: value Crystal Resonator -> XTAL RES FDC 16MHz
- renumbered U16 to U0
Connections:
- net +12V: now also FPU_0.16 (VDD), JP21.2 (B)
- net +5V: now also C21.2, R43.1, C26.2, FDC_0.24 (PCVAL), FDC_0.40 (VCC), JP22.2 (B), JP24.3 (B), R44.1, RN2.1 (common), U18.12, U18.14 (VCC), U18.9, U19.7 (GND), U20.16 (VCC), U20.6 (E2)
- net CLK: now also JP20.1 (A)
- net GND: now also C21.1, FDD_0.1 (Pin_1), FDD_0.11 (Pin_11), FDD_0.13 (Pin_13), FDD_0.15 (Pin_15), FDD_0.17 (Pin_17), FDD_0.19 (Pin_19), FDD_0.21 (Pin_21), FDD_0.23 (Pin_23), FDD_0.25 (Pin_25), FDD_0.27 (Pin_27), FDD_0.29 (Pin_29), FDD_0.31 (Pin_31), FDD_0.33 (Pin_33), FDD_0.4 (Pin_4), FDD_0.5 (Pin_5), FDD_0.7 (Pin_7), FDD_0.9 (Pin_9), R42.2, C24.2, C26.1, C27.2, FDC_0.22 (DRV), FDC_0.31 (VSS), R49.1, U18.7 (GND), U19.14 (VCC), U20.5 (~{E1}), U20.8 (GND); no longer C21.2
- net IRQ_FPU: now also FPU_0.24 (~{END})
- net RD: now also FDC_0.1 (~{RD}), U18.5
- net RESET: now also U1.11, U18.13
- net SEL_FDC: now also U20.4 (~{E0})
- net SEL_FPU: now also FPU_0.18 (~{CS})
- net WAIT: now also FPU_0.17 (~{PAUSE})
- net WR: now also FDC_0.2 (~{WR})
- net at U1.13: no longer U1.10
- net at R43.2: now also FDC_0.5 (~{DACK}), JP23.2 (C); no longer XTAL_RES_1.2
- net at FPU_0.22 (RESET): now also U1.10
- net CLK_FPU: now reaches FPU_0.23 (CLK)
- net at FPU_0.3 (~{EACK}): now also R44.2
- net at FDD_0.10 (Pin_10): now also FDC_0.33 (~{DS3}~{MO1})
- net at FDD_0.12 (Pin_12): now also FDC_0.32 (~{DS2})
- net at FDD_0.14 (Pin_14): now also FDC_0.30 (~{DS1})
- net at FDD_0.16 (Pin_16): now also FDC_0.34 (~{DS4}~{MO2})
- net at FDD_0.18 (Pin_18): now also FDC_0.28 (~{DIRC})
- net at FDD_0.2 (Pin_2): now also FDC_0.36 (~{RPM}~{RWC})
- net at FDD_0.20 (Pin_20): now also FDC_0.29 (~{STEP})
- net at FDD_0.22 (Pin_22): now also FDC_0.27 (~{WD})
- net at FDD_0.24 (Pin_24): now also FDC_0.26 (~{WE})
- net at FDD_0.26 (Pin_26): now also FDC_0.38 (~{TR00}), RN2.3 (R2)
- net at FDD_0.28 (Pin_28): now also FDC_0.37 (WP), RN2.4 (R3)
- net at FDD_0.3 (Pin_3): now also JP22.1 (A)
- net at FDD_0.30 (Pin_30): now also FDC_0.20 (~{RDD}), RN2.6 (R5)
- net at FDD_0.32 (Pin_32): now also FDC_0.25 (~{HS})
- net at FDD_0.34 (Pin_34): now also FDD_0.8 (Pin_8), FDC_0.39 (~{IDX}), RN2.2 (R1), RN2.5 (R4), U18.2
- net at FDD_0.6 (Pin_6): now also JP21.1 (A)
- new net: FDC_0.19 (RST), R42.1, U18.11
- new net: JP23.1 (A), U18.6
- new net: JP23.3 (B), U20.15 (~{Y0})
- new net: C28.2, R48.1, U19.11
- new net: R48.2, U19.10, U19.13, XTAL_RES_2.2
- new net: R46.2, U19.4, U19.5, XTAL_RES_1.2
- new net: JP7.1 (A), U19.6
- new net: C25.2, R46.1, U19.3
- new net: C27.1, R47.1, U19.9, XTAL_RES_2.1
- new net: C28.1, R47.2, U19.8
- new net: C25.1, R45.2, U19.2
- new net: FDC_0.6 (TC), JP24.2 (C), R49.2
- new net: U18.10, U20.14 (~{Y1})
- new net: JP24.1 (A), U18.8
- new net: U18.1, U20.7 (~{Y7})
- new net: FDC_0.17 (~{LDOR}), U18.4, U20.9 (~{Y6})
- new net: FDC_0.18 (~{LDCR}), U20.13 (~{Y2})
- new net: FDC_0.3 (~{CS}), U20.11 (~{Y4})
- new net: C24.1, R45.1, U19.1, XTAL_RES_1.1
- new net CLK_FDC16: FDC_0.23 (CLK1), JP20.2 (B), JP7.2 (B)
- new net CLK_FDC96: FDC_0.21 (CLK2), U19.12
- no-connect marks 46 -> 52
Other:
- note added: "37C65 FDC"
- note added: "Connect SVREQ/ACK to spare IO pins?"
- note added: "Control Signal Pullups"
- note added: "D7"
- note added: "DACK"
- note added: "DMA Controller"
- note added: "FDC 16.0 MHz"
- note added: "FDC 9.6 MHz"
- note added: "Floating Point Unit"
- note added: "Floppy Disk Controller"
- note added: "IBM Floppy 34 Pin"
- note added: "PATA IDE 40 Pin"
- note added: "TC"
- note added: "U0 requires +5VSB for ATX POWER switch."
- note added: "Y0: +00 = DACK (opt) Y1: +04 = TC (opt) Y2: +08 = CCR Y4: +10 = CS Y6: +18 = DOR Y7: +1C = DC"
- note added: "Z80 CPU NMOS/CMOS <20 MHz"
- note added: "check caps if need to be polarized eg 1nf"
- note added: "check which ic need to be socket or directrly soldered"
- note removed: "U14 requires +5VSB for ATX POWER switch."
- moved on the sheet: C15, C16, C17, C18, C19, C20, C4, C5, C6, DMA_0, FDD_0, FPU_0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
