File: schematics/dATX_JC100.kicad_sch (KiCad schematic)
At the start: 169 parts, among them SW1 RESET, SW2 RESET, U0 74LS00, U1 74LS04, U10 MAX232, U11 MAX232, U12 74LS00, U13 74HCT74, U14 74LS32, U15 74HCT138, U16 74LS00, U17 74LS00, U18 74AHCT125, U19 74LS04, U2 DS1233, U20 74HCT138, U3 74AHCT125, U4 74HCT139, U5 74HCT688, U6 74HCT273, U7 74HCT157, U8 74HCT138, U9 74HCT273

Commit message: pres
Parts:
- removed TS_0: TAPE_IN, Jack_3.5mm_CUI_SJ1-3525N_Horizontal, symbol Connector_Audio:AudioJack2
- removed TS_1: TAPE_OUT, Jack_3.5mm_CUI_SJ1-3525N_Horizontal, symbol Connector_Audio:AudioJack2
- added C22, C23: 100nF, symbol Device:C
- added JP25: CLK_FPU_CLK2, symbol Jumper:SolderJumper_2_Open
- added JP26: CLK_FPU_CLK, symbol Jumper:SolderJumper_2_Open
- added JP27: POWER, Connector_PinHeader_2.54mm:PinHeader_1x02_P2.54mm_Vertical, symbol Jumper:Jumper_2_Open
- added JP28: FPU_CLKd1, Connector_PinHeader_2.54mm:PinHeader_1x02_P2.54mm_Vertical, symbol Jumper:Jumper_2_Open
- added JP29: FPU_CLKd2, Connector_PinHeader_2.54mm:PinHeader_1x02_P2.54mm_Vertical, symbol Jumper:Jumper_2_Open
- added JP30: FPU_CLKd4, Connector_PinHeader_2.54mm:PinHeader_1x02_P2.54mm_Vertical, symbol Jumper:Jumper_2_Open
- added U21: 74LS74, Package_DIP:DIP-14_W7.62mm, symbol 74xx:74LS74
- added U22: 74LS139, Package_DIP:DIP-16_W7.62mm, symbol 74xx:74LS139
- CTC_0, ROM_0, ROM_1: footprint Package_DIP:DIP-28_W15.24mm -> Package_DIP:DIP-28_W15.24mm_Socket
- DMA_0, PIO_0, SIO_0: footprint Package_DIP:DIP-40_W15.24mm -> Package_DIP:DIP-40_W15.24mm_Socket
- FPU_0, RAM_1: footprint Package_DIP:DIP-24_W15.24mm -> Package_DIP:DIP-24_W15.24mm_Socket
- RAM_0: footprint Package_DIP:DIP-32_W15.24mm -> Package_DIP:DIP-32_W15.24mm_Socket
- SW2: value RESET -> POWER
- U18: footprint (none) -> Package_DIP:DIP-14_W7.62mm
- U20, U7: footprint (none) -> Package_DIP:DIP-16_W7.62mm
- U5, U6: footprint (none) -> Package_DIP:DIP-20_W7.62mm
Connections:
- net +12V: now also JCBUS_0.b2 (Pin_b2), JCBUS_0.b50 (Pin_b50), JCBUS_1.b2 (Pin_b2), JCBUS_1.b50 (Pin_b50), JCBUS_2.b2 (Pin_b2), JCBUS_2.b50 (Pin_b50), JCBUS_3.b2 (Pin_b2), JCBUS_3.b50 (Pin_b50), JCBUS_4.b2 (Pin_b2), JCBUS_4.b50 (Pin_b50), JCBUS_5.b2 (Pin_b2), JCBUS_5.b50 (Pin_b50)
- net +3.3V: now also JCBUS_0.b4 (Pin_b4), JCBUS_1.b4 (Pin_b4), JCBUS_2.b4 (Pin_b4), JCBUS_3.b4 (Pin_b4), JCBUS_4.b4 (Pin_b4), JCBUS_5.b4 (Pin_b4)
- net +5V: now also JCBUS_0.b1 (Pin_b1), JCBUS_0.b49 (Pin_b49), JCBUS_1.b1 (Pin_b1), JCBUS_1.b49 (Pin_b49), JCBUS_2.b1 (Pin_b1), JCBUS_2.b49 (Pin_b49), JCBUS_3.b1 (Pin_b1), JCBUS_3.b49 (Pin_b49), JCBUS_4.b1 (Pin_b1), JCBUS_4.b49 (Pin_b49), JCBUS_5.b1 (Pin_b1), JCBUS_5.b49 (Pin_b49), C22.2, C23.2, U21.7 (GND), U22.8 (GND)
- net -12V: now also JCBUS_0.b3 (Pin_b3), JCBUS_1.b3 (Pin_b3), JCBUS_2.b3 (Pin_b3), JCBUS_3.b3 (Pin_b3), JCBUS_4.b3 (Pin_b3), JCBUS_5.b3 (Pin_b3)
- net CLK: now also JCBUS_0.b7 (Pin_b7), JCBUS_1.b7 (Pin_b7), JCBUS_2.b7 (Pin_b7), JCBUS_3.b7 (Pin_b7), JCBUS_4.b7 (Pin_b7), JCBUS_5.b7 (Pin_b7), JP26.2 (B)
- net CLK2: now also JCBUS_0.b5 (Pin_b5), JCBUS_1.b5 (Pin_b5), JCBUS_2.b5 (Pin_b5), JCBUS_3.b5 (Pin_b5), JCBUS_4.b5 (Pin_b5), JCBUS_5.b5 (Pin_b5), JP25.2 (B)
- net GND: now also JCBUS_0.a1 (Pin_a1), JCBUS_0.a2 (Pin_a2), JCBUS_0.a3 (Pin_a3), JCBUS_0.a4 (Pin_a4), JCBUS_0.a49 (Pin_a49), JCBUS_0.a50 (Pin_a50), JCBUS_1.a1 (Pin_a1), JCBUS_1.a2 (Pin_a2), JCBUS_1.a3 (Pin_a3), JCBUS_1.a4 (Pin_a4), JCBUS_1.a49 (Pin_a49), JCBUS_1.a50 (Pin_a50), JCBUS_2.a1 (Pin_a1), JCBUS_2.a2 (Pin_a2), JCBUS_2.a3 (Pin_a3), JCBUS_2.a4 (Pin_a4), JCBUS_2.a49 (Pin_a49), JCBUS_2.a50 (Pin_a50), JCBUS_3.a1 (Pin_a1), JCBUS_3.a2 (Pin_a2), JCBUS_3.a3 (Pin_a3), JCBUS_3.a4 (Pin_a4), JCBUS_3.a49 (Pin_a49), JCBUS_3.a50 (Pin_a50), JCBUS_4.a1 (Pin_a1), JCBUS_4.a2 (Pin_a2), JCBUS_4.a3 (Pin_a3), JCBUS_4.a4 (Pin_a4), JCBUS_4.a49 (Pin_a49), JCBUS_4.a50 (Pin_a50), JCBUS_5.a1 (Pin_a1), JCBUS_5.a2 (Pin_a2), JCBUS_5.a3 (Pin_a3), JCBUS_5.a4 (Pin_a4), JCBUS_5.a49 (Pin_a49), JCBUS_5.a50 (Pin_a50), C22.1, C23.1, U21.14 (VCC), U22.16 (VCC)
- net HALT: now also JCBUS_0.b17 (Pin_b17), JCBUS_1.b17 (Pin_b17), JCBUS_2.b17 (Pin_b17), JCBUS_3.b17 (Pin_b17), JCBUS_4.b17 (Pin_b17), JCBUS_5.b17 (Pin_b17)
- net INT: now also JCBUS_0.b14 (Pin_b14), JCBUS_1.b14 (Pin_b14), JCBUS_2.b14 (Pin_b14), JCBUS_3.b14 (Pin_b14), JCBUS_4.b14 (Pin_b14), JCBUS_5.b14 (Pin_b14)
- net IORQ: now also JCBUS_0.b10 (Pin_b10), JCBUS_1.b10 (Pin_b10), JCBUS_2.b10 (Pin_b10), JCBUS_3.b10 (Pin_b10), JCBUS_4.b10 (Pin_b10), JCBUS_5.b10 (Pin_b10), U22.1 (E)
- net IRQ0: now also JCBUS_0.b21 (Pin_b21), JCBUS_1.b21 (Pin_b21), JCBUS_2.b21 (Pin_b21), JCBUS_3.b21 (Pin_b21), JCBUS_4.b21 (Pin_b21), JCBUS_5.b21 (Pin_b21)
- net IRQ1: now also JCBUS_0.b22 (Pin_b22), JCBUS_1.b22 (Pin_b22), JCBUS_2.b22 (Pin_b22), JCBUS_3.b22 (Pin_b22), JCBUS_4.b22 (Pin_b22), JCBUS_5.b22 (Pin_b22)
- net IRQ2: now also JCBUS_0.b23 (Pin_b23), JCBUS_1.b23 (Pin_b23), JCBUS_2.b23 (Pin_b23), JCBUS_3.b23 (Pin_b23), JCBUS_4.b23 (Pin_b23), JCBUS_5.b23 (Pin_b23)
- net IRQ3: now also JCBUS_0.b24 (Pin_b24), JCBUS_1.b24 (Pin_b24), JCBUS_2.b24 (Pin_b24), JCBUS_3.b24 (Pin_b24), JCBUS_4.b24 (Pin_b24), JCBUS_5.b24 (Pin_b24)
- net IRQ4: now also JCBUS_0.b41 (Pin_b41), JCBUS_1.b41 (Pin_b41), JCBUS_2.b41 (Pin_b41), JCBUS_3.b41 (Pin_b41), JCBUS_4.b41 (Pin_b41), JCBUS_5.b41 (Pin_b41)
- net IRQ5: now also JCBUS_0.b42 (Pin_b42), JCBUS_1.b42 (Pin_b42), JCBUS_2.b42 (Pin_b42), JCBUS_3.b42 (Pin_b42), JCBUS_4.b42 (Pin_b42), JCBUS_5.b42 (Pin_b42)
- net IRQ6: now also JCBUS_0.b43 (Pin_b43), JCBUS_1.b43 (Pin_b43), JCBUS_2.b43 (Pin_b43), JCBUS_3.b43 (Pin_b43), JCBUS_4.b43 (Pin_b43), JCBUS_5.b43 (Pin_b43)
- net IRQ7: now also JCBUS_0.b44 (Pin_b44), JCBUS_1.b44 (Pin_b44), JCBUS_2.b44 (Pin_b44), JCBUS_3.b44 (Pin_b44), JCBUS_4.b44 (Pin_b44), JCBUS_5.b44 (Pin_b44)
- net M1: now also JCBUS_0.b13 (Pin_b13), JCBUS_1.b13 (Pin_b13), JCBUS_2.b13 (Pin_b13), JCBUS_3.b13 (Pin_b13), JCBUS_4.b13 (Pin_b13), JCBUS_5.b13 (Pin_b13)
- net MREQ: now also JCBUS_0.b9 (Pin_b9), JCBUS_1.b9 (Pin_b9), JCBUS_2.b9 (Pin_b9), JCBUS_3.b9 (Pin_b9), JCBUS_4.b9 (Pin_b9), JCBUS_5.b9 (Pin_b9)
- net NMI: now also JCBUS_0.b15 (Pin_b15), JCBUS_1.b15 (Pin_b15), JCBUS_2.b15 (Pin_b15), JCBUS_3.b15 (Pin_b15), JCBUS_4.b15 (Pin_b15), JCBUS_5.b15 (Pin_b15)
- net RD: now also JCBUS_0.b12 (Pin_b12), JCBUS_1.b12 (Pin_b12), JCBUS_2.b12 (Pin_b12), JCBUS_3.b12 (Pin_b12), JCBUS_4.b12 (Pin_b12), JCBUS_5.b12 (Pin_b12), U22.3 (A1)
- net RESET: now also JCBUS_0.b8 (Pin_b8), JCBUS_1.b8 (Pin_b8), JCBUS_2.b8 (Pin_b8), JCBUS_3.b8 (Pin_b8), JCBUS_4.b8 (Pin_b8), JCBUS_5.b8 (Pin_b8)
- net RFSH: now also JCBUS_0.b20 (Pin_b20), JCBUS_1.b20 (Pin_b20), JCBUS_2.b20 (Pin_b20), JCBUS_3.b20 (Pin_b20), JCBUS_4.b20 (Pin_b20), JCBUS_5.b20 (Pin_b20)
- net RX: now also JCBUS_0.a8 (Pin_a8), JCBUS_1.a8 (Pin_a8), JCBUS_2.a8 (Pin_a8), JCBUS_3.a8 (Pin_a8), JCBUS_4.a8 (Pin_a8), JCBUS_5.a8 (Pin_a8)
- net RX2: now also JCBUS_0.a6 (Pin_a6), JCBUS_1.a6 (Pin_a6), JCBUS_2.a6 (Pin_a6), JCBUS_3.a6 (Pin_a6), JCBUS_4.a6 (Pin_a6), JCBUS_5.a6 (Pin_a6)
- net TX: now also JCBUS_0.a7 (Pin_a7), JCBUS_1.a7 (Pin_a7), JCBUS_2.a7 (Pin_a7), JCBUS_3.a7 (Pin_a7), JCBUS_4.a7 (Pin_a7), JCBUS_5.a7 (Pin_a7)
- net TX2: now also JCBUS_0.a5 (Pin_a5), JCBUS_1.a5 (Pin_a5), JCBUS_2.a5 (Pin_a5), JCBUS_3.a5 (Pin_a5), JCBUS_4.a5 (Pin_a5), JCBUS_5.a5 (Pin_a5)
- net WAIT: now also JCBUS_0.b16 (Pin_b16), JCBUS_1.b16 (Pin_b16), JCBUS_2.b16 (Pin_b16), JCBUS_3.b16 (Pin_b16), JCBUS_4.b16 (Pin_b16), JCBUS_5.b16 (Pin_b16)
- net WR: now also JCBUS_0.b11 (Pin_b11), JCBUS_1.b11 (Pin_b11), JCBUS_2.b11 (Pin_b11), JCBUS_3.b11 (Pin_b11), JCBUS_4.b11 (Pin_b11), JCBUS_5.b11 (Pin_b11), U22.2 (A0)
- net at R36.2, R37.2, SW2.1: now also JP27.1 (A)
- net DREQ0: now reaches JCBUS_4.a41 (Pin_a41)
- net DREQ0: now also JCBUS_0.a41 (Pin_a41), JCBUS_1.a41 (Pin_a41), JCBUS_2.a41 (Pin_a41), JCBUS_3.a41 (Pin_a41), JCBUS_5.a41 (Pin_a41)
- net DACK0: now reaches JCBUS_4.a42 (Pin_a42)
- net DACK0: now also JCBUS_0.a42 (Pin_a42), JCBUS_1.a42 (Pin_a42), JCBUS_2.a42 (Pin_a42), JCBUS_3.a42 (Pin_a42), JCBUS_5.a42 (Pin_a42)
- net DREQ1: now reaches JCBUS_4.a43 (Pin_a43)
- net DREQ1: now also JCBUS_0.a43 (Pin_a43), JCBUS_1.a43 (Pin_a43), JCBUS_2.a43 (Pin_a43), JCBUS_3.a43 (Pin_a43), JCBUS_5.a43 (Pin_a43)
- net DACK1: now reaches JCBUS_4.a44 (Pin_a44)
- net DACK1: now also JCBUS_0.a44 (Pin_a44), JCBUS_1.a44 (Pin_a44), JCBUS_2.a44 (Pin_a44), JCBUS_3.a44 (Pin_a44), JCBUS_5.a44 (Pin_a44)
- net DREQ2: now reaches JCBUS_4.a45 (Pin_a45)
- net DREQ2: now also JCBUS_0.a45 (Pin_a45), JCBUS_1.a45 (Pin_a45), JCBUS_2.a45 (Pin_a45), JCBUS_3.a45 (Pin_a45), JCBUS_5.a45 (Pin_a45)
- net DACK2: now reaches JCBUS_4.a46 (Pin_a46)
- net DACK2: now also JCBUS_0.a46 (Pin_a46), JCBUS_1.a46 (Pin_a46), JCBUS_2.a46 (Pin_a46), JCBUS_3.a46 (Pin_a46), JCBUS_5.a46 (Pin_a46)
- net DREQ3: now reaches JCBUS_4.a47 (Pin_a47)
- net DREQ3: now also JCBUS_0.a47 (Pin_a47), JCBUS_1.a47 (Pin_a47), JCBUS_2.a47 (Pin_a47), JCBUS_3.a47 (Pin_a47), JCBUS_5.a47 (Pin_a47)
- net DACK3: now reaches JCBUS_4.a48 (Pin_a48)
- net DACK3: now also JCBUS_0.a48 (Pin_a48), JCBUS_1.a48 (Pin_a48), JCBUS_2.a48 (Pin_a48), JCBUS_3.a48 (Pin_a48), JCBUS_5.a48 (Pin_a48)
- net BUSREQ: now reaches JCBUS_4.b18 (Pin_b18)
- net BUSREQ: now also JCBUS_0.b18 (Pin_b18), JCBUS_1.b18 (Pin_b18), JCBUS_2.b18 (Pin_b18), JCBUS_3.b18 (Pin_b18), JCBUS_5.b18 (Pin_b18)
- net BUSACK: now reaches JCBUS_4.b19 (Pin_b19)
- net BUSACK: now also JCBUS_0.b19 (Pin_b19), JCBUS_1.b19 (Pin_b19), JCBUS_2.b19 (Pin_b19), JCBUS_3.b19 (Pin_b19), JCBUS_5.b19 (Pin_b19)
- net DREQ4: now reaches JCBUS_4.b45 (Pin_b45)
- net DREQ4: now also JCBUS_0.b45 (Pin_b45), JCBUS_1.b45 (Pin_b45), JCBUS_2.b45 (Pin_b45), JCBUS_3.b45 (Pin_b45), JCBUS_5.b45 (Pin_b45)
- net DACK4: now reaches JCBUS_4.b46 (Pin_b46)
- net DACK4: now also JCBUS_0.b46 (Pin_b46), JCBUS_1.b46 (Pin_b46), JCBUS_2.b46 (Pin_b46), JCBUS_3.b46 (Pin_b46), JCBUS_5.b46 (Pin_b46)
- net DREQ5: now reaches JCBUS_4.b47 (Pin_b47)
- net DREQ5: now also JCBUS_0.b47 (Pin_b47), JCBUS_1.b47 (Pin_b47), JCBUS_2.b47 (Pin_b47), JCBUS_3.b47 (Pin_b47), JCBUS_5.b47 (Pin_b47)
- net DACK5: now reaches JCBUS_4.b48 (Pin_b48)
- net DACK5: now also JCBUS_0.b48 (Pin_b48), JCBUS_1.b48 (Pin_b48), JCBUS_2.b48 (Pin_b48), JCBUS_3.b48 (Pin_b48), JCBUS_5.b48 (Pin_b48)
- net RESET2: now reaches JCBUS_4.b6 (Pin_b6)
- net RESET2: now also JCBUS_0.b6 (Pin_b6), JCBUS_1.b6 (Pin_b6), JCBUS_2.b6 (Pin_b6), JCBUS_3.b6 (Pin_b6), JCBUS_5.b6 (Pin_b6)
- net at C16.2, R35.1, SW2.2: now also JP27.2 (B)
- net WR_FPU: now reaches FPU_0.19 (~{WR})
- net WR_FPU: now also U22.6 (O2)
- net RD_FPU: now reaches FPU_0.20 (~{RD})
- net RD_FPU: now also U22.5 (O1)
- net CLK_FDC16: no longer names the net of FDC_0.23 (CLK1), JP20.2 (B), JP7.2 (B)
- net CLK_FDC96: no longer names the net of FDC_0.21 (CLK2), U19.12
- net CLK_FPU: no longer names the net of FPU_0.23 (CLK)
- net CLK_FPU: now also JP28.1 (A), JP29.1 (A), JP30.1 (A)
- new net: JP29.2 (B), U21.11 (C), U21.5 (Q)
- new net: JP25.1 (A), JP26.1 (A), JP28.2 (B), U21.3 (C)
- new net: U21.12 (D), U21.8 (~{Q})
- new net: JP30.2 (B), U21.9 (Q)
- new net: U21.2 (D), U21.6 (~{Q})
- no-connect marks 52 -> 58
Other:
- note added: "÷1"
- note added: "÷2"
- note added: "÷3"
- note removed: "Connect SVREQ/ACK to spare IO pins?"
- note removed: "check caps if need to be polarized eg 1nf"
- moved on the sheet: JCBUS_1, JCBUS_2, JCBUS_3, JCBUS_4, JCBUS_5, SW2, U14B

Commit message: agn
Parts:
- R3, R4, R5, R6: footprint (none) -> Resistor_THT:R_Axial_DIN0207_L6.3mm_D2.5mm_P10.16mm_Horizontal
Changed lines of the file:
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@@
 			)
 		)
-		(property "Footprint" ""
+		(property "Footprint" "Resistor_THT:R_Axial_DIN0207_L6.3mm_D2.5mm_P10.16mm_Horizontal"
 			(at 159.258 240.03 90)
 			(effects
@@
 			)
 		)
-		(property "Footprint" ""
+		(property "Footprint" "Resistor_THT:R_Axial_DIN0207_L6.3mm_D2.5mm_P10.16mm_Horizontal"
 			(at 174.498 240.03 90)
 			(effects
@@
 			)
 		)
-		(property "Footprint" ""
+		(property "Footprint" "Resistor_THT:R_Axial_DIN0207_L6.3mm_D2.5mm_P10.16mm_Horizontal"
 			(at 182.118 240.03 90)
 			(effects
@@
 			)
 		)
-		(property "Footprint" ""
+		(property "Footprint" "Resistor_THT:R_Axial_DIN0207_L6.3mm_D2.5mm_P10.16mm_Horizontal"
 			(at 166.878 240.03 90)
 			(effects

Commit message: rev0
Other:
- note removed: "check which ic need to be socket or directrly soldered"
- moved on the sheet: JCBUS_0, JCBUS_1, JCBUS_2, JCBUS_3, JCBUS_4, JCBUS_5, U16C, U16D, U1F, U22B

Commit message: ceptmmu
Parts:
- added BT1: BATT_RTC, symbol Device:Battery_Cell
- added C29, C30: 100nF, symbol Device:C
- added J1: PORT_RTC_IO, Connector_PinHeader_2.54mm:PinHeader_2x06_P2.54mm_Vertical, symbol Connector_Generic:Conn_02x06_Counter_Clockwise
- added JP31: DMA_RDYA, Connector_PinHeader_2.54mm:PinHeader_1x02_P2.54mm_Vertical, symbol Jumper:Jumper_2_Open
- added JP32: DMA_RDYB, Connector_PinHeader_2.54mm:PinHeader_1x02_P2.54mm_Vertical, symbol Jumper:Jumper_2_Open
- added JP33: SEL_LIO, symbol Jumper:SolderJumper_2_Open
- added JP34: SEL_DMA, symbol Jumper:SolderJumper_2_Open
- added R50: 100K, Resistor_THT:R_Axial_DIN0207_L6.3mm_D2.5mm_P10.16mm_Horizontal, symbol Device:R
- added RAM_1: IDT6116, Package_DIP:DIP-24_W15.24mm_Socket, symbol Carboni_Library:IDT6116
- added U23: 74LS32, Package_DIP:DIP-14_W7.62mm, symbol 74xx:74LS32
- added U24: 74HCT273, symbol 74xx:74HCT273
- added U25: DS1302+, Package_DIP:DIP-8_W7.62mm_Socket, symbol Timer_RTC:DS1302+
- added U26: 74AHCT125, Package_DIP:DIP-14_W7.62mm, symbol 74xx:74AHCT125
- added XTAL_RES_3: XTAL RTC 32KHz, Crystal:Crystal_Round_D3.0mm_Vertical, symbol Device:Crystal
- XTAL_RES_1: value XTAL RES FDC 16MHz -> XTAL FDC 16MHz
- XTAL_RES_2: value XTAL RES FDC 9.6MHz -> XTAL FDC 9.6MHz
- renumbered RAM_1 to RAM_2
Connections:
- net +5V: now also C29.2, C30.2, R50.2, RAM_1.24 (VCC), U23.7 (GND), U24.20 (VCC), U25.1 (VCC2), U26.7 (GND)
- net BUSREQ: now also DMA_0.15 (~{BUSREQ})
- net GND: now also BT1.2 (-), C29.1, C30.1, J1.10 (Pin_10), J1.11 (Pin_11), J1.12 (Pin_12), J1.7 (Pin_7), J1.8 (Pin_8), J1.9 (Pin_9), RAM_1.12 (GND), U23.14 (VCC), U24.10 (GND), U25.4 (GND), U26.14 (VCC)
- net INT: now also DMA_0.37 (~{INT/PULSE})
- net RD: now also RAM_1.20 (~{OE}), U23.2
- net RESET: now also U24.1 (~{Mr})
- net WR: now also RAM_1.21 (~{WE}), U23.4
- net RDYA: now reaches SIO_0.10 (~{W}/~{RDYA})
- net RDYA: now also JP31.1 (A)
- net RDYB: now reaches SIO_0.30 (~{W}/~{RDYB})
- net RDYB: now also JP32.1 (A)
- net at SIO_0.35 (~{CE}): now also U8.11 (~{Y4}); no longer U8.15 (~{Y0})
- net at U3.10: now also JP33.1 (A); no longer U8.11 (~{Y4})
- net at R20.1, RAM_2.18 (~{CS}): now also U23.8; no longer JP5.3 (B)
- net SEL_DMA: now reaches DMA_0.16 (~{C5/}WAIT)
- net SEL_DMA: now also JP34.1 (A)
- net RDY: now reaches DMA_0.25 (RDY)
- net RDY: now also JP31.2 (B), JP32.2 (B)
- net at U1.12: now also U23.10
- net at U1.13: now also U23.12
- new net: U25.2 (X1), XTAL_RES_3.2
- new net: U25.3 (X2), XTAL_RES_3.1
- new net: U24.6 (Q2), U25.5 (CE)
- new net: U25.6 (I/O), U26.11, U26.9
- new net: U24.9 (Q3), U25.7 (SCLK)
- new net: BT1.1 (+), U25.8 (VCC1)
- new net: U23.3, U24.11 (Cp), U26.10
- new net: JP33.2 (B), JP34.2 (B), U8.15 (~{Y0})
- new net: R50.1, RAM_1.18 (~{CS}), U23.11
- new net: U23.6, U26.1, U26.4
- new net: J1.5 (Pin_5), U26.2
- new net: JP5.3 (B), U23.13, U23.9
- new net: J1.6 (Pin_6), U26.5
- new net: J1.1 (Pin_1), U24.2 (Q0)
- new net: J1.2 (Pin_2), U24.19 (Q7)
- new net: J1.3 (Pin_3), U24.5 (Q1)
- new net: J1.4 (Pin_4), U24.16 (Q6)
- new net: U24.12 (Q4), U26.12
- new net: U24.15 (Q5), U26.13
- new net RCT_DATA: U26.8
- new net SEL_RTC: U23.1, U23.5
Other:
- note added: "/IORD"
- note added: "/IOWR"
- note added: "A11"
- note added: "ATX Power Control"
- note added: "D4"
- note added: "I/O write to: 0x7X = 0111 100X"
- note added: "If SIO baud rate using CLK2: Must be < half rate of CLK due to sync of CTC."
- note added: "Real Time Clock"
- note added: "U0 requires +5VSB for ATX PS_ON."
- note added: "W27C512 does not support erasure."
- note added: "Y0: /DMA = /IORQ 0x80 Y2: /CTC = /IORQ 0x88 Y4: /SIO = /IORQ 0x90 Y6: /PIO = /IORQ 0x98"
- note added: "÷4"
- note removed: "ATX Power Switch"
- note removed: "I/O write to 0x78 or 0x79 = 0111 100X"
- note removed: "If SIO baud rate using CLK2: Must be less than half rate of CLK due to internal sync of CTC."
- note removed: "PCB ideally has 2x IDT6116 for 4KB, selected by line A11 && SEL_RAM. W27C512 does not support erasure."
- note removed: "U0 requires +5VSB for ATX POWER switch."
- note removed: "Y0: /SIO = /IORQ 0x80 Y2: /CTC = /IORQ 0x88 Y4: /LIO = /IORQ 0x90 Y6: /PIO = /IORQ 0x98"
- note removed: "÷3"
- moved on the sheet: C15, C16, C17, C18, C19, C20, C21, C22, C23, C26, C3, C4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

Commit message: yurr
check mmu address decode map
Connections:
- net SEL_TAPE is gone; now on net SEL_RTC: U15.13 (~{Y2})
- net IRQ_FDC: now also FDC_0.16 (IRQ)
- net IRQ_TAPE: no longer names the net of PIO_0.14 (PA1)
- no-connect marks 58 -> 59
Other:
- note added: "Y0: /FPU = 0x80 Y2: /RTC = 0x88 Y4: /FDC = 0x90 Y6: /IDE = 0x98"
- note removed: "Y0: /FPU = 0x80 Y2: /TAP = 0x88 Y4: /FDC = 0x90 Y6: /IDE = 0x98"
- moved on the sheet: C15, C16, C17, C18, C19, C20, C21, C22, C23, C26, C29, C30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

Commit message: rev1
Parts:
- BT1: footprint (none) -> Battery:BatteryHolder_MYOUNG_BS-07-A1BJ001_CR2032
- renumbered IDE_0 to IDE_1
Connections:
- net CLK: now also JP1.1 (A); no longer JP1.2 (B)
- net GND: now also C1.1; no longer C1.2
- net at XTAL_OSC_0.3: now also JP1.2 (B); no longer JP1.1 (A)
- net at R1.1, U1.1, XTAL_RES_0.1: now also C1.2; no longer C1.1
- removed net DACK4: JCBUS_0.b46 (Pin_b46), JCBUS_1.b46 (Pin_b46), JCBUS_2.b46 (Pin_b46), JCBUS_3.b46 (Pin_b46), JCBUS_4.b46 (Pin_b46), JCBUS_5.b46 (Pin_b46)
- removed net DACK5: JCBUS_0.b48 (Pin_b48), JCBUS_1.b48 (Pin_b48), JCBUS_2.b48 (Pin_b48), JCBUS_3.b48 (Pin_b48), JCBUS_4.b48 (Pin_b48), JCBUS_5.b48 (Pin_b48)
- removed net DREQ4: JCBUS_0.b45 (Pin_b45), JCBUS_1.b45 (Pin_b45), JCBUS_2.b45 (Pin_b45), JCBUS_3.b45 (Pin_b45), JCBUS_4.b45 (Pin_b45), JCBUS_5.b45 (Pin_b45)
- removed net DREQ5: JCBUS_0.b47 (Pin_b47), JCBUS_1.b47 (Pin_b47), JCBUS_2.b47 (Pin_b47), JCBUS_3.b47 (Pin_b47), JCBUS_4.b47 (Pin_b47), JCBUS_5.b47 (Pin_b47)
- net IDER: no longer names the net of IDE_1.23 (Pin_23), U14.8
- net IDEW: no longer names the net of IDE_1.25 (Pin_25), U14.6
- no-connect marks 59 -> 83
Other:
- note added: "Chipset Device Decode 1"
- note removed: "Chipset Device SEL Decode"
- moved on the sheet: ATX_PWR_0, BT1, C1, C10, C11, C12, C13, C14, C15, C16, C17, C18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
