File: schematics/dATX_JC100.kicad_pcb (KiCad board)
At the start: 2 copper layers, 300 x 200 mm, 31 parts

Commit message: lots
Parts:
- added C1: 120pF, Capacitor_THT:C_Disc_D3.0mm_W1.6mm_P2.50mm, F.Cu at (57.4, 214.6)
- added C10: 1uF, Capacitor_THT:CP_Radial_D4.0mm_P1.50mm, F.Cu at (232.8, 233.9)
- added C11: 1uF, Capacitor_THT:CP_Radial_D4.0mm_P1.50mm, F.Cu at (238.4, 228.4)
- added C12: 1uF, Capacitor_THT:CP_Radial_D4.0mm_P1.50mm, F.Cu at (238.4, 233.9)
- added C13: 1uF, Capacitor_THT:CP_Radial_D4.0mm_P1.50mm, F.Cu at (244.0, 228.4)
- added C14: 1uF, Capacitor_THT:CP_Radial_D4.0mm_P1.50mm, F.Cu at (244.0, 233.9)
- added C2: 100nF, Capacitor_THT:C_Disc_D3.0mm_W1.6mm_P2.50mm, F.Cu at (64.4, 214.6)
- added C3: 1nF, Capacitor_THT:C_Disc_D3.0mm_W1.6mm_P2.50mm, F.Cu at (391.0, 186.3)
- added C7: 1uF, Capacitor_THT:CP_Radial_D4.0mm_P1.50mm, F.Cu at (227.2, 228.4)
- added C8: 1uF, Capacitor_THT:CP_Radial_D4.0mm_P1.50mm, F.Cu at (227.2, 233.9)
- added C9: 1uF, Capacitor_THT:CP_Radial_D4.0mm_P1.50mm, F.Cu at (232.8, 228.4)
- added D1: RESET, LED_THT:LED_D5.0mm, F.Cu at (367.3, 165.2)
- added D10: L7, LED_THT:LED_D5.0mm, F.Cu at (368.7, 211.8)
- added D11: L6, LED_THT:LED_D5.0mm, F.Cu at (376.1, 204.3)
- added D12: L5, LED_THT:LED_D5.0mm, F.Cu at (376.1, 211.8)
- added D13: L4, LED_THT:LED_D5.0mm, F.Cu at (383.6, 204.3)
- added D14: L3, LED_THT:LED_D5.0mm, F.Cu at (383.6, 211.8)
- added D15: L2, LED_THT:LED_D5.0mm, F.Cu at (391.1, 204.3)
- added D16: L1, LED_THT:LED_D5.0mm, F.Cu at (391.1, 211.8)
- added D2: CLK, LED_THT:LED_D5.0mm, F.Cu at (367.3, 172.7)
- added D3: CLK2, LED_THT:LED_D5.0mm, F.Cu at (374.8, 165.2)
- added D4: +5V, LED_THT:LED_D5.0mm, F.Cu at (374.8, 172.7)
- added D5: +12V, LED_THT:LED_D5.0mm, F.Cu at (382.3, 165.2)
- added D6: -12V, LED_THT:LED_D5.0mm, F.Cu at (382.3, 172.7)
- added D7: 3.3V, LED_THT:LED_D5.0mm, F.Cu at (389.8, 165.2)
- added D8: -5V, LED_THT:LED_D5.0mm, F.Cu at (389.8, 172.7)
- added D9: L8, LED_THT:LED_D5.0mm, F.Cu at (368.7, 204.3)
- added JP10: CLK_SIOA, Connector_PinHeader_2.54mm:PinHeader_1x02_P2.54mm_Vertical, F.Cu at (372.7, 150.4)
- added JP12: CTC_SIOA, Connector_PinHeader_2.54mm:PinHeader_1x02_P2.54mm_Vertical, F.Cu at (377.3, 150.4)
- added JP13: CLK_SIOB, Connector_PinHeader_2.54mm:PinHeader_1x02_P2.54mm_Vertical, F.Cu at (381.9, 150.4)
- added JP14: CLK2_SIOB, Connector_PinHeader_2.54mm:PinHeader_1x02_P2.54mm_Vertical, F.Cu at (386.5, 150.4)
- added JP4: RESET, Connector_PinHeader_2.54mm:PinHeader_1x02_P2.54mm_Vertical, F.Cu at (387.1, 187.0)
- added JP5: RAM_SELECT, Connector_PinHeader_2.54mm:PinHeader_1x03_P2.54mm_Vertical, F.Cu at (373.3, 181.3)
- added JP6: ROM_SELECT, Connector_PinHeader_2.54mm:PinHeader_1x03_P2.54mm_Vertical, F.Cu at (377.9, 181.3)
- added JP7: ROM_WRITE, Connector_PinHeader_2.54mm:PinHeader_1x03_P2.54mm_Vertical, F.Cu at (382.5, 181.3)
- added JP8: CLK_CTC, Connector_PinHeader_2.54mm:PinHeader_1x02_P2.54mm_Vertical, F.Cu at (368.1, 150.4)
- added R10: R, Resistor_THT:R_Axial_DIN0207_L6.3mm_D2.5mm_P10.16mm_Horizontal, F.Cu at (346.1, 170.7)
- added R11: R, Resistor_THT:R_Axial_DIN0207_L6.3mm_D2.5mm_P10.16mm_Horizontal, F.Cu at (346.1, 174.8)
- added R12: R, Resistor_THT:R_Axial_DIN0207_L6.3mm_D2.5mm_P10.16mm_Horizontal, F.Cu at (346.1, 178.8)
- added R13: R, Resistor_THT:R_Axial_DIN0207_L6.3mm_D2.5mm_P10.16mm_Horizontal, F.Cu at (346.1, 182.9)
- added R14: R, Resistor_THT:R_Axial_DIN0207_L6.3mm_D2.5mm_P10.16mm_Horizontal, F.Cu at (346.1, 186.9)
- added R15: 4K7, Resistor_THT:R_Axial_DIN0207_L6.3mm_D2.5mm_P10.16mm_Horizontal, F.Cu at (346.1, 191.0)
- added R16: 10K, Resistor_THT:R_Axial_DIN0207_L6.3mm_D2.5mm_P10.16mm_Horizontal, F.Cu at (346.1, 195.0)
- added R17: 100K, Resistor_THT:R_Axial_DIN0207_L6.3mm_D2.5mm_P10.16mm_Horizontal, F.Cu at (346.1, 199.1)
- added R18: 4K7, Resistor_THT:R_Axial_DIN0207_L6.3mm_D2.5mm_P10.16mm_Horizontal, F.Cu at (346.1, 203.1)
- added R19: 100K, Resistor_THT:R_Axial_DIN0207_L6.3mm_D2.5mm_P10.16mm_Horizontal, F.Cu at (346.1, 207.2)
- added R20: 100K, Resistor_THT:R_Axial_DIN0207_L6.3mm_D2.5mm_P10.16mm_Horizontal, F.Cu at (346.1, 211.2)
- added R21: 100K, Resistor_THT:R_Axial_DIN0207_L6.3mm_D2.5mm_P10.16mm_Horizontal, F.Cu at (346.1, 215.3)
- added R22: 100K, Resistor_THT:R_Axial_DIN0207_L6.3mm_D2.5mm_P10.16mm_Horizontal, F.Cu at (346.1, 219.3)
- added R23: 2K2, Resistor_THT:R_Axial_DIN0207_L6.3mm_D2.5mm_P10.16mm_Horizontal, F.Cu at (213.4, 205.6)
- added R24: 2K2, Resistor_THT:R_Axial_DIN0207_L6.3mm_D2.5mm_P10.16mm_Horizontal, F.Cu at (213.4, 209.7)
- added R25: 2K2, Resistor_THT:R_Axial_DIN0207_L6.3mm_D2.5mm_P10.16mm_Horizontal, F.Cu at (213.4, 213.7)
- added R26: 2K2, Resistor_THT:R_Axial_DIN0207_L6.3mm_D2.5mm_P10.16mm_Horizontal, F.Cu at (213.4, 217.8)
- added R27: 100K, Resistor_THT:R_Axial_DIN0207_L6.3mm_D2.5mm_P10.16mm_Horizontal, F.Cu at (213.4, 221.8)
- added R28: 100K, Resistor_THT:R_Axial_DIN0207_L6.3mm_D2.5mm_P10.16mm_Horizontal, F.Cu at (213.4, 225.9)
- added R29: 2K2, Resistor_THT:R_Axial_DIN0207_L6.3mm_D2.5mm_P10.16mm_Horizontal, F.Cu at (213.4, 229.9)
- added R30: 2K2, Resistor_THT:R_Axial_DIN0207_L6.3mm_D2.5mm_P10.16mm_Horizontal, F.Cu at (213.4, 234.0)
- added R31: 2K2, Resistor_THT:R_Axial_DIN0207_L6.3mm_D2.5mm_P10.16mm_Horizontal, F.Cu at (213.4, 238.0)
- added R32: 2K2, Resistor_THT:R_Axial_DIN0207_L6.3mm_D2.5mm_P10.16mm_Horizontal, F.Cu at (213.4, 242.1)
- added R33: 100K, Resistor_THT:R_Axial_DIN0207_L6.3mm_D2.5mm_P10.16mm_Horizontal, F.Cu at (213.4, 246.1)
- added R34: 100K, Resistor_THT:R_Axial_DIN0207_L6.3mm_D2.5mm_P10.16mm_Horizontal, F.Cu at (213.4, 250.2)
- added R7: R, Resistor_THT:R_Axial_DIN0207_L6.3mm_D2.5mm_P10.16mm_Horizontal, F.Cu at (346.1, 158.6)
- added R8: R, Resistor_THT:R_Axial_DIN0207_L6.3mm_D2.5mm_P10.16mm_Horizontal, F.Cu at (346.1, 162.6)
- added R9: R, Resistor_THT:R_Axial_DIN0207_L6.3mm_D2.5mm_P10.16mm_Horizontal, F.Cu at (346.1, 166.7)
- added RAM_0: AS6C4008, Package_DIP:DIP-32_W15.24mm, F.Cu at (374.6, 36.8)
- added RAM_1: IDT6116, Package_DIP:DIP-24_W15.24mm, F.Cu at (374.6, 80.0)
- added RN1: 1K, Resistor_THT:R_Array_SIP9, F.Cu at (368.3, 217.6)
- added ROM_0: W27C512, Package_DIP:DIP-28_W15.24mm, F.Cu at (355.6, 36.8)
- added ROM_1: W27C512, Package_DIP:DIP-28_W15.24mm, F.Cu at (355.6, 74.9)
- added SW1: RESET, Button_Switch_THT:SW_PUSH_6mm, F.Cu at (373.1, 190.7)
- added U10: MAX232, Package_DIP:DIP-16_W7.62mm_Socket, F.Cu at (227.1, 205.7)
- added U11: MAX232, Package_DIP:DIP-16_W7.62mm_Socket, F.Cu at (238.8, 205.7)
- added U2: DS1233, Package_TO_SOT_THT:TO-92L_Inline, F.Cu at (386.9, 182.3)
- added XTAL_OSC_0: Crystal Oscillator, Oscillator:Oscillator_DIP-8, F.Cu at (41.9, 222.2)
- added XTAL_RES_0: Crystal Resonator, Crystal:Resonator-2Pin_W6.0mm_H3.0mm, F.Cu at (58.5, 223.5)
- ATX_PWR_0: value Conn_02x12_Top_Bottom -> Power Supply
- moved CTC_0 119.6 mm to (215.9, 142.4)
- moved DMA_0 96.0 mm to (180.3, 142.4)
- moved SIO_0 77.0 mm to (215.9, 76.3)
- moved PATA_0 66.5 mm to (284.5, 78.9)
- moved FLOPPY_0 65.2 mm to (299.7, 78.9)
- moved CPU_0 32.7 mm to (180.3, 76.3)
- moved FPU_0 26.3 mm to (248.9, 142.4)
- moved PIO_0 20.1 mm to (248.9, 76.3)
- moved ? 19.0 mm to (101.6, 45.7)
- moved ? 19.0 mm to (325.1, 68.6)
- moved ? 19.0 mm to (167.6, 45.7)
- moved ? 19.0 mm to (325.1, 200.7)
- moved ? 19.0 mm to (121.9, 45.7)
- moved ? 19.0 mm to (167.6, 200.7)
- moved ? 19.0 mm to (121.9, 200.7)
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Connections:
- ATX_PWR_0 pad 1: unconnected-(ATX_PWR_0-Pin_1-Pad1) -> +3.3V
- ATX_PWR_0 pad 10: unconnected-(ATX_PWR_0-Pin_10-Pad10) -> +12V
- ATX_PWR_0 pad 11: unconnected-(ATX_PWR_0-Pin_11-Pad11) -> +12V
- ATX_PWR_0 pad 12: unconnected-(ATX_PWR_0-Pin_12-Pad12) -> +3.3V
- ATX_PWR_0 pad 13: unconnected-(ATX_PWR_0-Pin_13-Pad13) -> +3.3V
- ATX_PWR_0 pad 14: unconnected-(ATX_PWR_0-Pin_14-Pad14) -> -12V
- ATX_PWR_0 pad 15: unconnected-(ATX_PWR_0-Pin_15-Pad15) -> GND
- ATX_PWR_0 pad 16: unconnected-(ATX_PWR_0-Pin_16-Pad16) -> PS_ON
- ATX_PWR_0 pad 17: unconnected-(ATX_PWR_0-Pin_17-Pad17) -> GND
- ATX_PWR_0 pad 18: unconnected-(ATX_PWR_0-Pin_18-Pad18) -> GND
- ATX_PWR_0 pad 19: unconnected-(ATX_PWR_0-Pin_19-Pad19) -> GND
- ATX_PWR_0 pad 2: unconnected-(ATX_PWR_0-Pin_2-Pad2) -> +3.3V
- ATX_PWR_0 pad 20: unconnected-(ATX_PWR_0-Pin_20-Pad20) -> -5V
- ATX_PWR_0 pad 21: unconnected-(ATX_PWR_0-Pin_21-Pad21) -> +5V
- ATX_PWR_0 pad 22: unconnected-(ATX_PWR_0-Pin_22-Pad22) -> +5V
- ATX_PWR_0 pad 23: unconnected-(ATX_PWR_0-Pin_23-Pad23) -> +5V
- ATX_PWR_0 pad 24: unconnected-(ATX_PWR_0-Pin_24-Pad24) -> GND
- ATX_PWR_0 pad 3: unconnected-(ATX_PWR_0-Pin_3-Pad3) -> GND
- ATX_PWR_0 pad 4: unconnected-(ATX_PWR_0-Pin_4-Pad4) -> +5V
- ATX_PWR_0 pad 5: unconnected-(ATX_PWR_0-Pin_5-Pad5) -> GND
- ATX_PWR_0 pad 6: unconnected-(ATX_PWR_0-Pin_6-Pad6) -> +5V
- ATX_PWR_0 pad 7: unconnected-(ATX_PWR_0-Pin_7-Pad7) -> GND
- ATX_PWR_0 pad 8: unconnected-(ATX_PWR_0-Pin_8-Pad8) -> PWR_OK
- ATX_PWR_0 pad 9: unconnected-(ATX_PWR_0-Pin_9-Pad9) -> +5VSB
- CPU_0 pad 11: unconnected-(CPU_0-VCC-Pad11) -> +5V
- CPU_0 pad 16: unconnected-(CPU_0-INT-Pad16) -> INT
- CPU_0 pad 17: unconnected-(CPU_0-NMI-Pad17) -> NMI
- CPU_0 pad 18: unconnected-(CPU_0-HALT-Pad18) -> HALT
- CPU_0 pad 19: unconnected-(CPU_0-MREQ-Pad19) -> MREQ
- CPU_0 pad 20: unconnected-(CPU_0-IORQ-Pad20) -> IORQ
- CPU_0 pad 21: unconnected-(CPU_0-RD-Pad21) -> RD
- CPU_0 pad 22: unconnected-(CPU_0-WR-Pad22) -> WR
- CPU_0 pad 23: unconnected-(CPU_0-BUSAK-Pad23) -> BUSAK
- CPU_0 pad 24: unconnected-(CPU_0-WAIT-Pad24) -> WAIT
- CPU_0 pad 25: unconnected-(CPU_0-BUSRQ-Pad25) -> BUSRQ
- CPU_0 pad 26: unconnected-(CPU_0-RESET-Pad26) -> RESET
- CPU_0 pad 27: unconnected-(CPU_0-M1-Pad27) -> M1
- CPU_0 pad 28: unconnected-(CPU_0-RFSH-Pad28) -> RFSH
- CPU_0 pad 29: unconnected-(CPU_0-GND-Pad29) -> GND
- CPU_0 pad 6: unconnected-(CPU_0-CLK-Pad6) -> CLK
- CTC_0 pad 10: unconnected-(CTC_0-~{IORQ}-Pad10) -> IORQ
- CTC_0 pad 11: unconnected-(CTC_0-IEO-Pad11) -> IE_1
- CTC_0 pad 12: unconnected-(CTC_0-~{INT}-Pad12) -> INT
- CTC_0 pad 13: unconnected-(CTC_0-IEI-Pad13) -> IE_0
- CTC_0 pad 14: unconnected-(CTC_0-~{M1}-Pad14) -> M1
- CTC_0 pad 15: unconnected-(CTC_0-CLK-Pad15) -> CLK
- CTC_0 pad 16: unconnected-(CTC_0-~{CE}-Pad16) -> Net-(CTC_0-~{CE})
- CTC_0 pad 17: unconnected-(CTC_0-~{RESET}-Pad17) -> RESET
- CTC_0 pad 18: unconnected-(CTC_0-CS0-Pad18) -> Net-(CTC_0-CS0)
- CTC_0 pad 19: unconnected-(CTC_0-CS1-Pad19) -> Net-(CTC_0-CS1)
- CTC_0 pad 20: unconnected-(CTC_0-CLK/TRG3-Pad20) -> Net-(CTC_0-CLK/TRG0)
- CTC_0 pad 21: unconnected-(CTC_0-CLK/TRG2-Pad21) -> Net-(CTC_0-CLK/TRG0)
- CTC_0 pad 22: unconnected-(CTC_0-CLK/TRG1-Pad22) -> Net-(CTC_0-CLK/TRG0)
- CTC_0 pad 23: unconnected-(CTC_0-CLK/TRG0-Pad23) -> Net-(CTC_0-CLK/TRG0)
- CTC_0 pad 24: unconnected-(CTC_0-+5V-Pad24) -> +5V
- CTC_0 pad 5: unconnected-(CTC_0-GND-Pad5) -> GND
- CTC_0 pad 6: unconnected-(CTC_0-~{RD}-Pad6) -> RD
- CTC_0 pad 7: unconnected-(CTC_0-ZC/TO0-Pad7) -> Net-(CTC_0-ZC/TO0)
- CTC_0 pad 8: unconnected-(CTC_0-ZC/TO1-Pad8) -> Net-(CTC_0-ZC/TO1)
- CTC_0 pad 9: unconnected-(CTC_0-ZC/TO2-Pad9) -> Net-(CTC_0-CLK/TRG0)
- DMA_0 pad 10: unconnected-(DMA_0-~{IORQ}-Pad10) -> MREQ
- DMA_0 pad 11: unconnected-(DMA_0-VCC-Pad11) -> +5V
- DMA_0 pad 12: unconnected-(DMA_0-~{MREQ}-Pad12) -> IORQ
- DMA_0 pad 26: unconnected-(DMA_0-~{M1}-Pad26) -> M1
- DMA_0 pad 30: unconnected-(DMA_0-GND-Pad30) -> GND
- DMA_0 pad 36: unconnected-(DMA_0-IEO-Pad36) -> IE_0
- DMA_0 pad 38: unconnected-(DMA_0-IEI-Pad38) -> +5V
- DMA_0 pad 7: unconnected-(DMA_0-CLK-Pad7) -> CLK
- DMA_0 pad 8: unconnected-(DMA_0-~{WR}-Pad8) -> WR
- DMA_0 pad 9: unconnected-(DMA_0-~{RD}-Pad9) -> RD
- FPU_0 pad 1: unconnected-(FPU_0-VSS-Pad1) -> GND
- PIO_0 pad 11: unconnected-(PIO_0-GND-Pad11) -> GND
- PIO_0 pad 22: unconnected-(PIO_0-IEO-Pad22) -> IE_3
- PIO_0 pad 24: unconnected-(PIO_0-IEI-Pad24) -> IE_2
- PIO_0 pad 26: unconnected-(PIO_0-VCC-Pad26) -> +5V
- SERIAL_0 pad 2: unconnected-(SERIAL_0-Pad2) -> Net-(U10-R1I)
- SERIAL_0 pad 3: unconnected-(SERIAL_0-Pad3) -> Net-(U10-T1O)
- SERIAL_0 pad 5: unconnected-(SERIAL_0-Pad5) -> GND
- SERIAL_0 pad 7: unconnected-(SERIAL_0-Pad7) -> Net-(U10-T2O)
- SERIAL_0 pad 8: unconnected-(SERIAL_0-Pad8) -> Net-(U10-R2I)
- SERIAL_1 pad 2: unconnected-(SERIAL_1-Pad2) -> Net-(U11-R1I)
- SERIAL_1 pad 3: unconnected-(SERIAL_1-Pad3) -> Net-(U11-T1O)
- SERIAL_1 pad 5: unconnected-(SERIAL_1-Pad5) -> GND
- SERIAL_1 pad 7: unconnected-(SERIAL_1-Pad7) -> Net-(U11-T2O)
- SERIAL_1 pad 8: unconnected-(SERIAL_1-Pad8) -> Net-(U11-R2I)
- SIO_0 pad 12: unconnected-(SIO_0-RXDA-Pad12) -> RXA
- SIO_0 pad 13: unconnected-(SIO_0-~{RXCA}-Pad13) -> Net-(JP10-B)
- SIO_0 pad 14: unconnected-(SIO_0-~{TXCA}-Pad14) -> Net-(JP10-B)
- SIO_0 pad 15: unconnected-(SIO_0-TXDA-Pad15) -> TXA
- SIO_0 pad 17: unconnected-(SIO_0-~{RTSA}-Pad17) -> Net-(SIO_0-~{RTSA})
- SIO_0 pad 18: unconnected-(SIO_0-~{CTSA}-Pad18) -> Net-(SIO_0-~{CTSA})
- SIO_0 pad 19: unconnected-(SIO_0-~{DCDA}-Pad19) -> GND
- SIO_0 pad 20: unconnected-(SIO_0-F-Pad20) -> CLK
- SIO_0 pad 21: unconnected-(SIO_0-~{RESET}-Pad21) -> RESET
- SIO_0 pad 22: unconnected-(SIO_0-~{DCDB}-Pad22) -> GND
- SIO_0 pad 23: unconnected-(SIO_0-~{CTSB}-Pad23) -> Net-(SIO_0-~{CTSB})
- SIO_0 pad 24: unconnected-(SIO_0-~{RTSB}-Pad24) -> Net-(SIO_0-~{RTSB})
- SIO_0 pad 26: unconnected-(SIO_0-TXDB-Pad26) -> TXB
- SIO_0 pad 27: unconnected-(SIO_0-~{TXCB}-Pad27) -> Net-(JP13-B)
- SIO_0 pad 28: unconnected-(SIO_0-~{RXCB}-Pad28) -> Net-(JP13-B)
- SIO_0 pad 29: unconnected-(SIO_0-RXDB-Pad29) -> RXB
- SIO_0 pad 31: unconnected-(SIO_0-GND-Pad31) -> GND
- SIO_0 pad 32: unconnected-(SIO_0-~{RD}-Pad32) -> RD
- SIO_0 pad 33: unconnected-(SIO_0-C/~{D}-Pad33) -> Net-(SIO_0-C/~{D})
- SIO_0 pad 34: unconnected-(SIO_0-B/~{A}-Pad34) -> Net-(CTC_0-CS1)
- SIO_0 pad 35: unconnected-(SIO_0-~{CE}-Pad35) -> Net-(SIO_0-~{CE})
- SIO_0 pad 36: unconnected-(SIO_0-~{IORQ}-Pad36) -> IORQ
- SIO_0 pad 5: unconnected-(SIO_0-~{INT}-Pad5) -> INT
- SIO_0 pad 6: unconnected-(SIO_0-IEI-Pad6) -> IE_1
- SIO_0 pad 7: unconnected-(SIO_0-IEO-Pad7) -> IE_2
- SIO_0 pad 8: unconnected-(SIO_0-~{M1}-Pad8) -> M1
- SIO_0 pad 9: unconnected-(SIO_0-+5V-Pad9) -> +5V

Commit message: heaps
Parts:
- removed KEYBD_0, MOUSE_0: Mini-DIN-6, Carboni_Library:Mini_DIN_6
- added C16: 100nF, Capacitor_THT:C_Disc_D3.0mm_W1.6mm_P2.50mm, F.Cu at (302.9, 155.6)
- added C17: 100nF, Capacitor_THT:C_Disc_D3.0mm_W1.6mm_P2.50mm, F.Cu at (302.9, 158.7)
- added JP16: TX1, Connector_PinHeader_2.54mm:PinHeader_1x03_P2.54mm_Vertical, F.Cu at (285.3, 156.3)
- added JP17: RX1, Connector_PinHeader_2.54mm:PinHeader_1x03_P2.54mm_Vertical, F.Cu at (289.9, 156.3)
- added JP18: TX2, Connector_PinHeader_2.54mm:PinHeader_1x03_P2.54mm_Vertical, F.Cu at (294.4, 156.3)
- added JP19: RX2, Connector_PinHeader_2.54mm:PinHeader_1x03_P2.54mm_Vertical, F.Cu at (299.0, 156.3)
- added R35: 100K, Resistor_THT:R_Axial_DIN0207_L6.3mm_D2.5mm_P10.16mm_Horizontal, F.Cu at (284.5, 165.7)
- added R36: 1K, Resistor_THT:R_Axial_DIN0207_L6.3mm_D2.5mm_P10.16mm_Horizontal, F.Cu at (284.5, 169.7)
- added R37: 10K, Resistor_THT:R_Axial_DIN0207_L6.3mm_D2.5mm_P10.16mm_Horizontal, F.Cu at (284.5, 173.8)
- added SW2: RESET, Button_Switch_THT:SW_PUSH_6mm, F.Cu at (298.3, 165.7)
- moved SERIAL_0 77.7 mm to (317.0, 46.0)
- moved SERIAL_1 76.9 mm to (278.9, 46.0)
- moved TAPE_IN_0 75.1 mm to (230.6, 38.1)
- moved TAPE_OUT_0 75.1 mm to (245.6, 38.1)
- moved FLOPPY_0 6.71 mm to (302.3, 85.1)
- moved PATA_0 6.71 mm to (287.0, 85.1)
Connections:
- net Net-(SIO_0-~{CTSA}) renamed CTSA
- net Net-(SIO_0-~{RTSA}) renamed RTSA
- PIO_0 pad 10: unconnected-(PIO_0-PA4-Pad10) -> IRQ_IDE
- PIO_0 pad 12: unconnected-(PIO_0-PA3-Pad12) -> IRQ_FDC
- PIO_0 pad 13: unconnected-(PIO_0-PA2-Pad13) -> IRQ_TAPE
- PIO_0 pad 14: unconnected-(PIO_0-PA1-Pad14) -> IRQ_FPU
- PIO_0 pad 15: unconnected-(PIO_0-PA0-Pad15) -> IRQ_PS2
- PIO_0 pad 23: unconnected-(PIO_0-~{INT}-Pad23) -> INT
- PIO_0 pad 25: unconnected-(PIO_0-CLK-Pad25) -> CLK
- PIO_0 pad 27: unconnected-(PIO_0-PB0-Pad27) -> IRQ0
- PIO_0 pad 28: unconnected-(PIO_0-PB1-Pad28) -> IRQ1
- PIO_0 pad 29: unconnected-(PIO_0-PB2-Pad29) -> IRQ2
- PIO_0 pad 30: unconnected-(PIO_0-PB3-Pad30) -> IRQ3
- PIO_0 pad 31: unconnected-(PIO_0-PB4-Pad31) -> IRQ4
- PIO_0 pad 32: unconnected-(PIO_0-PB5-Pad32) -> IRQ5
- PIO_0 pad 33: unconnected-(PIO_0-PB6-Pad33) -> IRQ6
- PIO_0 pad 34: unconnected-(PIO_0-PB7-Pad34) -> IRQ7
- PIO_0 pad 35: unconnected-(PIO_0-~{RD}-Pad35) -> RD
- PIO_0 pad 36: unconnected-(PIO_0-~{IORQ}-Pad36) -> IORQ
- PIO_0 pad 37: unconnected-(PIO_0-~{M1}-Pad37) -> Net-(PIO_0-~{M1})
- PIO_0 pad 4: unconnected-(PIO_0-~{CE}-Pad4) -> SEL_PIO
Other:
- board text removed: "ATX I/O Shield (safe zone)"

Commit message: yee
Parts:
- added D17: BUSY, LED_THT:LED_D5.0mm, F.Cu at (312.4, 179.1)
- added R38: 4K7, Resistor_THT:R_Axial_DIN0207_L6.3mm_D2.5mm_P10.16mm_Horizontal, F.Cu at (298.2, 177.4)
- added R39: 4K7, Resistor_THT:R_Axial_DIN0207_L6.3mm_D2.5mm_P10.16mm_Horizontal, F.Cu at (298.2, 181.4)
- added R40: 4K7, Resistor_THT:R_Axial_DIN0207_L6.3mm_D2.5mm_P10.16mm_Horizontal, F.Cu at (298.2, 185.5)
- added R41: 4K7, Resistor_THT:R_Axial_DIN0207_L6.3mm_D2.5mm_P10.16mm_Horizontal, F.Cu at (298.2, 189.5)
- added U1: 74LS04, Package_DIP:DIP-14_W7.62mm, F.Cu at (132.8, 215.6)
- added U12: 74LS00, Package_DIP:DIP-14_W7.62mm, F.Cu at (154.3, 215.6)
- added U13: 74HCT74, Package_DIP:DIP-14_W7.62mm, F.Cu at (165.1, 215.6)
- added U14: 74LS32, Package_DIP:DIP-14_W7.62mm, F.Cu at (175.9, 215.6)
- added U14: 74LS32, Package_DIP:DIP-14_W7.62mm, F.Cu at (181.6, 241.3)
- added U15: 74HCT138, Package_DIP:DIP-16_W7.62mm, F.Cu at (154.3, 234.9)
- added U16: 74LS00, Package_DIP:DIP-14_W7.62mm, F.Cu at (186.7, 215.6)
- added U3: 74AHCT125, Package_DIP:DIP-14_W7.62mm, F.Cu at (143.5, 215.6)
- added U4: 74HCT139, Package_DIP:DIP-16_W7.62mm, F.Cu at (132.8, 234.9)
- added U8: 74HCT138, Package_DIP:DIP-16_W7.62mm, F.Cu at (143.5, 234.9)
- added U9: 74HCT273, Package_DIP:DIP-20_W7.62mm, F.Cu at (165.1, 234.9)
- FDD_0: renamed from FLOPPY_0; value Conn_02x17_Odd_Even -> Floppy_IBM
- IDE_0: renamed from PATA_0; value Conn_02x20_Odd_Even -> CompactFlash
- JCBUS_0, JCBUS_1, JCBUS_2, JCBUS_3, JCBUS_4, JCBUS_5: value Conn_02x50_Row_Letter_First -> JC100
- TS_0: renamed from TAPE_OUT_0; value AudioJack2 -> TAPE_IN
- TS_1: renamed from TAPE_IN_0; value AudioJack2 -> TAPE_OUT
Connections:
- FPU_0 pad 2: unconnected-(FPU_0-VCC-Pad2) -> +5V
- IDE_0 pad 1: unconnected-(PATA_0-Pin_1-Pad1) -> RESET
- IDE_0 pad 19: unconnected-(PATA_0-Pin_19-Pad19) -> GND
- IDE_0 pad 2: unconnected-(PATA_0-Pin_2-Pad2) -> GND
- IDE_0 pad 20: unconnected-(PATA_0-Pin_20-Pad20) -> +5V
- IDE_0 pad 22: unconnected-(PATA_0-Pin_22-Pad22) -> GND
- IDE_0 pad 23: unconnected-(PATA_0-Pin_23-Pad23) -> IDER
- IDE_0 pad 24: unconnected-(PATA_0-Pin_24-Pad24) -> GND
- IDE_0 pad 25: unconnected-(PATA_0-Pin_25-Pad25) -> IDEW
- IDE_0 pad 26: unconnected-(PATA_0-Pin_26-Pad26) -> GND
- IDE_0 pad 29: unconnected-(PATA_0-Pin_29-Pad29) -> Net-(IDE_0-Pin_29)
- IDE_0 pad 30: unconnected-(PATA_0-Pin_30-Pad30) -> GND
- IDE_0 pad 34: unconnected-(PATA_0-Pin_34-Pad34) -> Net-(IDE_0-Pin_34)
- IDE_0 pad 37: unconnected-(PATA_0-Pin_37-Pad37) -> Net-(IDE_0-Pin_37)
- IDE_0 pad 38: unconnected-(PATA_0-Pin_38-Pad38) -> Net-(IDE_0-Pin_38)
- IDE_0 pad 39: unconnected-(PATA_0-Pin_39-Pad39) -> Net-(IDE_0-Pin_39)
- IDE_0 pad 40: unconnected-(PATA_0-Pin_40-Pad40) -> GND
- PIO_0 pad 10: IRQ_IDE -> unconnected-(PIO_0-PA4-Pad10)
- PIO_0 pad 12: IRQ_FDC -> IRQ_IDE
- PIO_0 pad 13: IRQ_TAPE -> IRQ_FDC
- PIO_0 pad 14: IRQ_FPU -> IRQ_TAPE
- PIO_0 pad 15: IRQ_PS2 -> IRQ_FPU

Commit message: yurr
Parts:
- added C21: 120pF, Capacitor_THT:C_Disc_D3.0mm_W1.6mm_P2.50mm, F.Cu at (96.5, 234.8)
- added C22: 100nF, Capacitor_THT:C_Disc_D3.0mm_W1.6mm_P2.50mm, F.Cu at (96.5, 237.9)
- added C24: 120pF, Capacitor_THT:C_Disc_D3.0mm_W1.6mm_P2.50mm, F.Cu at (96.5, 241.1)
- added C25: 100nF, Capacitor_THT:C_Disc_D3.0mm_W1.6mm_P2.50mm, F.Cu at (96.5, 244.2)
- added C27: 120pF, Capacitor_THT:C_Disc_D3.0mm_W1.6mm_P2.50mm, F.Cu at (96.5, 247.4)
- added C28: 100nF, Capacitor_THT:C_Disc_D3.0mm_W1.6mm_P2.50mm, F.Cu at (96.5, 250.5)
- added FDC_0: GM82C765B, Package_DIP:DIP-40_W15.24mm_Socket, F.Cu at (77.7, 216.0)
- added JP23: FDC_JP1, Connector_PinHeader_2.54mm:PinHeader_1x03_P2.54mm_Vertical, F.Cu at (51.6, 253.3)
- added JP24: FDC_JP2, Connector_PinHeader_2.54mm:PinHeader_1x03_P2.54mm_Vertical, F.Cu at (56.2, 253.3)
- added R42: 1K, Resistor_THT:R_Axial_DIN0207_L6.3mm_D2.5mm_P10.16mm_Horizontal, F.Cu at (50.8, 264.2)
- added R44: 10K, Resistor_THT:R_Axial_DIN0207_L6.3mm_D2.5mm_P10.16mm_Horizontal, F.Cu at (110.4, 235.2)
- added RN2: 10K, Resistor_THT:R_Array_SIP9, F.Cu at (40.6, 248.9)
- added U0: 74LS00, Package_DIP:DIP-14_W7.62mm, F.Cu at (96.5, 215.9)
- added U1: 74LS04, Package_DIP:DIP-14_W7.62mm, F.Cu at (107.3, 215.9)
- added U19: 74LS04, Package_DIP:DIP-14_W7.62mm, F.Cu at (40.1, 253.1)
- added U19: 74LS04, Package_DIP:DIP-14_W7.62mm, F.Cu at (118.1, 215.9)
- added XTAL_RES_1: XTAL RES FDC 16MHz, Crystal:Resonator-2Pin_W6.0mm_H3.0mm, F.Cu at (102.2, 240.8)
- added XTAL_RES_1: Crystal Resonator, Crystal:Resonator-2Pin_W6.0mm_H3.0mm, F.Cu at (102.2, 235.7)
- added XTAL_RES_2: XTAL RES FDC 9.6MHz, Crystal:Resonator-2Pin_W6.0mm_H3.0mm, F.Cu at (102.2, 245.8)
- D17: value BUSY -> BUSY_IDE
Connections:
- FDD_0 pad 1: unconnected-(FDD_0-Pin_1-Pad1) -> GND
- FDD_0 pad 10: unconnected-(FDD_0-Pin_10-Pad10) -> Net-(FDC_0-~{DS3}~{MO1})
- FDD_0 pad 11: unconnected-(FDD_0-Pin_11-Pad11) -> GND
- FDD_0 pad 12: unconnected-(FDD_0-Pin_12-Pad12) -> Net-(FDC_0-~{DS2})
- FDD_0 pad 13: unconnected-(FDD_0-Pin_13-Pad13) -> GND
- FDD_0 pad 14: unconnected-(FDD_0-Pin_14-Pad14) -> Net-(FDC_0-~{DS1})
- FDD_0 pad 15: unconnected-(FDD_0-Pin_15-Pad15) -> GND
- FDD_0 pad 16: unconnected-(FDD_0-Pin_16-Pad16) -> Net-(FDC_0-~{DS4}~{MO2})
- FDD_0 pad 17: unconnected-(FDD_0-Pin_17-Pad17) -> GND
- FDD_0 pad 18: unconnected-(FDD_0-Pin_18-Pad18) -> Net-(FDC_0-~{DIRC})
- FDD_0 pad 19: unconnected-(FDD_0-Pin_19-Pad19) -> GND
- FDD_0 pad 2: unconnected-(FDD_0-Pin_2-Pad2) -> Net-(FDC_0-~{RPM}~{RWC})
- FDD_0 pad 20: unconnected-(FDD_0-Pin_20-Pad20) -> Net-(FDC_0-~{STEP})
- FDD_0 pad 21: unconnected-(FDD_0-Pin_21-Pad21) -> GND
- FDD_0 pad 22: unconnected-(FDD_0-Pin_22-Pad22) -> Net-(FDC_0-~{WD})
- FDD_0 pad 23: unconnected-(FDD_0-Pin_23-Pad23) -> GND
- FDD_0 pad 24: unconnected-(FDD_0-Pin_24-Pad24) -> Net-(FDC_0-~{WE})
- FDD_0 pad 25: unconnected-(FDD_0-Pin_25-Pad25) -> GND
- FDD_0 pad 26: unconnected-(FDD_0-Pin_26-Pad26) -> Net-(FDC_0-~{TR00})
- FDD_0 pad 27: unconnected-(FDD_0-Pin_27-Pad27) -> GND
- FDD_0 pad 28: unconnected-(FDD_0-Pin_28-Pad28) -> Net-(FDC_0-WP)
- FDD_0 pad 29: unconnected-(FDD_0-Pin_29-Pad29) -> GND
- FDD_0 pad 3: unconnected-(FDD_0-Pin_3-Pad3) -> Net-(FDD_0-Pin_3)
- FDD_0 pad 30: unconnected-(FDD_0-Pin_30-Pad30) -> Net-(FDC_0-~{RDD})
- FDD_0 pad 31: unconnected-(FDD_0-Pin_31-Pad31) -> GND
- FDD_0 pad 32: unconnected-(FDD_0-Pin_32-Pad32) -> Net-(FDC_0-~{HS})
- FDD_0 pad 33: unconnected-(FDD_0-Pin_33-Pad33) -> GND
- FDD_0 pad 34: unconnected-(FDD_0-Pin_34-Pad34) -> Net-(FDC_0-~{IDX})
- FDD_0 pad 4: unconnected-(FDD_0-Pin_4-Pad4) -> GND
- FDD_0 pad 5: unconnected-(FDD_0-Pin_5-Pad5) -> GND
- FDD_0 pad 6: unconnected-(FDD_0-Pin_6-Pad6) -> Net-(FDD_0-Pin_6)
- FDD_0 pad 7: unconnected-(FDD_0-Pin_7-Pad7) -> GND
- FDD_0 pad 8: unconnected-(FDD_0-Pin_8-Pad8) -> Net-(FDC_0-~{IDX})
- FDD_0 pad 9: unconnected-(FDD_0-Pin_9-Pad9) -> GND
- FPU_0 pad 16: unconnected-(FPU_0-VDD-Pad16) -> +12V
- FPU_0 pad 17: unconnected-(FPU_0-~{PAUSE}-Pad17) -> WAIT
- FPU_0 pad 18: unconnected-(FPU_0-~{CS}-Pad18) -> SEL_FPU
- FPU_0 pad 21: unconnected-(FPU_0-C/~{D}-Pad21) -> ADDRESS
- FPU_0 pad 22: unconnected-(FPU_0-RESET-Pad22) -> Net-(FPU_0-RESET)
- FPU_0 pad 23: unconnected-(FPU_0-CLK-Pad23) -> CLK_FPU
- FPU_0 pad 24: unconnected-(FPU_0-~{END}-Pad24) -> IRQ_FPU
- FPU_0 pad 3: unconnected-(FPU_0-~{EACK}-Pad3) -> Net-(FPU_0-~{EACK})
- U16 pad 14: GND -> (no net)
- U16 pad 7: +5VSB -> (no net)

Commit message: pres
Parts:
- removed TS_0: TAPE_IN, Connector_Audio:Jack_3.5mm_CUI_SJ1-3525N_Horizontal
- removed TS_1: TAPE_OUT, Connector_Audio:Jack_3.5mm_CUI_SJ1-3525N_Horizontal
- added JP27: POWER, Connector_PinHeader_2.54mm:PinHeader_1x02_P2.54mm_Vertical, F.Cu at (308.6, 166.4)
- added JP28: FPU_CLKd1, Connector_PinHeader_2.54mm:PinHeader_1x02_P2.54mm_Vertical, F.Cu at (270.6, 290.1)
- added JP29: FPU_CLKd2, Connector_PinHeader_2.54mm:PinHeader_1x02_P2.54mm_Vertical, F.Cu at (275.2, 290.1)
- added JP30: FPU_CLKd4, Connector_PinHeader_2.54mm:PinHeader_1x02_P2.54mm_Vertical, F.Cu at (279.8, 290.1)
- added U18: 74AHCT125, Package_DIP:DIP-14_W7.62mm, F.Cu at (269.9, 270.5)
- added U20: 74HCT138, Package_DIP:DIP-16_W7.62mm, F.Cu at (259.1, 248.6)
- added U21: 74LS74, Package_DIP:DIP-14_W7.62mm, F.Cu at (280.7, 270.5)
- added U22: 74LS139, Package_DIP:DIP-16_W7.62mm, F.Cu at (269.9, 248.6)
- added U5: 74HCT688, Package_DIP:DIP-20_W7.62mm, F.Cu at (248.3, 270.5)
- added U6: 74HCT273, Package_DIP:DIP-20_W7.62mm, F.Cu at (259.1, 270.5)
- added U7: 74HCT157, Package_DIP:DIP-16_W7.62mm, F.Cu at (248.3, 248.6)
- CTC_0, ROM_0, ROM_1: footprint Package_DIP:DIP-28_W15.24mm -> Package_DIP:DIP-28_W15.24mm_Socket
- DMA_0, PIO_0, SIO_0: footprint Package_DIP:DIP-40_W15.24mm -> Package_DIP:DIP-40_W15.24mm_Socket
- FPU_0, RAM_1: footprint Package_DIP:DIP-24_W15.24mm -> Package_DIP:DIP-24_W15.24mm_Socket
- RAM_0: footprint Package_DIP:DIP-32_W15.24mm -> Package_DIP:DIP-32_W15.24mm_Socket
- SW2: value RESET -> POWER
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Connections:
- net CLK_FDC16 renamed Net-(FDC_0-CLK1)
- FDC_0 pad 21: CLK_FDC96 -> Net-(FDC_0-CLK2)
- FPU_0 pad 19: unconnected-(FPU_0-~{WR}-Pad19) -> WR_FPU
- FPU_0 pad 20: unconnected-(FPU_0-~{RD}-Pad20) -> RD_FPU
- FPU_0 pad 23: CLK_FPU -> Net-(FPU_0-CLK)
- JCBUS_0 pad a1: unconnected-(JCBUS_0-Pin_a1-Pada1) -> GND
- JCBUS_0 pad a2: unconnected-(JCBUS_0-Pin_a2-Pada2) -> GND
- JCBUS_0 pad a3: unconnected-(JCBUS_0-Pin_a3-Pada3) -> GND
- JCBUS_0 pad a4: unconnected-(JCBUS_0-Pin_a4-Pada4) -> GND
- JCBUS_0 pad a41: unconnected-(JCBUS_0-Pin_a41-Pada41) -> DREQ0
- JCBUS_0 pad a42: unconnected-(JCBUS_0-Pin_a42-Pada42) -> DACK0
- JCBUS_0 pad a43: unconnected-(JCBUS_0-Pin_a43-Pada43) -> DREQ1
- JCBUS_0 pad a44: unconnected-(JCBUS_0-Pin_a44-Pada44) -> DACK1
- JCBUS_0 pad a45: unconnected-(JCBUS_0-Pin_a45-Pada45) -> DREQ2
- JCBUS_0 pad a46: unconnected-(JCBUS_0-Pin_a46-Pada46) -> DACK2
- JCBUS_0 pad a47: unconnected-(JCBUS_0-Pin_a47-Pada47) -> DREQ3
- JCBUS_0 pad a48: unconnected-(JCBUS_0-Pin_a48-Pada48) -> DACK3
- JCBUS_0 pad a49: unconnected-(JCBUS_0-Pin_a49-Pada49) -> GND
- JCBUS_0 pad a5: unconnected-(JCBUS_0-Pin_a5-Pada5) -> TX2
- JCBUS_0 pad a50: unconnected-(JCBUS_0-Pin_a50-Pada50) -> GND
- JCBUS_0 pad a6: unconnected-(JCBUS_0-Pin_a6-Pada6) -> RX2
- JCBUS_0 pad a7: unconnected-(JCBUS_0-Pin_a7-Pada7) -> TX
- JCBUS_0 pad a8: unconnected-(JCBUS_0-Pin_a8-Pada8) -> RX
- JCBUS_0 pad b1: unconnected-(JCBUS_0-Pin_b1-Padb1) -> +5V
- JCBUS_0 pad b10: unconnected-(JCBUS_0-Pin_b10-Padb10) -> IORQ
- JCBUS_0 pad b11: unconnected-(JCBUS_0-Pin_b11-Padb11) -> WR
- JCBUS_0 pad b12: unconnected-(JCBUS_0-Pin_b12-Padb12) -> RD
- JCBUS_0 pad b13: unconnected-(JCBUS_0-Pin_b13-Padb13) -> M1
- JCBUS_0 pad b14: unconnected-(JCBUS_0-Pin_b14-Padb14) -> INT
- JCBUS_0 pad b15: unconnected-(JCBUS_0-Pin_b15-Padb15) -> NMI
- JCBUS_0 pad b16: unconnected-(JCBUS_0-Pin_b16-Padb16) -> WAIT
- JCBUS_0 pad b17: unconnected-(JCBUS_0-Pin_b17-Padb17) -> HALT
- JCBUS_0 pad b18: unconnected-(JCBUS_0-Pin_b18-Padb18) -> BUSREQ
- JCBUS_0 pad b19: unconnected-(JCBUS_0-Pin_b19-Padb19) -> BUSACK
- JCBUS_0 pad b2: unconnected-(JCBUS_0-Pin_b2-Padb2) -> +12V
- JCBUS_0 pad b20: unconnected-(JCBUS_0-Pin_b20-Padb20) -> RFSH
- JCBUS_0 pad b21: unconnected-(JCBUS_0-Pin_b21-Padb21) -> IRQ0
- JCBUS_0 pad b22: unconnected-(JCBUS_0-Pin_b22-Padb22) -> IRQ1
- JCBUS_0 pad b23: unconnected-(JCBUS_0-Pin_b23-Padb23) -> IRQ2
- JCBUS_0 pad b24: unconnected-(JCBUS_0-Pin_b24-Padb24) -> IRQ3
- JCBUS_0 pad b3: unconnected-(JCBUS_0-Pin_b3-Padb3) -> -12V
- JCBUS_0 pad b4: unconnected-(JCBUS_0-Pin_b4-Padb4) -> +3.3V
- JCBUS_0 pad b41: unconnected-(JCBUS_0-Pin_b41-Padb41) -> IRQ4
- JCBUS_0 pad b42: unconnected-(JCBUS_0-Pin_b42-Padb42) -> IRQ5
- JCBUS_0 pad b43: unconnected-(JCBUS_0-Pin_b43-Padb43) -> IRQ6
- JCBUS_0 pad b44: unconnected-(JCBUS_0-Pin_b44-Padb44) -> IRQ7
- JCBUS_0 pad b45: unconnected-(JCBUS_0-Pin_b45-Padb45) -> DREQ4
- JCBUS_0 pad b46: unconnected-(JCBUS_0-Pin_b46-Padb46) -> DACK4
- JCBUS_0 pad b47: unconnected-(JCBUS_0-Pin_b47-Padb47) -> DREQ5
- JCBUS_0 pad b48: unconnected-(JCBUS_0-Pin_b48-Padb48) -> DACK5
- JCBUS_0 pad b49: unconnected-(JCBUS_0-Pin_b49-Padb49) -> +5V
- JCBUS_0 pad b5: unconnected-(JCBUS_0-Pin_b5-Padb5) -> CLK2
- JCBUS_0 pad b50: unconnected-(JCBUS_0-Pin_b50-Padb50) -> +12V
- JCBUS_0 pad b6: unconnected-(JCBUS_0-Pin_b6-Padb6) -> RESET2
- JCBUS_0 pad b7: unconnected-(JCBUS_0-Pin_b7-Padb7) -> CLK
- JCBUS_0 pad b8: unconnected-(JCBUS_0-Pin_b8-Padb8) -> RESET
- JCBUS_0 pad b9: unconnected-(JCBUS_0-Pin_b9-Padb9) -> MREQ
- JCBUS_1 pad a1: unconnected-(JCBUS_1-Pin_a1-Pada1) -> GND
- JCBUS_1 pad a2: unconnected-(JCBUS_1-Pin_a2-Pada2) -> GND
- JCBUS_1 pad a3: unconnected-(JCBUS_1-Pin_a3-Pada3) -> GND
- JCBUS_1 pad a4: unconnected-(JCBUS_1-Pin_a4-Pada4) -> GND
- JCBUS_1 pad a41: unconnected-(JCBUS_1-Pin_a41-Pada41) -> DREQ0
- JCBUS_1 pad a42: unconnected-(JCBUS_1-Pin_a42-Pada42) -> DACK0
- JCBUS_1 pad a43: unconnected-(JCBUS_1-Pin_a43-Pada43) -> DREQ1
- JCBUS_1 pad a44: unconnected-(JCBUS_1-Pin_a44-Pada44) -> DACK1
- JCBUS_1 pad a45: unconnected-(JCBUS_1-Pin_a45-Pada45) -> DREQ2
- JCBUS_1 pad a46: unconnected-(JCBUS_1-Pin_a46-Pada46) -> DACK2
- JCBUS_1 pad a47: unconnected-(JCBUS_1-Pin_a47-Pada47) -> DREQ3
- JCBUS_1 pad a48: unconnected-(JCBUS_1-Pin_a48-Pada48) -> DACK3
- JCBUS_1 pad a49: unconnected-(JCBUS_1-Pin_a49-Pada49) -> GND
- JCBUS_1 pad a5: unconnected-(JCBUS_1-Pin_a5-Pada5) -> TX2
- JCBUS_1 pad a50: unconnected-(JCBUS_1-Pin_a50-Pada50) -> GND
- JCBUS_1 pad a6: unconnected-(JCBUS_1-Pin_a6-Pada6) -> RX2
- JCBUS_1 pad a7: unconnected-(JCBUS_1-Pin_a7-Pada7) -> TX
- JCBUS_1 pad a8: unconnected-(JCBUS_1-Pin_a8-Pada8) -> RX
- JCBUS_1 pad b1: unconnected-(JCBUS_1-Pin_b1-Padb1) -> +5V
- JCBUS_1 pad b10: unconnected-(JCBUS_1-Pin_b10-Padb10) -> IORQ
- JCBUS_1 pad b11: unconnected-(JCBUS_1-Pin_b11-Padb11) -> WR
- JCBUS_1 pad b12: unconnected-(JCBUS_1-Pin_b12-Padb12) -> RD
- JCBUS_1 pad b13: unconnected-(JCBUS_1-Pin_b13-Padb13) -> M1
- JCBUS_1 pad b14: unconnected-(JCBUS_1-Pin_b14-Padb14) -> INT
- JCBUS_1 pad b15: unconnected-(JCBUS_1-Pin_b15-Padb15) -> NMI
- JCBUS_1 pad b16: unconnected-(JCBUS_1-Pin_b16-Padb16) -> WAIT
- JCBUS_1 pad b17: unconnected-(JCBUS_1-Pin_b17-Padb17) -> HALT
- JCBUS_1 pad b18: unconnected-(JCBUS_1-Pin_b18-Padb18) -> BUSREQ
- JCBUS_1 pad b19: unconnected-(JCBUS_1-Pin_b19-Padb19) -> BUSACK
- JCBUS_1 pad b2: unconnected-(JCBUS_1-Pin_b2-Padb2) -> +12V
- JCBUS_1 pad b20: unconnected-(JCBUS_1-Pin_b20-Padb20) -> RFSH
- JCBUS_1 pad b21: unconnected-(JCBUS_1-Pin_b21-Padb21) -> IRQ0
- JCBUS_1 pad b22: unconnected-(JCBUS_1-Pin_b22-Padb22) -> IRQ1
- JCBUS_1 pad b23: unconnected-(JCBUS_1-Pin_b23-Padb23) -> IRQ2
- JCBUS_1 pad b24: unconnected-(JCBUS_1-Pin_b24-Padb24) -> IRQ3
- JCBUS_1 pad b3: unconnected-(JCBUS_1-Pin_b3-Padb3) -> -12V
- JCBUS_1 pad b4: unconnected-(JCBUS_1-Pin_b4-Padb4) -> +3.3V
- JCBUS_1 pad b41: unconnected-(JCBUS_1-Pin_b41-Padb41) -> IRQ4
- JCBUS_1 pad b42: unconnected-(JCBUS_1-Pin_b42-Padb42) -> IRQ5
- JCBUS_1 pad b43: unconnected-(JCBUS_1-Pin_b43-Padb43) -> IRQ6
- JCBUS_1 pad b44: unconnected-(JCBUS_1-Pin_b44-Padb44) -> IRQ7
- JCBUS_1 pad b45: unconnected-(JCBUS_1-Pin_b45-Padb45) -> DREQ4
- JCBUS_1 pad b46: unconnected-(JCBUS_1-Pin_b46-Padb46) -> DACK4
- JCBUS_1 pad b47: unconnected-(JCBUS_1-Pin_b47-Padb47) -> DREQ5
- JCBUS_1 pad b48: unconnected-(JCBUS_1-Pin_b48-Padb48) -> DACK5
- JCBUS_1 pad b49: unconnected-(JCBUS_1-Pin_b49-Padb49) -> +5V
- JCBUS_1 pad b5: unconnected-(JCBUS_1-Pin_b5-Padb5) -> CLK2
- JCBUS_1 pad b50: unconnected-(JCBUS_1-Pin_b50-Padb50) -> +12V
- JCBUS_1 pad b6: unconnected-(JCBUS_1-Pin_b6-Padb6) -> RESET2
- JCBUS_1 pad b7: unconnected-(JCBUS_1-Pin_b7-Padb7) -> CLK
- JCBUS_1 pad b8: unconnected-(JCBUS_1-Pin_b8-Padb8) -> RESET
- JCBUS_1 pad b9: unconnected-(JCBUS_1-Pin_b9-Padb9) -> MREQ
- JCBUS_2 pad a1: unconnected-(JCBUS_2-Pin_a1-Pada1) -> GND
- JCBUS_2 pad a2: unconnected-(JCBUS_2-Pin_a2-Pada2) -> GND
- JCBUS_2 pad a3: unconnected-(JCBUS_2-Pin_a3-Pada3) -> GND
- JCBUS_2 pad a4: unconnected-(JCBUS_2-Pin_a4-Pada4) -> GND
- JCBUS_2 pad a41: unconnected-(JCBUS_2-Pin_a41-Pada41) -> DREQ0
- JCBUS_2 pad a42: unconnected-(JCBUS_2-Pin_a42-Pada42) -> DACK0
- JCBUS_2 pad a43: unconnected-(JCBUS_2-Pin_a43-Pada43) -> DREQ1
- JCBUS_2 pad a44: unconnected-(JCBUS_2-Pin_a44-Pada44) -> DACK1
- JCBUS_2 pad a45: unconnected-(JCBUS_2-Pin_a45-Pada45) -> DREQ2
- JCBUS_2 pad a46: unconnected-(JCBUS_2-Pin_a46-Pada46) -> DACK2
- JCBUS_2 pad a47: unconnected-(JCBUS_2-Pin_a47-Pada47) -> DREQ3
- JCBUS_2 pad a48: unconnected-(JCBUS_2-Pin_a48-Pada48) -> DACK3
- JCBUS_2 pad a49: unconnected-(JCBUS_2-Pin_a49-Pada49) -> GND
- JCBUS_2 pad a5: unconnected-(JCBUS_2-Pin_a5-Pada5) -> TX2
- JCBUS_2 pad a50: unconnected-(JCBUS_2-Pin_a50-Pada50) -> GND
- JCBUS_2 pad a6: unconnected-(JCBUS_2-Pin_a6-Pada6) -> RX2
- JCBUS_2 pad a7: unconnected-(JCBUS_2-Pin_a7-Pada7) -> TX
- JCBUS_2 pad a8: unconnected-(JCBUS_2-Pin_a8-Pada8) -> RX
- JCBUS_2 pad b1: unconnected-(JCBUS_2-Pin_b1-Padb1) -> +5V
- JCBUS_2 pad b10: unconnected-(JCBUS_2-Pin_b10-Padb10) -> IORQ
- JCBUS_2 pad b11: unconnected-(JCBUS_2-Pin_b11-Padb11) -> WR
- JCBUS_2 pad b12: unconnected-(JCBUS_2-Pin_b12-Padb12) -> RD
- JCBUS_2 pad b13: unconnected-(JCBUS_2-Pin_b13-Padb13) -> M1
- JCBUS_2 pad b14: unconnected-(JCBUS_2-Pin_b14-Padb14) -> INT
- JCBUS_2 pad b15: unconnected-(JCBUS_2-Pin_b15-Padb15) -> NMI
- JCBUS_2 pad b16: unconnected-(JCBUS_2-Pin_b16-Padb16) -> WAIT
- JCBUS_2 pad b17: unconnected-(JCBUS_2-Pin_b17-Padb17) -> HALT
- JCBUS_2 pad b18: unconnected-(JCBUS_2-Pin_b18-Padb18) -> BUSREQ
- JCBUS_2 pad b19: unconnected-(JCBUS_2-Pin_b19-Padb19) -> BUSACK
- JCBUS_2 pad b2: unconnected-(JCBUS_2-Pin_b2-Padb2) -> +12V
- JCBUS_2 pad b20: unconnected-(JCBUS_2-Pin_b20-Padb20) -> RFSH
- JCBUS_2 pad b21: unconnected-(JCBUS_2-Pin_b21-Padb21) -> IRQ0
- JCBUS_2 pad b22: unconnected-(JCBUS_2-Pin_b22-Padb22) -> IRQ1
- JCBUS_2 pad b23: unconnected-(JCBUS_2-Pin_b23-Padb23) -> IRQ2
- JCBUS_2 pad b24: unconnected-(JCBUS_2-Pin_b24-Padb24) -> IRQ3
- JCBUS_2 pad b3: unconnected-(JCBUS_2-Pin_b3-Padb3) -> -12V
- JCBUS_2 pad b4: unconnected-(JCBUS_2-Pin_b4-Padb4) -> +3.3V
- JCBUS_2 pad b41: unconnected-(JCBUS_2-Pin_b41-Padb41) -> IRQ4
- JCBUS_2 pad b42: unconnected-(JCBUS_2-Pin_b42-Padb42) -> IRQ5
- JCBUS_2 pad b43: unconnected-(JCBUS_2-Pin_b43-Padb43) -> IRQ6
- JCBUS_2 pad b44: unconnected-(JCBUS_2-Pin_b44-Padb44) -> IRQ7
- JCBUS_2 pad b45: unconnected-(JCBUS_2-Pin_b45-Padb45) -> DREQ4
- JCBUS_2 pad b46: unconnected-(JCBUS_2-Pin_b46-Padb46) -> DACK4
- JCBUS_2 pad b47: unconnected-(JCBUS_2-Pin_b47-Padb47) -> DREQ5
- JCBUS_2 pad b48: unconnected-(JCBUS_2-Pin_b48-Padb48) -> DACK5
- JCBUS_2 pad b49: unconnected-(JCBUS_2-Pin_b49-Padb49) -> +5V
- JCBUS_2 pad b5: unconnected-(JCBUS_2-Pin_b5-Padb5) -> CLK2
- JCBUS_2 pad b50: unconnected-(JCBUS_2-Pin_b50-Padb50) -> +12V
- JCBUS_2 pad b6: unconnected-(JCBUS_2-Pin_b6-Padb6) -> RESET2
- JCBUS_2 pad b7: unconnected-(JCBUS_2-Pin_b7-Padb7) -> CLK
- JCBUS_2 pad b8: unconnected-(JCBUS_2-Pin_b8-Padb8) -> RESET
- JCBUS_2 pad b9: unconnected-(JCBUS_2-Pin_b9-Padb9) -> MREQ
- JCBUS_3 pad a1: unconnected-(JCBUS_3-Pin_a1-Pada1) -> GND
- JCBUS_3 pad a2: unconnected-(JCBUS_3-Pin_a2-Pada2) -> GND
- JCBUS_3 pad a3: unconnected-(JCBUS_3-Pin_a3-Pada3) -> GND
- JCBUS_3 pad a4: unconnected-(JCBUS_3-Pin_a4-Pada4) -> GND
- JCBUS_3 pad a41: unconnected-(JCBUS_3-Pin_a41-Pada41) -> DREQ0
- JCBUS_3 pad a42: unconnected-(JCBUS_3-Pin_a42-Pada42) -> DACK0
- JCBUS_3 pad a43: unconnected-(JCBUS_3-Pin_a43-Pada43) -> DREQ1
- JCBUS_3 pad a44: unconnected-(JCBUS_3-Pin_a44-Pada44) -> DACK1
- JCBUS_3 pad a45: unconnected-(JCBUS_3-Pin_a45-Pada45) -> DREQ2
- JCBUS_3 pad a46: unconnected-(JCBUS_3-Pin_a46-Pada46) -> DACK2
- JCBUS_3 pad a47: unconnected-(JCBUS_3-Pin_a47-Pada47) -> DREQ3
- JCBUS_3 pad a48: unconnected-(JCBUS_3-Pin_a48-Pada48) -> DACK3
- JCBUS_3 pad a49: unconnected-(JCBUS_3-Pin_a49-Pada49) -> GND
- JCBUS_3 pad a5: unconnected-(JCBUS_3-Pin_a5-Pada5) -> TX2
- JCBUS_3 pad a50: unconnected-(JCBUS_3-Pin_a50-Pada50) -> GND
- JCBUS_3 pad a6: unconnected-(JCBUS_3-Pin_a6-Pada6) -> RX2
- JCBUS_3 pad a7: unconnected-(JCBUS_3-Pin_a7-Pada7) -> TX
- JCBUS_3 pad a8: unconnected-(JCBUS_3-Pin_a8-Pada8) -> RX
- JCBUS_3 pad b1: unconnected-(JCBUS_3-Pin_b1-Padb1) -> +5V
- JCBUS_3 pad b10: unconnected-(JCBUS_3-Pin_b10-Padb10) -> IORQ
- JCBUS_3 pad b11: unconnected-(JCBUS_3-Pin_b11-Padb11) -> WR
- JCBUS_3 pad b12: unconnected-(JCBUS_3-Pin_b12-Padb12) -> RD
- JCBUS_3 pad b13: unconnected-(JCBUS_3-Pin_b13-Padb13) -> M1
- JCBUS_3 pad b14: unconnected-(JCBUS_3-Pin_b14-Padb14) -> INT
- JCBUS_3 pad b15: unconnected-(JCBUS_3-Pin_b15-Padb15) -> NMI
- JCBUS_3 pad b16: unconnected-(JCBUS_3-Pin_b16-Padb16) -> WAIT
- JCBUS_3 pad b17: unconnected-(JCBUS_3-Pin_b17-Padb17) -> HALT
- JCBUS_3 pad b18: unconnected-(JCBUS_3-Pin_b18-Padb18) -> BUSREQ
- JCBUS_3 pad b19: unconnected-(JCBUS_3-Pin_b19-Padb19) -> BUSACK
- JCBUS_3 pad b2: unconnected-(JCBUS_3-Pin_b2-Padb2) -> +12V
- JCBUS_3 pad b20: unconnected-(JCBUS_3-Pin_b20-Padb20) -> RFSH
- JCBUS_3 pad b21: unconnected-(JCBUS_3-Pin_b21-Padb21) -> IRQ0
- JCBUS_3 pad b22: unconnected-(JCBUS_3-Pin_b22-Padb22) -> IRQ1
- JCBUS_3 pad b23: unconnected-(JCBUS_3-Pin_b23-Padb23) -> IRQ2
- JCBUS_3 pad b24: unconnected-(JCBUS_3-Pin_b24-Padb24) -> IRQ3
- JCBUS_3 pad b3: unconnected-(JCBUS_3-Pin_b3-Padb3) -> -12V
- JCBUS_3 pad b4: unconnected-(JCBUS_3-Pin_b4-Padb4) -> +3.3V
- JCBUS_3 pad b41: unconnected-(JCBUS_3-Pin_b41-Padb41) -> IRQ4
- JCBUS_3 pad b42: unconnected-(JCBUS_3-Pin_b42-Padb42) -> IRQ5
- JCBUS_3 pad b43: unconnected-(JCBUS_3-Pin_b43-Padb43) -> IRQ6
- JCBUS_3 pad b44: unconnected-(JCBUS_3-Pin_b44-Padb44) -> IRQ7
- JCBUS_3 pad b45: unconnected-(JCBUS_3-Pin_b45-Padb45) -> DREQ4
- JCBUS_3 pad b46: unconnected-(JCBUS_3-Pin_b46-Padb46) -> DACK4
- JCBUS_3 pad b47: unconnected-(JCBUS_3-Pin_b47-Padb47) -> DREQ5
- JCBUS_3 pad b48: unconnected-(JCBUS_3-Pin_b48-Padb48) -> DACK5
- JCBUS_3 pad b49: unconnected-(JCBUS_3-Pin_b49-Padb49) -> +5V
- JCBUS_3 pad b5: unconnected-(JCBUS_3-Pin_b5-Padb5) -> CLK2
- JCBUS_3 pad b50: unconnected-(JCBUS_3-Pin_b50-Padb50) -> +12V
- JCBUS_3 pad b6: unconnected-(JCBUS_3-Pin_b6-Padb6) -> RESET2
- JCBUS_3 pad b7: unconnected-(JCBUS_3-Pin_b7-Padb7) -> CLK
- JCBUS_3 pad b8: unconnected-(JCBUS_3-Pin_b8-Padb8) -> RESET
- JCBUS_3 pad b9: unconnected-(JCBUS_3-Pin_b9-Padb9) -> MREQ
- JCBUS_4 pad a1: unconnected-(JCBUS_4-Pin_a1-Pada1) -> GND
- JCBUS_4 pad a2: unconnected-(JCBUS_4-Pin_a2-Pada2) -> GND
- JCBUS_4 pad a3: unconnected-(JCBUS_4-Pin_a3-Pada3) -> GND
- JCBUS_4 pad a4: unconnected-(JCBUS_4-Pin_a4-Pada4) -> GND
- JCBUS_4 pad a41: unconnected-(JCBUS_4-Pin_a41-Pada41) -> DREQ0
- JCBUS_4 pad a42: unconnected-(JCBUS_4-Pin_a42-Pada42) -> DACK0
- JCBUS_4 pad a43: unconnected-(JCBUS_4-Pin_a43-Pada43) -> DREQ1
- JCBUS_4 pad a44: unconnected-(JCBUS_4-Pin_a44-Pada44) -> DACK1
- JCBUS_4 pad a45: unconnected-(JCBUS_4-Pin_a45-Pada45) -> DREQ2
- JCBUS_4 pad a46: unconnected-(JCBUS_4-Pin_a46-Pada46) -> DACK2
- JCBUS_4 pad a47: unconnected-(JCBUS_4-Pin_a47-Pada47) -> DREQ3
- JCBUS_4 pad a48: unconnected-(JCBUS_4-Pin_a48-Pada48) -> DACK3
- JCBUS_4 pad a49: unconnected-(JCBUS_4-Pin_a49-Pada49) -> GND
- JCBUS_4 pad a5: unconnected-(JCBUS_4-Pin_a5-Pada5) -> TX2
- JCBUS_4 pad a50: unconnected-(JCBUS_4-Pin_a50-Pada50) -> GND
- JCBUS_4 pad a6: unconnected-(JCBUS_4-Pin_a6-Pada6) -> RX2
- JCBUS_4 pad a7: unconnected-(JCBUS_4-Pin_a7-Pada7) -> TX
- JCBUS_4 pad a8: unconnected-(JCBUS_4-Pin_a8-Pada8) -> RX
- JCBUS_4 pad b1: unconnected-(JCBUS_4-Pin_b1-Padb1) -> +5V
- JCBUS_4 pad b10: unconnected-(JCBUS_4-Pin_b10-Padb10) -> IORQ
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
Commit message: agn
Parts:
- added R3: 10K, Resistor_THT:R_Axial_DIN0207_L6.3mm_D2.5mm_P10.16mm_Horizontal, F.Cu at (170.2, 121.2)
- added R4: 10K, Resistor_THT:R_Axial_DIN0207_L6.3mm_D2.5mm_P10.16mm_Horizontal, F.Cu at (170.2, 125.2)
- added R5: 10K, Resistor_THT:R_Axial_DIN0207_L6.3mm_D2.5mm_P10.16mm_Horizontal, F.Cu at (170.2, 129.3)
- added R6: 10K, Resistor_THT:R_Axial_DIN0207_L6.3mm_D2.5mm_P10.16mm_Horizontal, F.Cu at (170.2, 133.3)
- moved C3 341.3 mm to (56.8, 255.5)
- moved D2 333.3 mm to (70.1, 323.7)
- moved D3 333.3 mm to (77.6, 316.2)
- moved D4 333.3 mm to (77.6, 323.7)
- moved D7 333.3 mm to (92.6, 316.2)
- moved D8 333.3 mm to (92.6, 323.7)
- moved R10 333.3 mm to (48.9, 321.7)
- moved R11 333.3 mm to (48.9, 325.8)
- moved R12 333.3 mm to (48.9, 329.8)
- moved R13 333.3 mm to (48.9, 333.9)
- moved R14 333.3 mm to (48.9, 337.9)
- moved R8 333.3 mm to (48.9, 313.6)
- moved R9 333.3 mm to (48.9, 317.6)
- moved D5 333.3 mm to (85.1, 316.2)
- moved D6 333.3 mm to (85.1, 323.7)
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