File: schematics/dATX_JC100.kicad_pcb (KiCad board)
At the start: 2 copper layers, 300 x 200 mm, 162 parts, among them SW1 RESET, SW2 POWER, U0 74LS00, U1 74LS04, U10 MAX232, U11 MAX232, U12 74LS00, U13 74HCT74, U14 74LS32, U15 74HCT138, U16 74LS00, U18 74AHCT125, U19 74LS04, U2 DS1233, U20 74HCT138, U21 74LS74, U22 74LS139, U3 74AHCT125, U4 74HCT139, U5 74HCT688, U6 74HCT273, U7 74HCT157, U8 74HCT138, U9 74HCT273

Commit message: ceptmmu
Parts:
- added J1: PORT_RTC_IO, Connector_PinHeader_2.54mm:PinHeader_2x06_P2.54mm_Vertical, F.Cu at (137.2, 313.7)
- added JP31: DMA_RDYA, Connector_PinHeader_2.54mm:PinHeader_1x02_P2.54mm_Vertical, F.Cu at (205.2, 128.8)
- added JP32: DMA_RDYB, Connector_PinHeader_2.54mm:PinHeader_1x02_P2.54mm_Vertical, F.Cu at (209.8, 128.8)
- added R50: 100K, Resistor_THT:R_Axial_DIN0207_L6.3mm_D2.5mm_P10.16mm_Horizontal, F.Cu at (204.5, 124.5)
- added RAM_1: IDT6116, Package_DIP:DIP-24_W15.24mm_Socket, F.Cu at (236.2, 190.5)
- added U23: 74LS32, Package_DIP:DIP-14_W7.62mm, F.Cu at (114.9, 313.4)
- added U25: DS1302+, Package_DIP:DIP-8_W7.62mm_Socket, F.Cu at (115.3, 332.9)
- added U26: 74AHCT125, Package_DIP:DIP-14_W7.62mm, F.Cu at (125.7, 313.4)
- added XTAL_RES_3: XTAL RTC 32KHz, Crystal:Crystal_Round_D3.0mm_Vertical, F.Cu at (126.6, 333.3)
- XTAL_RES_1: value XTAL RES FDC 16MHz -> XTAL FDC 16MHz
- XTAL_RES_2: value XTAL RES FDC 9.6MHz -> XTAL FDC 9.6MHz
- renumbered RAM_1 to RAM_2
Connections:
- DMA_0 pad 15: unconnected-(DMA_0-~{BUSREQ}-Pad15) -> BUSREQ
- DMA_0 pad 16: unconnected-(DMA_0-~{C5/}WAIT-Pad16) -> SEL_DMA
- DMA_0 pad 25: unconnected-(DMA_0-RDY-Pad25) -> RDY
- DMA_0 pad 37: unconnected-(DMA_0-~{INT/PULSE}-Pad37) -> INT
- R20 pad 1: Net-(JP5-B) -> Net-(RAM_2-~{CS})
- RAM_2 pad 18: Net-(JP5-B) -> Net-(RAM_2-~{CS})
- SIO_0 pad 10: unconnected-(SIO_0-~{W}/~{RDYA}-Pad10) -> RDYA
- SIO_0 pad 30: unconnected-(SIO_0-~{W}/~{RDYB}-Pad30) -> RDYB
- U1 pad 12: unconnected-(U1-Pad12) -> Net-(U1-Pad12)
- U1 pad 13: unconnected-(U1-Pad13) -> Net-(U1-Pad13)
- U3 pad 10: Net-(U8-~{Y4}) -> Net-(JP33-A)
- U8 pad 11: Net-(U8-~{Y4}) -> Net-(SIO_0-~{CE})
- U8 pad 15: Net-(SIO_0-~{CE}) -> Net-(JP33-B)

Commit message: rev1
Parts:
- added BT1: BATT_RTC, Battery:BatteryHolder_MYOUNG_BS-07-A1BJ001_CR2032, F.Cu at (131.6, 346.7)
Connections:
- FDC_0 pad 16: unconnected-(FDC_0-IRQ-Pad16) -> IRQ_FDC
- PIO_0 pad 14: IRQ_TAPE -> unconnected-(PIO_0-PA1-Pad14)
- U15 pad 13: SEL_TAPE -> SEL_RTC
