File: schematics/Carbon_Z80/Carbon_Z80.kicad_pcb (KiCad board)
At the start: 2 copper layers, 300 x 200 mm, 172 parts, among them J1 PORT_RTC_IO, SW1 RESET, SW2 POWER, U0 74LS00, U1 74LS04, U10 MAX232, U11 MAX232, U12 74LS00, U13 74HCT74, U14 74LS32, U15 74HCT138, U16 74LS00, U18 74AHCT125, U19 74LS04, U2 DS1233, U20 74HCT138, U21 74LS74, U22 74LS139, U23 74LS32, U25 DS1302+, U26 74AHCT125, U3 74AHCT125, U4 74HCT139, U5 74HCT688, U6 74HCT273, U7 74HCT157, U8 74HCT138, U9 74HCT273

Commit message: 1
Parts:
- added D18: BUSY_IDE, LED_THT:LED_D5.0mm, F.Cu at (238.2, 375.6)
- added IDE_0: IDE_Full, Connector_IDC:IDC-Header_2x20_P2.54mm_Vertical, F.Cu at (209.6, 336.8)
- added R52: 10K, Resistor_THT:R_Axial_DIN0207_L6.3mm_D2.5mm_P10.16mm_Horizontal, F.Cu at (192.7, 332.7)
- added R53: 330R, Resistor_THT:R_Axial_DIN0207_L6.3mm_D2.5mm_P10.16mm_Horizontal, F.Cu at (192.7, 336.7)
- added R54: 10K, Resistor_THT:R_Axial_DIN0207_L6.3mm_D2.5mm_P10.16mm_Horizontal, F.Cu at (192.7, 340.8)
- added R60: 5K6, Resistor_THT:R_Axial_DIN0207_L6.3mm_D2.5mm_P10.16mm_Horizontal, F.Cu at (192.7, 344.8)
- added R61: 560R, Resistor_THT:R_Axial_DIN0207_L6.3mm_D2.5mm_P10.16mm_Horizontal, F.Cu at (192.7, 348.9)
- added R62: 56K, Resistor_THT:R_Axial_DIN0207_L6.3mm_D2.5mm_P10.16mm_Horizontal, F.Cu at (192.7, 352.9)
- added R63: 5K6, Resistor_THT:R_Axial_DIN0207_L6.3mm_D2.5mm_P10.16mm_Horizontal, F.Cu at (192.7, 357.0)
- added R64: 2K2, Resistor_THT:R_Axial_DIN0207_L6.3mm_D2.5mm_P10.16mm_Horizontal, F.Cu at (192.7, 361.0)
- added R65: 20K, Resistor_THT:R_Axial_DIN0207_L6.3mm_D2.5mm_P10.16mm_Horizontal, F.Cu at (192.7, 365.1)
- added R66: 100K, Resistor_THT:R_Axial_DIN0207_L6.3mm_D2.5mm_P10.16mm_Horizontal, F.Cu at (192.7, 369.1)
- added R67: 100K, Resistor_THT:R_Axial_DIN0207_L6.3mm_D2.5mm_P10.16mm_Horizontal, F.Cu at (192.7, 373.2)
- added R68: 1M, Resistor_THT:R_Axial_DIN0207_L6.3mm_D2.5mm_P10.16mm_Horizontal, F.Cu at (192.7, 377.2)
- added R69: 100K, Resistor_THT:R_Axial_DIN0207_L6.3mm_D2.5mm_P10.16mm_Horizontal, F.Cu at (192.7, 381.3)
- added R70: 390K, Resistor_THT:R_Axial_DIN0207_L6.3mm_D2.5mm_P10.16mm_Horizontal, F.Cu at (192.7, 385.3)
- added R71: 22K, Resistor_THT:R_Axial_DIN0207_L6.3mm_D2.5mm_P10.16mm_Horizontal, F.Cu at (192.7, 389.4)
- added R72: 390K, Resistor_THT:R_Axial_DIN0207_L6.3mm_D2.5mm_P10.16mm_Horizontal, F.Cu at (192.7, 393.4)
- added TP1: TestPoint, TestPoint:TestPoint_THTPad_1.5x1.5mm_Drill0.7mm, F.Cu at (237.5, 381.1)
- added TRS_0: TAPE_IN, Connector_Audio:Jack_3.5mm_CUI_SJ1-3525N_Horizontal, F.Cu at (223.4, 391.6)
- added TRS_1: TAPE_OUT, Connector_Audio:Jack_3.5mm_CUI_SJ1-3525N_Horizontal, F.Cu at (237.6, 391.6)
- added U17: 74LS00, Package_DIP:DIP-14_W7.62mm, F.Cu at (237.3, 354.6)
- added U27: 82C55A, Package_DIP:DIP-40_W15.24mm_Socket, F.Cu at (218.4, 332.7)
- added U29: 74HCT138, Package_DIP:DIP-16_W7.62mm, F.Cu at (237.3, 332.7)
- added U37: LM555xN, Package_DIP:DIP-8_W7.62mm, F.Cu at (206.0, 393.2)
- D17: value BUSY_IDE -> BUSY_CF
- renumbered IDE_0 to IDE_1, U16 to U0
Connections:
- net Net-(CTC_0-ZC/TO1) renamed CLK_768
- net Net-(JP33-A) renamed SEL_LIO
- C1 pad 1: Net-(C1-Pad1) -> GND
- C1 pad 2: GND -> Net-(C1-Pad2)
- CTC_0 pad 16: Net-(CTC_0-~{CE}) -> SEL_CTC
- CTC_0 pad 18: Net-(CTC_0-CS0) -> unconnected-(CTC_0-CS0-Pad18)
- CTC_0 pad 19: Net-(CTC_0-CS1) -> unconnected-(CTC_0-CS1-Pad19)
- CTC_0 pad 20: Net-(CTC_0-CLK/TRG0) -> Net-(CTC_0-CLK/TRG3)
- CTC_0 pad 9: Net-(CTC_0-CLK/TRG0) -> Net-(CTC_0-CLK/TRG3)
- IDE_1 pad 23: IDER -> Net-(IDE_1-Pin_23)
- IDE_1 pad 25: IDEW -> Net-(IDE_1-Pin_25)
- IDE_1 pad 37: Net-(IDE_0-Pin_37) -> Net-(IDE_1-Pin_37)
- JCBUS_0 pad b45: DREQ4 -> unconnected-(JCBUS_0-Pin_b45-Padb45)
- JCBUS_0 pad b46: DACK4 -> unconnected-(JCBUS_0-Pin_b46-Padb46)
- JCBUS_0 pad b47: DREQ5 -> unconnected-(JCBUS_0-Pin_b47-Padb47)
- JCBUS_0 pad b48: DACK5 -> unconnected-(JCBUS_0-Pin_b48-Padb48)
- JCBUS_1 pad b45: DREQ4 -> unconnected-(JCBUS_1-Pin_b45-Padb45)
- JCBUS_1 pad b46: DACK4 -> unconnected-(JCBUS_1-Pin_b46-Padb46)
- JCBUS_1 pad b47: DREQ5 -> unconnected-(JCBUS_1-Pin_b47-Padb47)
- JCBUS_1 pad b48: DACK5 -> unconnected-(JCBUS_1-Pin_b48-Padb48)
- JCBUS_2 pad b45: DREQ4 -> unconnected-(JCBUS_2-Pin_b45-Padb45)
- JCBUS_2 pad b46: DACK4 -> unconnected-(JCBUS_2-Pin_b46-Padb46)
- JCBUS_2 pad b47: DREQ5 -> unconnected-(JCBUS_2-Pin_b47-Padb47)
- JCBUS_2 pad b48: DACK5 -> unconnected-(JCBUS_2-Pin_b48-Padb48)
- JCBUS_3 pad b45: DREQ4 -> unconnected-(JCBUS_3-Pin_b45-Padb45)
- JCBUS_3 pad b46: DACK4 -> unconnected-(JCBUS_3-Pin_b46-Padb46)
- JCBUS_3 pad b47: DREQ5 -> unconnected-(JCBUS_3-Pin_b47-Padb47)
- JCBUS_3 pad b48: DACK5 -> unconnected-(JCBUS_3-Pin_b48-Padb48)
- JCBUS_4 pad b45: DREQ4 -> unconnected-(JCBUS_4-Pin_b45-Padb45)
- JCBUS_4 pad b46: DACK4 -> unconnected-(JCBUS_4-Pin_b46-Padb46)
- JCBUS_4 pad b47: DREQ5 -> unconnected-(JCBUS_4-Pin_b47-Padb47)
- JCBUS_4 pad b48: DACK5 -> unconnected-(JCBUS_4-Pin_b48-Padb48)
- JCBUS_5 pad b45: DREQ4 -> unconnected-(JCBUS_5-Pin_b45-Padb45)
- JCBUS_5 pad b46: DACK4 -> unconnected-(JCBUS_5-Pin_b46-Padb46)
- JCBUS_5 pad b47: DREQ5 -> unconnected-(JCBUS_5-Pin_b47-Padb47)
- JCBUS_5 pad b48: DACK5 -> unconnected-(JCBUS_5-Pin_b48-Padb48)
- JP13 pad 2: Net-(JP13-B) -> TCB
- JP14 pad 2: Net-(JP13-B) -> TCB
- SIO_0 pad 27: Net-(JP13-B) -> TCB
- SIO_0 pad 28: Net-(JP13-B) -> RCB
- SIO_0 pad 34: Net-(CTC_0-CS1) -> unconnected-(SIO_0-B/~{A}-Pad34)
- SIO_0 pad 35: Net-(SIO_0-~{CE}) -> SEL_SIO
- U0 pad 1: (no net) -> Net-(C17-Pad2) (x2)
- U0 pad 10: unconnected-(U16-Pad10) -> (no net)
- U0 pad 11: unconnected-(U16-Pad11) -> unconnected-(U0-Pad11)
- U0 pad 12: unconnected-(U16-Pad12) -> unconnected-(U0-Pad12)
- U0 pad 13: unconnected-(U16-Pad13) -> unconnected-(U0-Pad13)
- U0 pad 14: (no net) -> GND
- U0 pad 2: (no net) -> Net-(C17-Pad2) (x2)
- U0 pad 3: (no net) -> Net-(R35-Pad2) (x2)
- U0 pad 7: (no net) -> +5VSB
- U0 pad 8: unconnected-(U16-Pad8) -> (no net)
- U0 pad 9: unconnected-(U16-Pad9) -> (no net)
- U0 pad 11: (no net) -> unconnected-(U0-Pad11)
- U0 pad 12: (no net) -> unconnected-(U0-Pad12)
- U0 pad 13: (no net) -> unconnected-(U0-Pad13)
- U0 pad 4: (no net) -> Net-(R35-Pad2)
- U0 pad 5: (no net) -> Net-(R35-Pad2)
- U0 pad 6: (no net) -> PS_ON
- U1 pad 1: Net-(C1-Pad1) -> Net-(C1-Pad2)
- U1 pad 6: Net-(JP2-A) -> Net-(JP2-B)
- U1 pad 9: Net-(CTC_0-CS0) -> unconnected-(U1-Pad9)
- U14 pad 2: Net-(IDE_0-Pin_37) -> Net-(IDE_1-Pin_37)
- U14 pad 6: IDEW -> Net-(IDE_1-Pin_25)
- U14 pad 8: IDER -> Net-(IDE_1-Pin_23)
- U23 pad 3: Net-(U24-Cp) -> Net-(U23-Pad3)
- U23 pad 6: Net-(U23-Pad6) -> Net-(U24-Cp)
- U26 pad 1: Net-(U23-Pad6) -> Net-(U23-Pad3)
- U26 pad 10: Net-(U24-Cp) -> Net-(U23-Pad3)
- U26 pad 2: Net-(J1-Pin_5) -> TAPE_IN_RAW
- U26 pad 4: Net-(U23-Pad6) -> Net-(U23-Pad3)
- U26 pad 5: Net-(J1-Pin_6) -> TAPE_IN
- U26 pad 8: RCT_DATA -> unconnected-(U26-Pad8)
- U8 pad 10: unconnected-(U8-~{Y5}-Pad10) -> SEL_FPU
- U8 pad 11: Net-(SIO_0-~{CE}) -> SEL_RTC
- U8 pad 12: unconnected-(U8-~{Y3}-Pad12) -> SEL_DMA
- U8 pad 13: Net-(CTC_0-~{CE}) -> SEL_PIO
- U8 pad 14: unconnected-(U8-~{Y1}-Pad14) -> SEL_CTC
- U8 pad 15: Net-(JP33-B) -> SEL_SIO
- U8 pad 7: unconnected-(U8-~{Y7}-Pad7) -> SEL_FDC
- U8 pad 9: SEL_PIO -> SEL_FDC
- XTAL_RES_0 pad 1: Net-(C1-Pad1) -> Net-(C1-Pad2)

Commit message: pdf rev 1 dun
Parts:
- moved R10 415.3 mm to (385.3, 78.2)
- moved R11 415.3 mm to (385.3, 82.3)
- moved R12 415.3 mm to (385.3, 86.3)
- moved R13 415.3 mm to (385.3, 90.4)
- moved R14 415.3 mm to (385.3, 94.4)
- moved R8 415.3 mm to (385.3, 70.1)
- moved R9 415.3 mm to (385.3, 74.2)
- moved C16 381.0 mm to (363.6, 40.2)
- moved C17 381.0 mm to (363.6, 43.3)
- moved R36 380.2 mm to (366.2, 68.8)
- moved R37 380.2 mm to (366.2, 72.8)
- moved R35 380.2 mm to (366.2, 64.7)
- moved SW1 378.7 mm to (352.2, 40.1)
- moved JP27 378.6 mm to (375.4, 53.0)
- moved R15 378.6 mm to (384.8, 24.7)
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