File: schematics/Carbon_Z80/Carbon_Z80.kicad_pcb (KiCad board)
At the start: 2 copper layers, 300 x 200 mm, 321 parts, among them SW1 RESET, SW2 POWER, U0 74LS00, U1 74LS04, U10 MAX232, U11 MAX232, U12 74LS00, U13 74HCT74, U14 74LS32, U15 74LS02, U16 74LS161, U17 74LS00, U18 74AHCT125, U19 74LS04, U2 DS1233, U20 74HCT138, U21 74LS74, U22 74LS139, U23 74LS32, U24 74HCT273, U25 DS1302+, U26 74AHCT125, U27 82C55A, U28 74LS04, U29 74HCT138, U3 74AHCT125, U30 74LS08, U33 4049UB, U34 74LS76, U35 74LS76, U37 LM555xN, U38 4070, U39 74LS161, U4 74HCT139, U40 74LS00, U41 74LS161, U42 74LS74, U43 4046, U5 74HCT688, U6 74HCT273, U7 74HCT157, U8 74HCT138, U9 74HCT273

Commit message: again
Parts:
- moved XTAL_OSC_0 64.9 mm to (119.4, 232.4)
- moved ATX_PWR_0 63.9 mm to (177.6, 199.4)
- moved C1 51.7 mm to (137.8, 224.8)
- moved C2 51.7 mm to (144.8, 224.8)
- moved TP10 51.7 mm to (147.3, 233.4)
- moved TP9 51.7 mm to (147.3, 229.9)
- moved XTAL_RES_0 51.7 mm to (136.0, 232.4)
- moved U1 51.7 mm to (152.4, 221.0)
- moved U30 30.2 mm to (255.3, 163.8)
- moved U5 29.0 mm to (233.1, 160.0)
- moved U6 29.0 mm to (243.8, 160.0)
- moved TP29 22.9 mm to (269.2, 160.6)
- moved TP30 22.9 mm to (269.2, 164.1)
- moved TP31 22.9 mm to (269.2, 167.7)
- moved TP32 22.9 mm to (269.2, 171.2)
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Changed lines of the file:
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@@
 	(title_block
 		(title "Carbon Z80 Model 150")
-		(date "2025-08-10")
+		(date "2025-08-29")
 		(rev "1")
 		(company "Jules Carboni")
@@
 	(footprint "TestPoint:TestPoint_THTPad_1.5x1.5mm_Drill0.7mm"
 		(layer "F.Cu")
-		(at 194.31 208.28)
+		(at 147.32 229.87)
 		(descr "THT rectangular pad as test Point, square 1.5mm side length, hole diameter 0.7mm")
 		(tags "test point THT pad rectangle square")
@@
 	(footprint "TestPoint:TestPoint_THTPad_1.5x1.5mm_Drill0.7mm"
 		(layer "F.Cu")
-		(at 251.46 169.66)
+		(at 274.32 170.96)
 		(descr "THT rectangular pad as test Point, square 1.5mm side length, hole diameter 0.7mm")
 		(tags "test point THT pad rectangle square")
@@
 	(footprint "TestPoint:TestPoint_THTPad_1.5x1.5mm_Drill0.7mm"
 		(layer "F.Cu")
-		(at 246.38 177.02)
+		(at 269.24 178.32)
 		(descr "THT rectangular pad as test Point, square 1.5mm side length, hole diameter 0.7mm")
 		(tags "test point THT pad rectangle square")
@@
 	(footprint "Package_DIP:DIP-20_W7.62mm"
 		(layer "F.Cu")
-		(at 219.095 185.42)
+		(at 233.06 160.02)
 		(descr "20-lead though-hole mounted DIP package, row spacing 7.62mm (300 mils)")
 		(tags "THT DIP DIL PDIP 2.54mm 7.62mm 300mil")
@@
 	(footprint "Connector_Molex:Molex_Mini-Fit_Jr_5566-24A_2x12_P4.20mm_Vertical"
 		(layer "F.Cu")
-		(at 118.99 224.79)
+		(at 177.61 199.39)
 		(descr "Molex Mini-Fit Jr. Power Connectors, old mpn/engineering number: 5566-24A, example for new mpn: 39-28-x24x, 12 Pins per row, Mounting:  (http://www.molex.com/pdm_docs/sd/039281043_sd.pdf), generated with kicad-footprint-generator")
 		(tags "connector Molex Mini-Fit_Jr vertical")
@@
 	(footprint "Package_DIP:DIP-14_W7.62mm"
 		(layer "F.Cu")
-		(at 199.39 199.39)
+		(at 152.4 220.98)
 		(descr "14-lead though-hole mounted DIP package, row spacing 7.62mm (300 mils)")
 		(tags "THT DIP DIL PDIP 2.54mm 7.62mm 300mil")
@@
 	(footprint "TestPoint:TestPoint_THTPad_1.5x1.5mm_Drill0.7mm"
 		(layer "F.Cu")
-		(at 251.46 173.21)
+		(at 274.32 174.51)
 		(descr "THT rectangular pad as test Point, square 1.5mm side length, hole diameter 0.7mm")
 		(tags "test point THT pad rectangle square")
@@
 	(footprint "Package_DIP:DIP-14_W7.62mm"
 		(layer "F.Cu")
-		(at 243.84 191.77)
+		(at 255.27 163.83)
 		(descr "14-lead though-hole mounted DIP package, row spacing 7.62mm (300 mils)")
 		(tags "THT DIP DIL PDIP 2.54mm 7.62mm 300mil")
@@
 	(footprint "TestPoint:TestPoint_THTPad_1.5x1.5mm_Drill0.7mm"
 		(layer "F.Cu")
-		(at 246.38 159.27)
+		(at 269.24 160.57)
 		(descr "THT rectangular pad as test Point, square 1.5mm side length, hole diameter 0.7mm")
 		(tags "test point THT pad rectangle square")
@@
 	(footprint "Oscillator:Oscillator_DIP-8"
 		(layer "F.Cu")
-		(at 184.15 228.6)
+		(at 119.38 232.41)
 		(descr "Oscillator, DIP8,http://cdn-reichelt.de/documents/datenblatt/B400/OSZI.pdf")
 		(tags "oscillator")
@@
 	(footprint "Capacitor_THT:C_Disc_D3.0mm_W1.6mm_P2.50mm"
 		(layer "F.Cu")
-		(at 191.81 203.2)
+		(at 144.82 224.79)
 		(descr "C, Disc series, Radial, pin pitch=2.50mm, diameter*width=3.0*1.6mm^2, Capacitor, http://www.vishay.com/docs/45233/krseries.pdf")
 		(tags "C Disc series Radial pin pitch 2.50mm diameter 3.0mm width 1.6mm Capacitor")
@@
 	(footprint "TestPoint:TestPoint_THTPad_1.5x1.5mm_Drill0.7mm"
 		(layer "F.Cu")
-		(at 246.38 169.92)
+		(at 269.24 171.22)
 		(descr "THT rectangular pad as test Point, square 1.5mm side length, hole diameter 0.7mm")
 		(tags "test point THT pad rectangle square")
@@
 	(footprint "Package_DIP:DIP-20_W7.62mm"
 		(layer "F.Cu")
-		(at 229.875 185.42)
+		(at 243.84 160.02)
 		(descr "20-lead though-hole mounted DIP package, row spacing 7.62mm (300 mils)")
 		(tags "THT DIP DIL PDIP 2.54mm 7.62mm 300mil")
@@
 	(footprint "TestPoint:TestPoint_THTPad_1.5x1.5mm_Drill0.7mm"
 		(layer "F.Cu")
-		(at 251.46 180.31)
+		(at 274.32 181.61)
 		(descr "THT rectangular pad as test Point, square 1.5mm side length, hole diameter 0.7mm")
 		(tags "test point THT pad rectangle square")
@@
 	(footprint "Package_DIP:DIP-16_W7.62mm"
 		(layer "F.Cu")
-		(at 232.41 161.29)
+		(at 219.71 166.37)
 		(descr "16-lead though-hole mounted DIP package, row spacing 7.62mm (300 mils)")
 		(tags "THT DIP DIL PDIP 2.54mm 7.62mm 300mil")
@@
 	(footprint "TestPoint:TestPoint_THTPad_1.5x1.5mm_Drill0.7mm"
 		(layer "F.Cu")
-		(at 251.46 166.11)
+		(at 274.32 167.41)
 		(descr "THT rectangular pad as test Point, square 1.5mm side length, hole diameter 0.7mm")
 		(tags "test point THT pad rectangle square")
@@
 	(footprint "TestPoint:TestPoint_THTPad_1.5x1.5mm_Drill0.7mm"
 		(layer "F.Cu")
-		(at 251.46 176.76)
+		(at 274.32 178.06)
 		(descr "THT rectangular pad as test Point, square 1.5mm side length, hole diameter 0.7mm")
 		(tags "test point THT pad rectangle square")
@@
 	(footprint "Package_DIP:DIP-40_W15.24mm_Socket"
 		(layer "F.Cu")
-		(at 171.45 143.51)
+		(at 170.18 142.24)
 		(descr "40-lead though-hole mounted DIP package, row spacing 15.24mm (600 mils), Socket")
 		(tags "THT DIP DIL PDIP 2.54mm 15.24mm 600mil Socket")
@@
 	(footprint "TestPoint:TestPoint_THTPad_1.5x1.5mm_Drill0.7mm"
 		(layer "F.Cu")
-		(at 246.38 184.12)
+		(at 269.24 185.42)
 		(descr "THT rectangular pad as test Point, square 1.5mm side length, hole diameter 0.7mm")
 		(tags "test point THT pad rectangle square")
@@
 	(footprint "Capacitor_THT:C_Disc_D3.0mm_W1.6mm_P2.50mm"
 		(layer "F.Cu")
-		(at 184.81 203.2)
+		(at 137.82 224.79)
 		(descr "C, Disc series, Radial, pin pitch=2.50mm, diameter*width=3.0*1.6mm^2, Capacitor, http://www.vishay.com/docs/45233/krseries.pdf")
 		(tags "C Disc series Radial pin pitch 2.50mm diameter 3.0mm width 1.6mm Capacitor")
@@
 	(footprint "TestPoint:TestPoint_THTPad_1.5x1.5mm_Drill0.7mm"
 		(layer "F.Cu")
-		(at 194.31 211.83)
+		(at 147.32 233.42)
 		(descr "THT rectangular pad as test Point, square 1.5mm side length, hole diameter 0.7mm")
 		(tags "test point THT pad rectangle square")
@@
 	(footprint "TestPoint:TestPoint_THTPad_1.5x1.5mm_Drill0.7mm"
 		(layer "F.Cu")
-		(at 246.38 180.57)
+		(at 269.24 181.87)
 		(descr "THT rectangular pad as test Point, square 1.5mm side length, hole diameter 0.7mm")
 		(tags "test point THT pad rectangle square")
@@
 	(footprint "TestPoint:TestPoint_THTPad_1.5x1.5mm_Drill0.7mm"
 		(layer "F.Cu")
-		(at 246.38 173.47)
+		(at 269.24 174.77)
 		(descr "THT rectangular pad as test Point, square 1.5mm side length, hole diameter 0.7mm")
 		(tags "test point THT pad rectangle square")
@@
 	(footprint "TestPoint:TestPoint_THTPad_1.5x1.5mm_Drill0.7mm"
 		(layer "F.Cu")
-		(at 246.38 162.82)
+		(at 269.24 164.12)
 		(descr "THT rectangular pad as test Point, square 1.5mm side length, hole diameter 0.7mm")
 		(tags "test point THT pad rectangle square")
@@
 	(footprint "TestPoint:TestPoint_THTPad_1.5x1.5mm_Drill0.7mm"
 		(layer "F.Cu")
-		(at 246.38 166.37)
+		(at 269.24 167.67)
 		(descr "THT rectangular pad as test Point, square 1.5mm side length, hole diameter 0.7mm")
 		(tags "test point THT pad rectangle square")
@@
 	(footprint "Crystal:Resonator-2Pin_W6.0mm_H3.0mm"
 		(layer "F.Cu")
-		(at 182.96 210.82)
+		(at 135.97 232.41)
 		(descr "Ceramic Resonator/Filter, length 3.0mm, width 6.0mm, 2 pins")
 		(tags "ceramic")
@@
 	(footprint "TestPoint:TestPoint_THTPad_1.5x1.5mm_Drill0.7mm"
 		(layer "F.Cu")
-		(at 251.46 162.56)
+		(at 274.32 163.86)
 		(descr "THT rectangular pad as test Point, square 1.5mm side length, hole diameter 0.7mm")
 		(tags "test point THT pad rectangle square")
@@
 	(footprint "Package_DIP:DIP-16_W7.62mm"
 		(layer "F.Cu")
-		(at 219.095 163.55)
+		(at 219.71 140.97)
 		(descr "16-lead though-hole mounted DIP package, row spacing 7.62mm (300 mils)")
 		(tags "THT DIP DIL PDIP 2.54mm 7.62mm 300mil")
