File: schematics/Carbon_Z80/Carbon_Z80.kicad_sch (KiCad schematic)
At the start: 250 parts, among them SW1 RESET, SW2 POWER, U0 74LS00, U1 74LS04, U10 MAX232, U11 MAX232, U12 74LS00, U13 74HCT74, U14 74LS32, U15 74LS02, U16 74LS161, U17 74LS00, U18 74AHCT125, U19 74LS04, U2 DS1233, U20 74HCT138, U21 74LS74, U22 74LS139, U23 74LS32, U24 74HCT273, U25 DS1302+, U26 74AHCT125, U27 82C55A, U28 74LS04, U29 74HCT138, U3 74AHCT125, U33 4049UB, U34 74LS76, U35 74LS76, U36 74LS153, U37 LM555xN, U38 4070, U39 74LS161, U4 74HCT139, U40 74LS00, U41 74LS161, U42 74LS74, U43 4046, U5 74HCT688, U6 74HCT273, U7 74HCT157, U8 74HCT138, U9 74HCT273

Commit message: tidy
done won
Connections:
- net IORQ: now also U12.12
- net at U15.4: now also U29.5 (~{E1})
- net at U15.5: now also U12.11, U15.6
- net at U15.11: now also U12.10, U15.12
- net at U15.13: now also U12.13
- net at U15.10: now also U8.5 (~{E1})
- net at U15.8: now also U12.8, U15.9
- no-connect marks 94 -> 104
Other:
- note added: "TODO: TEST POINTS EVERYWHERE"
- note removed: "TODO: MAKE MMU DEV SEL reuse and gates to correctly map unused bits?"
- title: Project Carbon Z80 Motherboard -> Carbon Z80 Model 150
- moved on the sheet: ATX_PWR_0, BT1, C1, C10, C11, C12, C13, C14, C15, C16, C17, C18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

Commit message: formatting
Parts:
- TRS_0, TRS_1: footprint Jack_3.5mm_CUI_SJ1-3525N_Horizontal -> Connector_Audio:Jack_3.5mm_CUI_SJ1-3525N_Horizontal
Connections:
- net at FDC_0.39 (~{IDX}), FDD_0.34 (Pin_34), FDD_0.8 (Pin_8)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: now also FDC_0.37 (WP), FDD_0.28 (Pin_28), RN2.4 (R3)
- no-connect marks 104 -> 107
Other:
- note added: "Input: D0 - RTC_DIN D4 - TAPE_IN D5 - TAPE_IN_RAW Output: D0 - TAPE_SPD_L D1 - TAPE_SPD_H D2 - TAPE_MOTOR D3 - TAPE_OUT D4 - RTC_CE D5 - RTC_WE D6 - RTC_SCLK D7 - RTC_DOUT Note: SEL_RTC = SEL_TAPE"
- note added: "JC-64/100 Expansion Slots"
- note added: "Use unbuffered CMOS inverter in analog mode (4049UB/UBE)."
- note removed: "Input: D0 - RTC_DIN D4 - TAPE_IN D5 - TAPE_IN_RAW Output: D0 - TAPE_SPD_L D1 - TAPE_SPD_H D2 - TAPE_MOTOR D3 - TAPE_OUT D4 - RTC_CE D5 - RTC_WE D6 - RTC_SCLK D7 - RTC_DOUT"
- note removed: "Must use unbuffered inverter in analog mode (4049UB/UBE)."
- moved on the sheet: C15, C18, C19, C21, C22, C23, C26, C29, C30, C38, C39, C4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
