File: schematics/Carbon_Z80/Carbon_Z80.kicad_sch (KiCad schematic)
At the start: 250 parts, among them SW1 RESET, SW2 POWER, U0 74LS00, U1 74LS04, U10 MAX232, U11 MAX232, U12 74LS00, U13 74HCT74, U14 74LS32, U15 74LS02, U16 74LS161, U17 74LS00, U18 74AHCT125, U19 74LS04, U2 DS1233, U20 74HCT138, U21 74LS74, U22 74LS139, U23 74LS32, U24 74HCT273, U25 DS1302+, U26 74AHCT125, U27 82C55A, U28 74LS04, U29 74HCT138, U3 74AHCT125, U33 4049UB, U34 74LS76, U35 74LS76, U36 74LS153, U37 LM555xN, U38 4070, U39 74LS161, U4 74HCT139, U40 74LS00, U41 74LS161, U42 74LS74, U43 4046, U5 74HCT688, U6 74HCT273, U7 74HCT157, U8 74HCT138, U9 74HCT273

Commit message: y
Other:
- note removed: "LSB"
- note removed: "MSB"
- note removed: "Swap order"
Changed lines of the file:
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@@
+		)
+	)
+	(text "9600 Hz"
+		(exclude_from_sim no)
+		(at 297.688 233.68 0)
+		(effects
+			(font
+				(size 1.27 1.27)
+			)
+			(justify right)
 		)
 	)
@@
 		)
 	)
-	(text "LSB"
-		(exclude_from_sim no)
-		(at 306.07 259.08 0)
-		(effects
-			(font
-				(size 1.27 1.27)
-			)
-			(justify right)
-		)
-	)
 	(text "D1-5"
 		(exclude_from_sim no)
@@
 		)
 	)
-	(text "MSB"
-		(exclude_from_sim no)
-		(at 306.07 270.51 0)
-		(effects
-			(font
-				(size 1.27 1.27)
-			)
-			(justify right)
-		)
-	)
 	(text "I/O write to:\n0x7X = 0111 100X"
 		(exclude_from_sim no)
@@
 		)
 	)
+	(text "19.2 kHz"
+		(exclude_from_sim no)
+		(at 297.688 231.14 0)
+		(effects
+			(font
+				(size 1.27 1.27)
+			)
+			(justify right)
+		)
+	)
 	(text "Device Decode 1:\n0x80-83 = /SIO (4b)\n0x84-87 = /CTC (4b)\n0x88-8B = /PIO (4b)\n0x8C-8F = /DMA (4b)\n0x90-90 = /AUX (1b)\n0x94-97 = /FPU (4b)\n0x98-9F = /FDC (8b)\n\nDevice Decode 2:\n0xA0-AB = /IDE (12b)\n0xAC-AF = /MMU (4b)\n0xB0-BF = /BANK (16b)"
 		(exclude_from_sim no)
@@
 		)
 	)
-	(text "MSB"
-		(exclude_from_sim no)
-		(at 307.34 223.52 0)
-		(effects
-			(font
-				(size 1.27 1.27)
-			)
-			(justify right)
-		)
-	)
 	(text "Input:\nD0 - RTC_DIN\nD4 - TAPE_IN\nD5 - TAPE_IN_RAW\n\nOutput:\nD0 - TAPE_SPD_L\nD1 - TAPE_SPD_H\nD2 - TAPE_MOTOR\nD3 - TAPE_OUT\nD4 - RTC_CE\nD5 - RTC_WE\nD6 - RTC_SCLK\nD7 - RTC_DOUT\n\nNote: SEL_RTC = SEL_TAPE"
 		(exclude_from_sim no)
@@
 		)
 	)
-	(text "Swap order"
-		(exclude_from_sim no)
-		(at 300.482 253.492 90)
-		(effects
-			(font
-				(size 1.27 1.27)
-			)
-		)
-	)
 	(text "JC-64/100 Expansion Slots"
 		(exclude_from_sim no)
@@
 		)
 	)
+	(text "38.4 kHz"
+		(exclude_from_sim no)
+		(at 297.688 228.6 0)
+		(effects
+			(font
+				(size 1.27 1.27)
+			)
+			(justify right)
+		)
+	)
 	(text "IBM Floppy 34 Pin"
 		(exclude_from_sim no)
@@
 		)
 	)
-	(text "LSB"
-		(exclude_from_sim no)
-		(at 307.34 234.95 0)
-		(effects
-			(font
-				(size 1.27 1.27)
-			)
-			(justify right)
-		)
-	)
 	(text "D0"
 		(exclude_from_sim no)
@@
 		)
 	)
+	(text "4800 Hz"
+		(exclude_from_sim no)
+		(at 297.688 236.22 0)
+		(effects
+			(font
+				(size 1.27 1.27)
+			)
+			(justify right)
+		)
+	)

Commit message: b
Connections:
- net +5V: now also U5.18 (R7), U5.7 (R2); no longer U5.12 (R4), U5.16 (R6)
- net GND: now also U5.12 (R4), U5.16 (R6); no longer U5.18 (R7), U5.7 (R2)
- net SEL_MMU: no longer names the net of U29.12 (~{Y3})
- no-connect marks 107 -> 108
Other:
- note added: "Device Decode 1: 0x80-83 = /SIO 0x84-87 = /CTC 0x88-8B = /PIO 0x8C-8F = /DMA 0x90-93 = /RTC/TAPE 0x94-97 = /FPU 0x98-9F = /FDC Device Decode 2: 0xA0-AB = /IDE (x2) 0xAC-AF = /MMU 0xB0-BF = /BANK (x4)"
- note added: "MMU Controller I/O: 0xAC-AD = 1010 110X"
- note added: "RS-232 Serial SIO"
- note added: "~4800 Hz"
- note added: "~76.8 kHz"
- note removed: "Device Decode 1: 0x80-83 = /SIO (4b) 0x84-87 = /CTC (4b) 0x88-8B = /PIO (4b) 0x8C-8F = /DMA (4b) 0x90-90 = /AUX (1b) 0x94-97 = /FPU (4b) 0x98-9F = /FDC (8b) Device Decode 2: 0xA0-AB = /IDE (12b) 0xAC-AF = /MMU (4b) 0xB0-BF = /BANK (16b)"
- note removed: "I/O write to: 0x7X = 0111 100X"
- note removed: "RS-232 Serial"
- moved on the sheet: C16, C17, C20, CPU_0, DMA_0, JP27, PIO_0, R35, R36, R37, SW2, TP1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

Commit message: mmu dun
Connections:
- removed net SEL_BANK: U29.10 (~{Y5}), U29.11 (~{Y4}), U29.7 (~{Y7}), U29.9 (~{Y6})
- no-connect marks 108 -> 112
Changed lines of the file:
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@@
 	)
 	(junction
-		(at 231.14 516.89)
-		(diameter 0)
-		(color 0 0 0 0)
-	)
-	(junction
 		(at 354.33 223.52)
 		(diameter 0)
@@
 	)
 	(junction
-		(at 231.14 511.81)
-		(diameter 0)
-		(color 0 0 0 0)
-	)
-	(junction
 		(at 137.16 543.56)
 		(diameter 0)
@@
 	)
 	(junction
-		(at 231.14 514.35)
-		(diameter 0)
-		(color 0 0 0 0)
-	)
-	(junction
 		(at 220.98 66.04)
 		(diameter 0)
@@
 	)
 	(no_connect
+		(at 231.14 519.43)
+	)
+	(no_connect
 		(at 278.13 412.75)
 	)
@@
 	)
 	(no_connect
+		(at 231.14 514.35)
+	)
+	(no_connect
 		(at 274.32 361.95)
 	)
@@
 	)
 	(no_connect
+		(at 231.14 516.89)
+	)
+	(no_connect
 		(at 349.25 533.4)
 	)
@@
 	)
 	(no_connect
+		(at 231.14 511.81)
+	)
+	(no_connect
 		(at 151.13 405.13)
 	)
@@
 	(wire
 		(pts
-			(xy 229.87 511.81) (xy 231.14 511.81)
-		)
-		(stroke
-			(width 0)
-			(type default)
-		)
-	)
-	(wire
-		(pts
 			(xy 339.09 281.94) (xy 356.87 281.94)
 		)
@@
 	(wire
 		(pts
-			(xy 231.14 516.89) (xy 232.41 516.89)
-		)
-		(stroke
-			(width 0)
-			(type default)
-		)
-	)
-	(wire
-		(pts
 			(xy 151.13 139.7) (xy 157.48 139.7)
 		)
@@
 	(wire
 		(pts
-			(xy 232.41 519.43) (xy 231.14 519.43)
-		)
-		(stroke
-			(width 0)
-			(type default)
-		)
-	)
-	(wire
-		(pts
 			(xy 142.24 330.2) (xy 139.7 330.2)
 		)
@@
 	(wire
 		(pts
-			(xy 231.14 514.35) (xy 232.41 514.35)
-		)
-		(stroke
-			(width 0)
-			(type default)
-		)
-	)
-	(wire
-		(pts
 			(xy 96.52 132.08) (xy 90.17 132.08)
 		)
@@
 	(wire
 		(pts
+			(xy 231.14 511.81) (xy 232.41 511.81)
+		)
+		(stroke
+			(width 0)
+			(type default)
+		)
+	)
+	(wire
+		(pts
 			(xy 137.16 50.8) (xy 137.16 49.53)
 		)
@@
 	(wire
 		(pts
+			(xy 231.14 519.43) (xy 232.41 519.43)
+		)
+		(stroke
+			(width 0)
+			(type default)
+		)
+	)
+	(wire
+		(pts
 			(xy 323.85 408.94) (xy 317.5 408.94)
 		)
@@
 	(wire
 		(pts
-			(xy 231.14 516.89) (xy 231.14 514.35)
-		)
-		(stroke
-			(width 0)
-			(type default)
-		)
-	)
-	(wire
-		(pts
 			(xy 365.76 179.07) (xy 365.76 148.59)
 		)
@@
 	(wire
 		(pts
-			(xy 231.14 514.35) (xy 231.14 511.81)
-		)
-		(stroke
-			(width 0)
-			(type default)
-		)
-	)
-	(wire
-		(pts
 			(xy 181.61 370.84) (xy 181.61 351.79)
 		)
@@
 		)
 	)
-	(wire
-		(pts
-			(xy 231.14 519.43) (xy 231.14 516.89)
-		)
-		(stroke
-			(width 0)
-			(type default)
-		)
-	)
 	(bus
 		(pts
@@
 	(wire
 		(pts
+			(xy 231.14 514.35) (xy 232.41 514.35)
+		)
+		(stroke
+			(width 0)
+			(type default)
+		)
+	)
+	(wire
+		(pts
 			(xy 91.44 280.67) (xy 88.9 280.67)
 		)
@@
 	(wire
 		(pts
+			(xy 231.14 516.89) (xy 232.41 516.89)
+		)
+		(stroke
+			(width 0)
+			(type default)
+		)
+	)
+	(wire
+		(pts
 			(xy 322.58 358.14) (xy 322.58 419.1)
 		)
@@
 	(wire
 		(pts
-			(xy 231.14 511.81) (xy 232.41 511.81)
-		)
-		(stroke
-			(width 0)
-			(type default)
-		)
-	)
-	(wire
-		(pts
 			(xy 127 267.97) (xy 125.73 267.97)
 		)
@@
 				(hide yes)
 			)
-		)
-	)
-	(global_label "SEL_BANK"
-		(shape output)
-		(at 229.87 511.81 180)
-		(fields_autoplaced yes)
-		(effects
-			(font
-				(size 1.27 1.27)
-			)
-			(justify right)
-		)
-		(property "Intersheetrefs" "${INTERSHEET_REFS}"
-			(at 217.5715 511.81 0)
-			(effects
-				(font
-					(size 1.27 1.27)
-				)
-				(justify right)
-				(hide yes)
-			)

Commit message: mmu
Other:
- note added: "Device Decode 1: 0x80-83 = /SIO 0x84-87 = /CTC 0x88-8B = /PIO 0x8C-8F = /DMA 0x90-93 = /RTC/TAPE 0x94-97 = /FPU 0x98-9F = /FDC Device Decode 2: 0xA0-AB = /IDE (x3) 0xAC-AF = /MMU"
- note removed: "Device Decode 1: 0x80-83 = /SIO 0x84-87 = /CTC 0x88-8B = /PIO 0x8C-8F = /DMA 0x90-93 = /RTC/TAPE 0x94-97 = /FPU 0x98-9F = /FDC Device Decode 2: 0xA0-AB = /IDE (x2) 0xAC-AF = /MMU 0xB0-BF = /BANK (x4)"
Changed lines of the file:
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@@
 		)
 	)
-	(text "Device Decode 1:\n0x80-83 = /SIO\n0x84-87 = /CTC\n0x88-8B = /PIO\n0x8C-8F = /DMA\n0x90-93 = /RTC/TAPE\n0x94-97 = /FPU\n0x98-9F = /FDC\n\nDevice Decode 2:\n0xA0-AB = /IDE (x2)\n0xAC-AF = /MMU\n0xB0-BF = /BANK (x4)"
+	(text "Device Decode 1:\n0x80-83 = /SIO\n0x84-87 = /CTC\n0x88-8B = /PIO\n0x8C-8F = /DMA\n0x90-93 = /RTC/TAPE\n0x94-97 = /FPU\n0x98-9F = /FDC\n\nDevice Decode 2:\n0xA0-AB = /IDE (x3)\n0xAC-AF = /MMU"
 		(exclude_from_sim no)
-		(at 220.98 476.758 0)
+		(at 220.98 477.52 0)
 		(effects
 			(font

Commit message: fromage
Parts:
- added C45: 100nF, symbol Device:C
- added U30: 74LS08, symbol 74xx:74LS08
Connections:
- net +5V: now also C15.1, C18.1, C19.1, C21.1, C22.1, C23.1, C26.1, C29.1, C30.1, C38.1, C39.1, C4.1, C40.1, C41.1, C42.1, C43.1, C44.1, C5.1, C6.1, U13.14 (VCC), U14.14 (VCC), U15.14 (VCC), U19.14 (VCC), U21.14 (VCC), U22.16 (VCC), U23.14 (VCC), U26.14 (VCC), U28.14 (VCC), U33.1 (VCC), U34.5 (VCC), U38.14 (VDD), U40.14 (VCC), U42.14 (VCC), C45.1, U30.14 (VCC); no longer C15.2, C18.2, C19.2, C21.2, C22.2, C23.2, C26.2, C29.2, C30.2, C38.2, C39.2, C4.2, C40.2, C41.2, C42.2, C43.2, C44.2, C5.2, C6.2, U13.7 (GND), U14.7 (GND), U15.7 (GND), U19.7 (GND), U21.7 (GND), U22.8 (GND), U23.7 (GND), U26.7 (GND), U28.7 (GND), U33.8 (VSS), U34.13 (GND), U38.7 (VSS), U40.7 (GND), U42.7 (GND)
- net GND: now also C15.2, C18.2, C19.2, C21.2, C22.2, C23.2, C26.2, C29.2, C30.2, C38.2, C39.2, C4.2, C40.2, C41.2, C42.2, C43.2, C44.2, C5.2, C6.2, U13.7 (GND), U14.7 (GND), U15.7 (GND), U19.7 (GND), U21.7 (GND), U22.8 (GND), U23.7 (GND), U26.7 (GND), U28.7 (GND), U33.8 (VSS), U34.13 (GND), U38.7 (VSS), U40.7 (GND), U42.7 (GND), C45.2, U30.7 (GND); no longer C15.1, C18.1, C19.1, C21.1, C22.1, C23.1, C26.1, C29.1, C30.1, C38.1, C39.1, C4.1, C40.1, C41.1, C42.1, C43.1, C44.1, C5.1, C6.1, U13.14 (VCC), U14.14 (VCC), U15.14 (VCC), U19.14 (VCC), U21.14 (VCC), U22.16 (VCC), U23.14 (VCC), U26.14 (VCC), U28.14 (VCC), U33.1 (VCC), U34.5 (VCC), U38.14 (VDD), U40.14 (VCC), U42.14 (VCC)
- net SEL_FDC: now also U30.3; no longer U8.7 (~{Y7}), U8.9 (~{Y6})
- net SEL_IDE: now also U30.8; no longer U29.13 (~{Y2}), U29.14 (~{Y1}), U29.15 (~{Y0})
- new net: U30.2, U8.7 (~{Y7})
- new net: U30.1, U8.9 (~{Y6})
- new net: U29.13 (~{Y2}), U30.10
- new net: U30.6, U30.9
- new net: U29.14 (~{Y1}), U30.5
- new net: U29.15 (~{Y0}), U30.4
Other:
- moved on the sheet: C15, C18, C19, C21, C22, C23, C26, C29, C30, C38, C39, C4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
