File: schematics/Carbon_Z80/Carbon_Z80.kicad_sch (KiCad schematic)
At the start: 371 parts, among them SW1 RESET, SW2 POWER, U0 74LS00, U1 74LS04, U10 MAX232, U11 MAX232, U12 74LS00, U13 74HCT74, U14 74LS32, U15 74LS02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

Commit message: again
Connections:
- net -12V: now also D6.1 (K); no longer D6.2 (A)
- net -5V: now also D8.1 (K); no longer D8.2 (A)
- net at R12.2: now also D6.2 (A); no longer D6.1 (K)
- net at R14.2: now also D8.2 (A); no longer D8.1 (K)
Other:
- moved on the sheet: D4, D5, D6, D8, R10, R11, R12, R14
