File: schematics/Carbon_Z80/Carbon_Z80-backups/Carbon_Z80.kicad_pcb (KiCad board)
At the start: 2 copper layers, 300 x 200 mm, 321 parts, among them SW1 RESET, SW2 POWER, U0 74LS00, U1 74LS04, U10 MAX232, U11 MAX232, U12 74LS00, U13 74HCT74, U14 74LS32, U15 74LS02, U16 74LS161, U17 74LS00, U18 74AHCT125, U19 74LS04, U2 DS1233, U20 74HCT138, U21 74LS74, U22 74LS139, U23 74LS32, U24 74HCT273, U25 DS1302+, U26 74AHCT125, U27 82C55A, U28 74LS04, U29 74HCT138, U3 74AHCT125, U30 74LS08, U33 4049UB, U34 74LS76, U35 74LS76, U37 LM555xN, U38 4070, U39 74LS161, U4 74HCT139, U40 74LS00, U41 74LS161, U42 74LS74, U43 4046, U5 74HCT688, U6 74HCT273, U7 74HCT157, U8 74HCT138, U9 74HCT273

Commit message: pcb prog
Parts:
- removed the U0 at (142.2, 200.7)
- removed the U14 at (371.4, 45.7)
- removed the U15 at (207.0, 144.8)
- removed the U19 at (388.1, 193.6)
- added C21: 120pF, Capacitor_THT:C_Disc_D3.0mm_W1.6mm_P2.50mm, F.Cu at (367.2, 344.8)
- added JP7: ROM_WRITE, Connector_PinHeader_2.54mm:PinHeader_1x03_P2.54mm_Vertical, F.Cu at (368.3, 325.1)
- added U0: 74LS00, Package_DIP:DIP-14_W7.62mm, F.Cu at (153.7, 200.7)
- added U0: 74LS00, Package_DIP:DIP-14_W7.62mm, F.Cu at (141.0, 200.7)
- added U14: 74LS32, Package_DIP:DIP-14_W7.62mm, F.Cu at (215.9, 322.6)
- added U14: 74LS32, Package_DIP:DIP-14_W7.62mm, F.Cu at (218.6, 345.7)
- added U15: 74LS02, Package_DIP:DIP-14_W7.62mm, F.Cu at (383.5, 168.9)
- added U15: 74HCT138, Package_DIP:DIP-16_W7.62mm, F.Cu at (358.1, 198.1)
- added U19: 74LS04, Package_DIP:DIP-14_W7.62mm, F.Cu at (345.4, 322.6)
- added U19: 74LS04, Package_DIP:DIP-14_W7.62mm, F.Cu at (334.0, 321.3)
- moved U17 361.8 mm to (206.0, 345.7)
- moved R38 355.4 mm to (205.5, 367.9)
- moved R39 355.4 mm to (205.5, 371.9)
- moved R41 355.4 mm to (205.5, 380.0)
- moved R40 355.4 mm to (205.5, 376.0)
- moved U13 336.8 mm to (205.1, 322.6)
- moved D17 333.2 mm to (219.7, 369.6)
- moved IDE_1 326.2 mm to (256.5, 327.7)
- moved U28 313.0 mm to (232.4, 388.6), turned to 90 degrees
- moved R54 299.4 mm to (204.5, 396.2)
- moved R52 299.4 mm to (204.5, 388.1)
- moved R53 299.4 mm to (204.5, 392.2)
- moved D18 271.8 mm to (219.7, 379.7)
- moved U27 259.9 mm to (233.7, 323.9)
- moved IDE_0 258.0 mm to (268.0, 327.9)
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Other:
- board text removed: ".1"
- board text removed: ".2"
- board text removed: ".4"
- board text removed: ".6"
- board text removed: ".8"
- board text removed: "0"
- board text removed: "1"
- board text removed: "1.5"
- board text removed: "10"
- board text removed: "15"
- board text removed: "1{dblquote}"
- board text removed: "2"
- board text removed: "20"
- board text removed: "25"
- board text removed: "30"
- board text removed: "40"
- board text removed: "5"
- board text removed: "50"
- board text removed: "in"
- board text removed: "mm"
