File: schem/kicad9/generated/cores/Z90/Z90.kicad_sch (KiCad schematic)
At the start: 0 parts

Commit message: kicad: generate core-level hierarchical schematics
Detailed description:
- What changed: regenerated common and core schematics for Z85/Z90/Z380/Z480, Am9513/4/5, Am95xx, and CarbonIO/DMA placeholders
- Why it changed: update generated KiCad 9 outputs to reflect the final naming and tier model
- Files/paths affected: schem/kicad9/generated/common/* and schem/kicad9/generated/cores/*
- How to run it: scripts/gen_kicad.sh (or python tools/kicadgen/src/kicadgen.py)
- What remains TODO: regenerate and commit system-level schematics
Other:
- removed sheet blk_cai_link
- removed sheet blk_regfile
- added sheet blk_regfile_state (blk_regfile_state.kicad_sch)
- added sheet blk_z180_ext (blk_z180_ext.kicad_sch)
- title: Z90 (generated) -> Z90 (P3/Z180-class) (generated)
Changed lines of the file:
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@@
 	(version 20250114)
 	(generator "kicadgen")
-	(generator_version "0.1")
+	(generator_version "0.2")
 	(paper "A3")
 	(title_block
-		(title "Z90 (generated)")
+		(title "Z90 (P3/Z180-class) (generated)")
 		(company "Project Carbon")
 		(comment 1 "Generated - do not edit in generated/")
@@
 	)
 	(text_box
-		"Generated core top: Z90  (edit mapping specs; do not hand-edit generated/)"
+		"Generated core top: Z90 (P3/Z180-class)  (edit mapping specs; do not hand-edit generated/)"
 		(exclude_from_sim no)
 		(at
@@
 		)
 		(size 114.3 7.62)
+		(margins
+			1.27
+			1.27
+			1.27
+			1.27
+		)
+		(stroke
+			(width 0)
+			(type default)
+			(color
+				0
+				0
+				0
+				1
+			)
+		)
+		(fill
+			(type color)
+			(color
+				255
+				255
+				150
+				1
+			)
+		)
+		(effects
+			(font
+				(size 1.27 1.27)
+			)
+			(justify left)
+		)
+	)
+	(text_box
+		"Presented tier: P3 (Z180-class)\nHosts P0-P2 personalities"
+		(exclude_from_sim no)
+		(at
+			12.7
+			22.86
+			0
+		)
+		(size 114.3 12.7)
 		(margins
 			1.27
@@
 		(property
 			"Sheetname"
-			"blk_regfile"
+			"blk_regfile_state"
 			(at
 				127
@@
 		(property
 			"Sheetfile"
-			"blk_regfile.kicad_sch"
+			"blk_regfile_state.kicad_sch"
 			(at
 				127
@@
 		(property
 			"Sheetname"
-			"blk_mem_fabric"
+			"blk_z180_ext"
 			(at
 				127
@@
 		(property
 			"Sheetfile"
-			"blk_mem_fabric.kicad_sch"
+			"blk_z180_ext.kicad_sch"
 			(at
 				127
@@
 		(property
 			"Sheetname"
-			"blk_csr_irq_dbg"
+			"blk_mem_fabric"
 			(at
 				12.7
@@
 		(property
 			"Sheetfile"
-			"blk_csr_irq_dbg.kicad_sch"
+			"blk_mem_fabric.kicad_sch"
 			(at
 				12.7
@@
 		(property
 			"Sheetname"
-			"blk_cai_link"
+			"blk_csr_irq_dbg"
 			(at
 				127
@@
 		(property
 			"Sheetfile"
-			"blk_cai_link.kicad_sch"
+			"blk_csr_irq_dbg.kicad_sch"
 			(at
 				127
@@
 			180
 		)
-		(effects
-			(font
-				(size 1.27 1.27)
-			)
-			(justify right)
-		)
-	)
-	(hierarchical_label
-		"CAI_CMD[31:0]"
-		(shape input)
-		(at
-			7.62
-			71.12
-			180
-		)
-		(effects
-			(font
-				(size 1.27 1.27)
-			)
-			(justify right)
-		)
-	)
-	(hierarchical_label
-		"CAI_CMD_VALID"
-		(shape input)
-		(at
-			7.62
-			73.66
-			180
-		)
-		(effects
-			(font
-				(size 1.27 1.27)
-			)
-			(justify right)
-		)
-	)
-	(hierarchical_label
-		"CAI_CMD_READY"
-		(shape output)
-		(at
-			254
-			50.8
-			0
-		)
-		(effects
-			(font
-				(size 1.27 1.27)
-			)
-			(justify left)
-		)
-	)
-	(hierarchical_label
-		"CAI_RSP[31:0]"
-		(shape output)
-		(at
-			254
-			53.34
-			0
-		)
-		(effects
-			(font
-				(size 1.27 1.27)
-			)
-			(justify left)
-		)
-	)
-	(hierarchical_label
-		"CAI_RSP_VALID"
-		(shape output)
-		(at
-			254
-			55.88
-			0
-		)
-		(effects
-			(font
-				(size 1.27 1.27)
-			)
-			(justify left)
-		)
-	)
-	(hierarchical_label
-		"CAI_RSP_READY"
-		(shape input)
-		(at
-			7.62
-			76.2
-			180
-		)
