File: schem/kicad9/generated/systems/CarbonZ380/CarbonZ380.kicad_sch (KiCad schematic)
At the start: 0 parts

Commit message: kicad: generate Carbon system hierarchical schematics
Detailed description:
- What changed: generated CarbonZ80/Z90/Z380/Z480 system schematics with CPU/FPU, memory, fabric, and platform blocks
- Why it changed: align system-level schematics with the final Z* lineage and Am95xx personalities
- Files/paths affected: schem/kicad9/generated/systems/CarbonZ80/CarbonZ80.kicad_sch, schem/kicad9/generated/systems/CarbonZ90/CarbonZ90.kicad_sch, schem/kicad9/generated/systems/CarbonZ380/CarbonZ380.kicad_sch, schem/kicad9/generated/systems/CarbonZ480/CarbonZ480.kicad_sch
- How to run it: scripts/gen_kicad.sh (or python tools/kicadgen/src/kicadgen.py)
- What remains TODO: update generator docs and add consistency checks for schematic outputs
Other:
- removed sheet blk_rc2014_adapter
- removed sheet blk_s100_adapter
- added sheet blk_CarbonDMA (../../cores/CarbonDMA/CarbonDMA.kicad_sch)
- sheet blk_cpu: file ../../cores/Z85/Z85.kicad_sch -> ../../cores/Z380/Z380.kicad_sch
- title: CarbonZ80 (generated) -> CarbonZ380 (generated)
