File: schem/Model_150/Model_150.kicad_sch (KiCad schematic)
At the start: 371 parts, among them SW1 RESET, SW2 POWER, U0 74LS00, U1 74LS04, U10 MAX232, U11 MAX232, U12 74LS00, U13 74HCT74, U14 74LS32, U15 74LS02, U16 74LS161, U17 74LS00, U18 74AHCT125, U19 74LS04, U2 DS1233, U20 74HCT138, U21 74LS74, U22 74LS139, U23 74LS32, U24 74HCT273, U25 DS1302+, U26 74AHCT125, U27 82C55A, U28 74LS04, U29 74HCT138, U3 74AHCT125, U30 74LS08, U33 4049UB, U34 74LS76, U35 74LS76, U36 74LS153, U37 LM555xN, U38 4070, U39 74LS161, U4 74HCT139, U40 74LS00, U41 74LS161, U42 74LS74, U43 4046, U5 74HCT688, U6 74HCT273, U7 74HCT157, U8 74HCT138, U9 74HCT273

Commit message: woiken
Parts:
- R7: value R -> R?
Connections:
- net A19: now reaches TP69.1
- net A19: now also JCBUS_0.a28 (Pin_a28), JCBUS_1.a28 (Pin_a28), JCBUS_2.a28 (Pin_a28), JCBUS_3.a28 (Pin_a28), JCBUS_4.a28 (Pin_a28), JCBUS_5.a28 (Pin_a28)
- net A22: now reaches TP72.1
- net A22: now also JCBUS_0.a31 (Pin_a31), JCBUS_1.a31 (Pin_a31), JCBUS_2.a31 (Pin_a31), JCBUS_3.a31 (Pin_a31), JCBUS_4.a31 (Pin_a31), JCBUS_5.a31 (Pin_a31)
- net A13: now reaches TP63.1
- net A13: now also CPU_0.3 (A13), DMA_0.19 (A13), JCBUS_0.a22 (Pin_a22), JCBUS_1.a22 (Pin_a22), JCBUS_2.a22 (Pin_a22), JCBUS_3.a22 (Pin_a22), JCBUS_4.a22 (Pin_a22), JCBUS_5.a22 (Pin_a22), RAM_0.28 (A13), ROM_0.26 (A13), ROM_1.26 (A13)
- net D1: now reaches SIO_0.1 (D1)
- net D1: now also CPU_0.15 (D1), CTC_0.26 (D1), DMA_0.34 (D1), FDC_0.8 (DB1), FPU_0.9 (DB1), JCBUS_0.b26 (Pin_b26), JCBUS_1.b26 (Pin_b26), JCBUS_2.b26 (Pin_b26), JCBUS_3.b26 (Pin_b26), JCBUS_4.b26 (Pin_b26), JCBUS_5.b26 (Pin_b26), PIO_0.20 (D1), RAM_0.14 (DQ1), RAM_1.10 (IO1), RAM_2.10 (IO1), ROM_0.12 (D1), ROM_1.12 (D1), TP83.1, U24.4 (D1), U6.4 (D1), U9.4 (D1)
- net D3: now reaches SIO_0.2 (D3)
- net D3: now also CPU_0.8 (D3), CTC_0.28 (D3), DMA_0.32 (D3), FDC_0.10 (DB3), FPU_0.11 (DB3), JCBUS_0.b28 (Pin_b28), JCBUS_1.b28 (Pin_b28), JCBUS_2.b28 (Pin_b28), JCBUS_3.b28 (Pin_b28), JCBUS_4.b28 (Pin_b28), JCBUS_5.b28 (Pin_b28), PIO_0.40 (D3), RAM_0.17 (DQ3), RAM_1.13 (IO3), RAM_2.13 (IO3), ROM_0.15 (D3), ROM_1.15 (D3), TP85.1, U24.8 (D3), U6.8 (D3), U9.8 (D3)
- net D5: now reaches SIO_0.3 (D5)
- net D5: now also CPU_0.9 (D5), CTC_0.2 (D5), DMA_0.29 (D5), FDC_0.12 (DB5), FPU_0.13 (DB5), JCBUS_0.b30 (Pin_b30), JCBUS_1.b30 (Pin_b30), JCBUS_2.b30 (Pin_b30), JCBUS_3.b30 (Pin_b30), JCBUS_4.b30 (Pin_b30), JCBUS_5.b30 (Pin_b30), PIO_0.38 (D5), RAM_0.19 (DQ5), RAM_1.15 (IO5), RAM_2.15 (IO5), ROM_0.17 (D5), ROM_1.17 (D5), TP87.1, U24.14 (D5), U26.3, U6.14 (D5), U9.14 (D5)
- net A1: now reaches SIO_0.34 (B/~{A})
- net A1: now also CPU_0.31 (A1), CTC_0.19 (CS1), DMA_0.5 (A1), JCBUS_0.a10 (Pin_a10), JCBUS_1.a10 (Pin_a10), JCBUS_2.a10 (Pin_a10), JCBUS_3.a10 (Pin_a10), JCBUS_4.a10 (Pin_a10), JCBUS_5.a10 (Pin_a10), PIO_0.5 (C/~{D}), RAM_0.11 (A1), RAM_1.7 (A1), RAM_2.7 (A1), ROM_0.9 (A1), ROM_1.9 (A1), TP51.1, U5.4 (P1)
- net D6: now reaches SIO_0.37 (D6)
- net D6: now also CPU_0.10 (D6), CTC_0.3 (D6), DMA_0.28 (D6), FDC_0.13 (DB6), FPU_0.14 (DB6), JCBUS_0.b31 (Pin_b31), JCBUS_1.b31 (Pin_b31), JCBUS_2.b31 (Pin_b31), JCBUS_3.b31 (Pin_b31), JCBUS_4.b31 (Pin_b31), JCBUS_5.b31 (Pin_b31), PIO_0.3 (D6), RAM_0.20 (DQ6), RAM_1.16 (IO6), RAM_2.16 (IO6), ROM_0.18 (D6), ROM_1.18 (D6), TP88.1, U24.17 (D6), U9.17 (D6)
- net D4: now reaches SIO_0.38 (D4)
- net D4: now also CPU_0.7 (D4), CTC_0.1 (D4), DMA_0.31 (D4), FDC_0.11 (DB4), FPU_0.12 (DB4), JCBUS_0.b29 (Pin_b29), JCBUS_1.b29 (Pin_b29), JCBUS_2.b29 (Pin_b29), JCBUS_3.b29 (Pin_b29), JCBUS_4.b29 (Pin_b29), JCBUS_5.b29 (Pin_b29), PIO_0.39 (D4), RAM_0.18 (DQ4), RAM_1.14 (IO4), RAM_2.14 (IO4), ROM_0.16 (D4), ROM_1.16 (D4), TP86.1, U24.13 (D4), U26.6, U6.13 (D4), U9.13 (D4)
- net D2: now reaches SIO_0.39 (D2)
- net D2: now also CPU_0.12 (D2), CTC_0.27 (D2), DMA_0.33 (D2), FDC_0.9 (DB2), FPU_0.10 (DB2), JCBUS_0.b27 (Pin_b27), JCBUS_1.b27 (Pin_b27), JCBUS_2.b27 (Pin_b27), JCBUS_3.b27 (Pin_b27), JCBUS_4.b27 (Pin_b27), JCBUS_5.b27 (Pin_b27), PIO_0.1 (D2), RAM_0.15 (DQ2), RAM_1.11 (IO2), RAM_2.11 (IO2), ROM_0.13 (D2), ROM_1.13 (D2), TP84.1, U24.7 (D2), U6.7 (D2), U9.7 (D2)
- net D7: now reaches SIO_0.4 (D7)
- net D7: now also CPU_0.13 (D7), CTC_0.4 (D7), DMA_0.27 (D7), FDC_0.14 (DB7), FPU_0.15 (DB7), JCBUS_0.b32 (Pin_b32), JCBUS_1.b32 (Pin_b32), JCBUS_2.b32 (Pin_b32), JCBUS_3.b32 (Pin_b32), JCBUS_4.b32 (Pin_b32), JCBUS_5.b32 (Pin_b32), PIO_0.2 (D7), RAM_0.21 (DQ7), RAM_1.17 (IO7), RAM_2.17 (IO7), ROM_0.19 (D7), ROM_1.19 (D7), TP89.1, U18.3, U24.18 (D7), U9.18 (D7)
- net D0: now reaches SIO_0.40 (D0)
- net D0: now also CPU_0.14 (D0), CTC_0.25 (D0), DMA_0.35 (D0), FDC_0.7 (DB0), FPU_0.8 (DB0), JCBUS_0.b25 (Pin_b25), JCBUS_1.b25 (Pin_b25), JCBUS_2.b25 (Pin_b25), JCBUS_3.b25 (Pin_b25), JCBUS_4.b25 (Pin_b25), JCBUS_5.b25 (Pin_b25), PIO_0.19 (D0), RAM_0.13 (DQ0), RAM_1.9 (IO0), RAM_2.9 (IO0), ROM_0.11 (D0), ROM_1.11 (D0), TP82.1, U24.3 (D0), U26.8, U9.3 (D0)
- net A[0..31]: now reaches ROM_1.10 (A0)
- net A[0..31]: now also CPU_0.30 (A0), CTC_0.18 (CS0), DMA_0.6 (A0), FDC_0.4 (A0), JCBUS_0.a9 (Pin_a9), JCBUS_1.a9 (Pin_a9), JCBUS_2.a9 (Pin_a9), JCBUS_3.a9 (Pin_a9), JCBUS_4.a9 (Pin_a9), JCBUS_5.a9 (Pin_a9), PIO_0.6 (B/~{A}), RAM_0.12 (A0), RAM_1.8 (A0), RAM_2.8 (A0), ROM_0.10 (A0), TP50.1, U1.9
- net A12: now reaches ROM_1.2 (A12)
- net A12: now also CPU_0.2 (A12), DMA_0.20 (A12), JCBUS_0.a21 (Pin_a21), JCBUS_1.a21 (Pin_a21), JCBUS_2.a21 (Pin_a21), JCBUS_3.a21 (Pin_a21), JCBUS_4.a21 (Pin_a21), JCBUS_5.a21 (Pin_a21), RAM_0.4 (A12), ROM_0.2 (A12), TP62.1
- net A10: now reaches ROM_1.21 (A10)
- net A10: now also CPU_0.40 (A10), DMA_0.22 (A10), JCBUS_0.a19 (Pin_a19), JCBUS_1.a19 (Pin_a19), JCBUS_2.a19 (Pin_a19), JCBUS_3.a19 (Pin_a19), JCBUS_4.a19 (Pin_a19), JCBUS_5.a19 (Pin_a19), RAM_0.23 (A10), RAM_1.19 (A10), RAM_2.19 (A10), ROM_0.21 (A10), TP60.1
- net A11: now reaches ROM_1.23 (A11)
- net A11: now also CPU_0.1 (A11), DMA_0.21 (A11), JCBUS_0.a20 (Pin_a20), JCBUS_1.a20 (Pin_a20), JCBUS_2.a20 (Pin_a20), JCBUS_3.a20 (Pin_a20), JCBUS_4.a20 (Pin_a20), JCBUS_5.a20 (Pin_a20), RAM_0.25 (A11), ROM_0.23 (A11), TP61.1, U1.13, U23.12
- net A9: now reaches ROM_1.24 (A9)
- net A9: now also CPU_0.39 (A9), DMA_0.23 (A9), JCBUS_0.a18 (Pin_a18), JCBUS_1.a18 (Pin_a18), JCBUS_2.a18 (Pin_a18), JCBUS_3.a18 (Pin_a18), JCBUS_4.a18 (Pin_a18), JCBUS_5.a18 (Pin_a18), RAM_0.26 (A9), RAM_1.22 (A9), RAM_2.22 (A9), ROM_0.24 (A9), TP59.1
- net A8: now reaches ROM_1.25 (A8)
- net A8: now also CPU_0.38 (A8), DMA_0.24 (A8), JCBUS_0.a17 (Pin_a17), JCBUS_1.a17 (Pin_a17), JCBUS_2.a17 (Pin_a17), JCBUS_3.a17 (Pin_a17), JCBUS_4.a17 (Pin_a17), JCBUS_5.a17 (Pin_a17), RAM_0.27 (A8), RAM_1.23 (A8), RAM_2.23 (A8), ROM_0.25 (A8), TP58.1
- net A14: now reaches ROM_1.27 (A14)
- net A14: now also CPU_0.4 (A14), DMA_0.18 (A14), JCBUS_0.a23 (Pin_a23), JCBUS_1.a23 (Pin_a23), JCBUS_2.a23 (Pin_a23), JCBUS_3.a23 (Pin_a23), JCBUS_4.a23 (Pin_a23), JCBUS_5.a23 (Pin_a23), RAM_0.3 (A14), ROM_0.27 (A14), TP64.1
- net A7: now reaches ROM_1.3 (A7)
- net A7: now also CPU_0.37 (A7), DMA_0.39 (A7), JCBUS_0.a16 (Pin_a16), JCBUS_1.a16 (Pin_a16), JCBUS_2.a16 (Pin_a16), JCBUS_3.a16 (Pin_a16), JCBUS_4.a16 (Pin_a16), JCBUS_5.a16 (Pin_a16), RAM_0.5 (A7), RAM_1.1 (A7), RAM_2.1 (A7), ROM_0.3 (A7), TP57.1, U29.6 (E2), U5.17 (P7), U8.6 (E2)
- net A6: now reaches ROM_1.4 (A6)
- net A6: now also CPU_0.36 (A6), DMA_0.40 (A6), JCBUS_0.a15 (Pin_a15), JCBUS_1.a15 (Pin_a15), JCBUS_2.a15 (Pin_a15), JCBUS_3.a15 (Pin_a15), JCBUS_4.a15 (Pin_a15), JCBUS_5.a15 (Pin_a15), RAM_0.6 (A6), RAM_1.2 (A6), RAM_2.2 (A6), ROM_0.4 (A6), TP56.1, U29.4 (~{E0}), U5.15 (P6), U8.4 (~{E0})
- net A5: now reaches ROM_1.5 (A5)
- net A5: now also CPU_0.35 (A5), DMA_0.1 (A5), JCBUS_0.a14 (Pin_a14), JCBUS_1.a14 (Pin_a14), JCBUS_2.a14 (Pin_a14), JCBUS_3.a14 (Pin_a14), JCBUS_4.a14 (Pin_a14), JCBUS_5.a14 (Pin_a14), RAM_0.7 (A5), RAM_1.3 (A5), RAM_2.3 (A5), ROM_0.5 (A5), TP55.1, U12.10, U15.11, U15.12, U5.13 (P5)
- net A4: now reaches ROM_1.6 (A4)
- net A4: now also CPU_0.34 (A4), DMA_0.2 (A4), JCBUS_0.a13 (Pin_a13), JCBUS_1.a13 (Pin_a13), JCBUS_2.a13 (Pin_a13), JCBUS_3.a13 (Pin_a13), JCBUS_4.a13 (Pin_a13), JCBUS_5.a13 (Pin_a13), RAM_0.8 (A4), RAM_1.4 (A4), RAM_2.4 (A4), ROM_0.6 (A4), TP54.1, U20.3 (A2), U29.3 (A2), U5.11 (P4), U8.3 (A2)
- net A3: now reaches ROM_1.7 (A3)
- net A3: now also CPU_0.33 (A3), DMA_0.3 (A3), JCBUS_0.a12 (Pin_a12), JCBUS_1.a12 (Pin_a12), JCBUS_2.a12 (Pin_a12), JCBUS_3.a12 (Pin_a12), JCBUS_4.a12 (Pin_a12), JCBUS_5.a12 (Pin_a12), RAM_0.9 (A3), RAM_1.5 (A3), RAM_2.5 (A3), ROM_0.7 (A3), TP53.1, U20.2 (A1), U29.2 (A1), U5.8 (P3), U8.2 (A1)
- net A2: now reaches ROM_1.8 (A2)
- net A2: now also CPU_0.32 (A2), DMA_0.4 (A2), JCBUS_0.a11 (Pin_a11), JCBUS_1.a11 (Pin_a11), JCBUS_2.a11 (Pin_a11), JCBUS_3.a11 (Pin_a11), JCBUS_4.a11 (Pin_a11), JCBUS_5.a11 (Pin_a11), RAM_0.10 (A2), RAM_1.6 (A2), RAM_2.6 (A2), ROM_0.8 (A2), TP52.1, U20.1 (A0), U29.1 (A0), U5.6 (P2), U8.1 (A0)
- net DACK: now reaches FDC_0.5 (~{DACK}), JP23.2 (C), R43.2
- net D8: now reaches TP90.1
- net D8: now also JCBUS_0.b33 (Pin_b33), JCBUS_1.b33 (Pin_b33), JCBUS_2.b33 (Pin_b33), JCBUS_3.b33 (Pin_b33), JCBUS_4.b33 (Pin_b33), JCBUS_5.b33 (Pin_b33)
- net A24: now reaches TP74.1
- net A24: now also JCBUS_0.a33 (Pin_a33), JCBUS_1.a33 (Pin_a33), JCBUS_2.a33 (Pin_a33), JCBUS_3.a33 (Pin_a33), JCBUS_4.a33 (Pin_a33), JCBUS_5.a33 (Pin_a33)
- net A15: now reaches JCBUS_4.a24 (Pin_a24)
- net A15: now also CPU_0.5 (A15), DMA_0.17 (A15), JCBUS_0.a24 (Pin_a24), JCBUS_1.a24 (Pin_a24), JCBUS_2.a24 (Pin_a24), JCBUS_3.a24 (Pin_a24), JCBUS_5.a24 (Pin_a24), TP65.1, U4.15 (E), U7.1 (S)
- net A16: now reaches JCBUS_4.a25 (Pin_a25)
- net A16: now also JCBUS_0.a25 (Pin_a25), JCBUS_1.a25 (Pin_a25), JCBUS_2.a25 (Pin_a25), JCBUS_3.a25 (Pin_a25), JCBUS_5.a25 (Pin_a25), TP66.1
- net A17: now reaches JCBUS_4.a26 (Pin_a26)
- net A17: now also JCBUS_0.a26 (Pin_a26), JCBUS_1.a26 (Pin_a26), JCBUS_2.a26 (Pin_a26), JCBUS_3.a26 (Pin_a26), JCBUS_5.a26 (Pin_a26), TP67.1
- net A18: now reaches JCBUS_4.a27 (Pin_a27)
- net A18: now also JCBUS_0.a27 (Pin_a27), JCBUS_1.a27 (Pin_a27), JCBUS_2.a27 (Pin_a27), JCBUS_3.a27 (Pin_a27), JCBUS_5.a27 (Pin_a27), TP68.1
- net A20: now reaches JCBUS_4.a29 (Pin_a29)
- net A20: now also JCBUS_0.a29 (Pin_a29), JCBUS_1.a29 (Pin_a29), JCBUS_2.a29 (Pin_a29), JCBUS_3.a29 (Pin_a29), JCBUS_5.a29 (Pin_a29), TP70.1
- net A21: now reaches JCBUS_4.a30 (Pin_a30)
- net A21: now also JCBUS_0.a30 (Pin_a30), JCBUS_1.a30 (Pin_a30), JCBUS_2.a30 (Pin_a30), JCBUS_3.a30 (Pin_a30), JCBUS_5.a30 (Pin_a30), TP71.1
- net A23: now reaches JCBUS_4.a32 (Pin_a32)
- net A23: now also JCBUS_0.a32 (Pin_a32), JCBUS_1.a32 (Pin_a32), JCBUS_2.a32 (Pin_a32), JCBUS_3.a32 (Pin_a32), JCBUS_5.a32 (Pin_a32), TP73.1
- net A25: now reaches JCBUS_4.a34 (Pin_a34)
- net A25: now also JCBUS_0.a34 (Pin_a34), JCBUS_1.a34 (Pin_a34), JCBUS_2.a34 (Pin_a34), JCBUS_3.a34 (Pin_a34), JCBUS_5.a34 (Pin_a34), TP75.1
- net A26: now reaches JCBUS_4.a35 (Pin_a35)
- net A26: now also JCBUS_0.a35 (Pin_a35), JCBUS_1.a35 (Pin_a35), JCBUS_2.a35 (Pin_a35), JCBUS_3.a35 (Pin_a35), JCBUS_5.a35 (Pin_a35), TP76.1
- net A27: now reaches JCBUS_4.a36 (Pin_a36)
- net A27: now also JCBUS_0.a36 (Pin_a36), JCBUS_1.a36 (Pin_a36), JCBUS_2.a36 (Pin_a36), JCBUS_3.a36 (Pin_a36), JCBUS_5.a36 (Pin_a36), TP77.1
- net A28: now reaches JCBUS_4.a37 (Pin_a37)
- net A28: now also JCBUS_0.a37 (Pin_a37), JCBUS_1.a37 (Pin_a37), JCBUS_2.a37 (Pin_a37), JCBUS_3.a37 (Pin_a37), JCBUS_5.a37 (Pin_a37), TP78.1
- net A29: now reaches JCBUS_4.a38 (Pin_a38)
- net A29: now also JCBUS_0.a38 (Pin_a38), JCBUS_1.a38 (Pin_a38), JCBUS_2.a38 (Pin_a38), JCBUS_3.a38 (Pin_a38), JCBUS_5.a38 (Pin_a38), TP79.1
- net A30: now reaches JCBUS_4.a39 (Pin_a39)
- net A30: now also JCBUS_0.a39 (Pin_a39), JCBUS_1.a39 (Pin_a39), JCBUS_2.a39 (Pin_a39), JCBUS_3.a39 (Pin_a39), JCBUS_5.a39 (Pin_a39), TP80.1
- net A31: now reaches JCBUS_4.a40 (Pin_a40)
- net A31: now also JCBUS_0.a40 (Pin_a40), JCBUS_1.a40 (Pin_a40), JCBUS_2.a40 (Pin_a40), JCBUS_3.a40 (Pin_a40), JCBUS_5.a40 (Pin_a40), TP81.1
- net D9: now reaches JCBUS_4.b34 (Pin_b34)
- net D9: now also JCBUS_0.b34 (Pin_b34), JCBUS_1.b34 (Pin_b34), JCBUS_2.b34 (Pin_b34), JCBUS_3.b34 (Pin_b34), JCBUS_5.b34 (Pin_b34), TP91.1
- net D10: now reaches JCBUS_4.b35 (Pin_b35)
- net D10: now also JCBUS_0.b35 (Pin_b35), JCBUS_1.b35 (Pin_b35), JCBUS_2.b35 (Pin_b35), JCBUS_3.b35 (Pin_b35), JCBUS_5.b35 (Pin_b35), TP92.1
- net D11: now reaches JCBUS_4.b36 (Pin_b36)
- net D11: now also JCBUS_0.b36 (Pin_b36), JCBUS_1.b36 (Pin_b36), JCBUS_2.b36 (Pin_b36), JCBUS_3.b36 (Pin_b36), JCBUS_5.b36 (Pin_b36), TP93.1
- net D12: now reaches JCBUS_4.b37 (Pin_b37)
- net D12: now also JCBUS_0.b37 (Pin_b37), JCBUS_1.b37 (Pin_b37), JCBUS_2.b37 (Pin_b37), JCBUS_3.b37 (Pin_b37), JCBUS_5.b37 (Pin_b37), TP94.1
- net D13: now reaches JCBUS_4.b38 (Pin_b38)
- net D13: now also JCBUS_0.b38 (Pin_b38), JCBUS_1.b38 (Pin_b38), JCBUS_2.b38 (Pin_b38), JCBUS_3.b38 (Pin_b38), JCBUS_5.b38 (Pin_b38), TP95.1
- net D14: now reaches JCBUS_4.b39 (Pin_b39)
- net D14: now also JCBUS_0.b39 (Pin_b39), JCBUS_1.b39 (Pin_b39), JCBUS_2.b39 (Pin_b39), JCBUS_3.b39 (Pin_b39), JCBUS_5.b39 (Pin_b39), TP96.1
- net D15: now reaches JCBUS_4.b40 (Pin_b40)
- net D15: now also JCBUS_0.b40 (Pin_b40), JCBUS_1.b40 (Pin_b40), JCBUS_2.b40 (Pin_b40), JCBUS_3.b40 (Pin_b40), JCBUS_5.b40 (Pin_b40), TP97.1
- net TC: now reaches FDC_0.6 (TC), JP24.2 (C), R49.2
- net at U36.10 (I0b): now also U41.14 (Q0)
- net at U36.11 (I1b): now also U41.13 (Q1)
- net at U36.12 (I2b): now also U41.12 (Q2)
- net at U36.13 (I3b): now also U41.11 (Q3), U43.3 (RefIn)
- net at R19.2, RAM_0.22 (CE#): now also JP5.3 (B); no longer JP5.1 (A)
- net at U23.13, U23.9: now also JP5.1 (A); no longer JP5.3 (B)
- net at FDC_0.37 (WP), FDC_0.39 (~{IDX}), FDD_0.28 (Pin_28)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: no longer FDD_0.34 (Pin_34), RN2.2 (R1), RN2.5 (R4), U18.2
- net MA19: now reaches U4.12 (O0), U4.2 (A0)
- net LA19: now reaches U4.14 (A0), U6.15 (Q5)
- net LA18: now reaches U6.12 (Q4), U7.14 (I0d)
- net LA15: now reaches U6.5 (Q1), U7.2 (I0a)
- net LA16: now reaches U6.6 (Q2), U7.5 (I0b)
- net LA17: now reaches U6.9 (Q3), U7.11 (I0c)
- new net: FDD_0.34 (Pin_34), RN2.2 (R1), RN2.5 (R4), U18.2
Other:
- note added: "Compact Flash"
- note added: "Control Pullups"
- note added: "IDE Storage"
- note added: "JP10-12"
- note added: "JP13-15"
- note added: "LA15-19"
- note added: "RAM Memory"
- note added: "ROM Memory"
- note added: "Unused Chips"
- note removed: "A15"
- note removed: "A3"
- note removed: "A5"
- note removed: "A6"
- note removed: "A7"
- note removed: "Control Signal Pullups"
- note removed: "D0"
- note removed: "D4"
- note removed: "D5"
- note removed: "D7"
- note removed: "DACK"
- note removed: "LA15-18"
- note removed: "RAM and ROM"
- note removed: "TC"
- moved on the sheet: BT1, C1, C10, C11, C12, C13, C14, C2, C32, C33, C34, C35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

Commit message: Assign nets, add JP5 header, add backups
Add numerous Model_150 backup ZIPs and update KiCad project files. Model_150.kicad_pcb: replace many "unconnected-..." net placeholders with proper net names (A0..A31, D0..D15, A#/D# mappings for ROM/JCBUS/IDE/FDD signals), fix a sheet path UUID, and update some testpoint/net assignments. Also add a new footprint: Connector_PinHeader_2.54mm:PinHeader_1x03 (JP5) with properties for RAM_SELECT. Project/schematic/report files were updated to reflect these changes.
Parts:
- added JP33: SIO_A0_INVERT, symbol Jumper:Jumper_3_Bridged12
Connections:
- net A1: now also IDE_1.33 (Pin_33)
- net A2: now also IDE_1.36 (Pin_36)
- net A4: now also U13.12 (D)
- net A[0..31]: now also IDE_1.35 (Pin_35)
- net D0: now also U27.34 (D0)
- net D1: now also U27.33 (D1)
- net D2: now also U27.32 (D2)
- net D3: now also U27.31 (D3)
- net D4: now also U27.30 (D4)
- net D5: now also U27.29 (D5)
- net D6: now also U27.28 (D6)
- net D7: now also U27.27 (D7)
- net PA3: now reaches U27.1 (PA3)
- net PB0: now reaches U27.18 (PB0)
- net PB1: now reaches U27.19 (PB1)
- net PA2: now reaches U27.2 (PA2)
- net PB2: now reaches U27.20 (PB2)
- net PB3: now reaches U27.21 (PB3)
- net PB4: now reaches U27.22 (PB4)
- net PB5: now reaches U27.23 (PB5)
- net PB6: now reaches U27.24 (PB6)
- net PB7: now reaches U27.25 (PB7)
- net PA1: now reaches U27.3 (PA1)
- net PA7: now reaches R51.2, U27.37 (PA7)
- net PA6: now reaches U27.38 (PA6)
- net PA5: now reaches U27.39 (PA5)
- net PA0: now reaches U27.4 (PA0)
- net PA4: now reaches U27.40 (PA4)
Other:
- note added: "100x"
- note added: "10x"
- note added: "1x"
- note removed: "A2"
- note removed: "A4"
- moved on the sheet: BT1, C36, D18, D2, D3, D4, D5, D6, D7, D8, IDE_0, R10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

Commit message: Add docs and update Model_150 schematics/backups
Add two storage PDFs to docs/storage. Reorganize Model_150 backups: delete outdated zips, rename many timestamped backup archives, and add several new backup zip files. Update KiCad project files (Model_150.kicad_pcb, .kicad_pro, .kicad_sch), update the Carboni_Library symbol file and its backup, and refresh report.txt. PCB changes include adding a board stackup, adjusting footprints (positions/rotations), setting pad orientations, and updating UUIDs and fabrication parameters to keep the project consistent for manufacture and tracking.
Parts:
- removed U17: 74LS00, Package_DIP:DIP-14_W7.62mm, symbol 74xx:74LS00
- removed U35: 74LS76, Package_DIP:DIP-16_W7.62mm, symbol 74xx:74LS76
- removed XTAL_OSC_0: Crystal Oscillator, Oscillator:Oscillator_DIP-8, symbol Device:Crystal_GND24
- added JP34: DMA_FDC, Connector_PinHeader_2.54mm:PinHeader_1x02_P2.54mm_Vertical, symbol Jumper:Jumper_2_Open
- added TP121, TP122, TP123, TP124: NC, TestPoint:TestPoint_THTPad_1.5x1.5mm_Drill0.7mm, symbol Connector:TestPoint
- added TP125: RESET, TestPoint:TestPoint_THTPad_1.5x1.5mm_Drill0.7mm, symbol Connector:TestPoint
- added unit 1 of U34
- added XTAL_OSC_0: Crystal Oscillator, Oscillator:Oscillator_DIP-8, symbol Oscillator:CXO_DIP8
- C36: value 2.1uF -> 100pF
- C37: value 2.1uF -> 2.2uF
- FPU_0: footprint Package_DIP:DIP-24_W15.24mm_Socket -> Package_DIP:DIP-24_W15.24mm
- JP1, JP2: footprint (none) -> Connector_PinHeader_2.54mm:PinHeader_1x02_P2.54mm_Vertical
- R10, R11, R12, R13, R14, R8, R9: value R -> R220
- R7: value R? -> R220
- TP22: value BUSRQ -> BUSREQ
- TP23: value BUSAK -> BUSACK
Connections:
- net BUSAK is gone; now on net BUSACK: CPU_0.23 (BUSACK), TP23.1
- net BUSRQ is gone; now on net BUSREQ: CPU_0.25 (BUSREQ), R3.2, TP22.1
- net +5V: now also U34.3 (~{R}), XTAL_OSC_0.1 (EN), XTAL_OSC_0.8 (Vcc)
- net +5VSB: now also U0.14 (VCC); no longer U0.7 (GND)
- net A1: now also U27.8 (A1)
- net A[0..31]: no longer CPU_0.30 (A0), CTC_0.18 (CS0), DMA_0.6 (A0), FDC_0.4 (A0), IDE_1.35 (Pin_35), JCBUS_0.a9 (Pin_a9), JCBUS_1.a9 (Pin_a9), JCBUS_2.a9 (Pin_a9), JCBUS_3.a9 (Pin_a9), JCBUS_4.a9 (Pin_a9), JCBUS_5.a9 (Pin_a9), PIO_0.6 (B/~{A}), RAM_0.12 (A0), RAM_1.8 (A0), RAM_2.8 (A0), ROM_0.10 (A0), ROM_1.10 (A0), TP50.1, U1.9
- net GND: now also U0.7 (GND), XTAL_OSC_0.4 (GND); no longer U0.14 (VCC)
- net M1: now also U30.12
- net PA0: now also IDE_0.17 (Pin_17)
- net PA1: now also IDE_0.15 (Pin_15)
- net PA2: now also IDE_0.13 (Pin_13)
- net PA3: now also IDE_0.11 (Pin_11)
- net PA4: now also IDE_0.9 (Pin_9)
- net PA5: now also IDE_0.7 (Pin_7)
- net PA6: now also IDE_0.5 (Pin_5)
- net PA7: now also IDE_0.3 (Pin_3)
- net PB0: now also IDE_0.4 (Pin_4)
- net PB1: now also IDE_0.6 (Pin_6)
- net PB2: now also IDE_0.8 (Pin_8)
- net PB3: now also IDE_0.10 (Pin_10)
- net PB4: now also IDE_0.12 (Pin_12)
- net PB5: now also IDE_0.14 (Pin_14)
- net PB6: now also IDE_0.16 (Pin_16)
- net PB7: now also IDE_0.18 (Pin_18)
- net RDY: now also JP34.2 (B)
- net RESET2: now also TP125.1
- net at SIO_0.33 (C/~{D}): now also JP33.2 (C); no longer U1.8
- net at U30.11: now also IDE_1.37 (Pin_37), U14.2
- net at U30.13: now also U15.1
- net at TP120.1, U34.12 (K), U34.9 (J): now also U34.15 (Q)
- net at TP119.1, U16.11 (Q3), U34.6 (C)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: now also U34.1 (C)
- net at JP1.1 (A): now also XTAL_OSC_0.5 (OUT)
- net at JCBUS_5.b45 (Pin_b45): now also TP121.1
- net at JCBUS_5.b46 (Pin_b46): now also TP122.1
- net at JCBUS_5.b47 (Pin_b47): now also TP123.1
- net at JCBUS_5.b48 (Pin_b48): now also TP124.1
- net at U33.2: now also U34.16 (K), U34.4 (J)
- net at JP40.2 (B), U33.3: now also U34.2 (~{S})
- net A0: now reaches U27.9 (A0)
- net A0: now also CPU_0.30 (A0), CTC_0.18 (CS0), DMA_0.6 (A0), FDC_0.4 (A0), FPU_0.21 (C/~{D}), IDE_1.35 (Pin_35), JCBUS_0.a9 (Pin_a9), JCBUS_1.a9 (Pin_a9), JCBUS_2.a9 (Pin_a9), JCBUS_3.a9 (Pin_a9), JCBUS_4.a9 (Pin_a9), JCBUS_5.a9 (Pin_a9), JP33.1 (A), PIO_0.6 (B/~{A}), RAM_0.12 (A0), RAM_1.8 (A0), RAM_2.8 (A0), ROM_0.10 (A0), ROM_1.10 (A0), TP50.1, U1.9
- net at JP33.3 (B): now also U1.8
- net at FDC_0.15 (DMA): now also JP34.1 (A)
- no-connect marks 115 -> 116
Other:
- note added: "Central Processor"
- note added: "Mode-2 PIO Interrupts"
- note removed: "A1"
- moved on the sheet: JP16, JP17, JP18, JP19, JP25, JP26, JP28, JP29, JP30, JP31, JP32, JP33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
