File: schem/Model_150/Model_150.kicad_sch (KiCad schematic)
At the start: 376 parts, among them SW1 RESET, SW2 POWER, U0 74LS00, U1 74LS04, U10 MAX232, U11 MAX232, U12 74LS00, U13 74HCT74, U14 74LS32, U15 74LS02, U16 74LS161, U18 74AHCT125, U19 74LS04, U2 DS1233, U20 74HCT138, U21 74LS74, U22 74LS139, U23 74LS32, U24 74HCT273, U25 DS1302+, U26 74AHCT125, U27 82C55A, U28 74LS04, U29 74HCT138, U3 74AHCT125, U30 74LS08, U33 4049UB, U34 74LS76, U36 74LS153, U37 LM555xN, U38 4070, U39 74LS161, U4 74HCT139, U40 74LS00, U41 74LS161, U42 74LS74, U43 4046, U5 74HCT688, U6 74HCT273, U7 74HCT157, U8 74HCT138, U9 74HCT273

Commit message: Update Model_150 PCB and tidy backups
Bump PCB revision and apply footprint/layout fixes. Updated Model_150.kicad_pcb (rev 1→2): replaced THT capacitor footprint to 2.00mm pin pitch, adjusted reference/value positions and silkscreen lines, and regenerated UUIDs/effects. Updated project/schematic files and symbol libraries (Carboni and Zilog). Added PDF exports and updated report.txt. Also cleaned up, renamed and added many files under schem/Model_150/Model_150-backups (removed old backups, added new ones, and renamed several archives).
Parts:
- added JP44: RST_RST2, Connector_PinHeader_2.54mm:PinHeader_1x02_P2.54mm_Vertical, symbol Jumper:Jumper_2_Open
- added TP127: BMA_BAO, TestPoint:TestPoint_THTPad_1.5x1.5mm_Drill0.7mm, symbol Connector:TestPoint
- added TP128: FDC_HDL, TestPoint:TestPoint_THTPad_1.5x1.5mm_Drill0.7mm, symbol Connector:TestPoint
- added TP129: FPU_SVACK, TestPoint:TestPoint_THTPad_1.5x1.5mm_Drill0.7mm, symbol Connector:TestPoint
- added TP130: FPU_SVREQ, TestPoint:TestPoint_THTPad_1.5x1.5mm_Drill0.7mm, symbol Connector:TestPoint
- added U17: 74LS00, Package_DIP:DIP-14_W7.62mm, symbol 74xx:74LS00
- ATX_PWR_0: footprint Molex_Mini-Fit_Jr_5566-24A_2x12_P4.20mm_Vertical -> Connector_Molex:Molex_Mini-Fit_Jr_5566-24A_2x12_P4.20mm_Vertical
- C1, C24, C27: footprint Capacitor_THT:C_Disc_D3.0mm_W1.6mm_P2.50mm -> Capacitor_THT:C_Disc_D3.4mm_W2.1mm_P2.50mm
- C10, C11, C12, C13, C14, C7, C8, C9: footprint Capacitor_THT:CP_Radial_D4.0mm_P1.50mm -> Capacitor_THT:CP_Radial_D4.0mm_P2.00mm
- C15, C18, C19, C20, C21, C22, C23, C26, C29, C30, C38, C39, C4, C40, C41, C42, C43, C44, C45, C5, C6: footprint (none) -> Capacitor_THT:C_Disc_D5.0mm_W2.5mm_P2.50mm
- C16, C17, C2, C25, C28, C3: footprint Capacitor_THT:C_Disc_D3.0mm_W1.6mm_P2.50mm -> Capacitor_THT:C_Disc_D5.0mm_W2.5mm_P2.50mm
- C31: footprint (none) -> Capacitor_THT:C_Rect_L7.0mm_W3.5mm_P5.00mm
- C34, C37: footprint (none) -> Capacitor_THT:C_Radial_D5.0mm_H11.0mm_P2.00mm
- C35, C36: footprint (none) -> Capacitor_THT:C_Disc_D3.4mm_W2.1mm_P2.50mm
- CTC_0: footprint Package_DIP:DIP-28_W15.24mm_Socket -> Package_DIP:DIP-28_W15.24mm_LongPads
- FDD_0: footprint IDC-Header_2x17_P2.54mm_Vertical -> Connector_IDC:IDC-Header_2x17_P2.54mm_Vertical
- IDE_0, IDE_1: footprint IDC-Header_2x20_P2.54mm_Vertical -> Connector_IDC:IDC-Header_2x20_P2.54mm_Vertical
- JP21: value PWR_FDC_12V -> PWR_FDD_12V
- JP22: value PWR_FDC_5V -> PWR_FDD_5V
- SERIAL_0, SERIAL_1: footprint DSUB-9_Pins_Horizontal_P2.77x2.84mm_EdgePinOffset7.70mm_Housed_MountingHolesOffset9.12mm -> Connector_Dsub:DSUB-9_Pins_Horizontal_P2.77x2.84mm_EdgePinOffset7.70mm_Housed_MountingHolesOffset9.12mm
- XTAL_RES_0: footprint Crystal:Resonator-2Pin_W6.0mm_H3.0mm -> Crystal:Resonator-2Pin_W10.0mm_H5.0mm
Connections:
- net BUSACK: now also DMA_0.14 (~{BAI})
- net GND: now also FPU_0.6 (NC), FPU_0.7 (NC)
- net RESET: now also JP44.1 (A)
- net RESET2: now also JP44.2 (B)
- net at FDC_0.35 (~{HDL}): now also TP128.1
- net at DMA_0.13 (~{BA0}): now also TP127.1
- net at FPU_0.4 (~{SVACK}): now also TP129.1
- net at FPU_0.5 (SVREQ): now also TP130.1
- no-connect marks 116 -> 118
Other:
- note added: "A1"
- note added: "A2"
- note added: "A4"
- note added: "Device Decode 1: 0x80-83 = /SIO 0x84-87 = /CTC 0x88-8B = /PIO 0x8C-8F = /DMA 0x90-93 = /RTC/TAPE 0x94-97 = /FPU 0x98-9F = /FDC (x2) Device Decode 2: 0xA0-AB = /IDE (x3) 0xAC-AF = /MMU"
- note removed: "Device Decode 1: 0x80-83 = /SIO 0x84-87 = /CTC 0x88-8B = /PIO 0x8C-8F = /DMA 0x90-93 = /RTC/TAPE 0x94-97 = /FPU 0x98-9F = /FDC Device Decode 2: 0xA0-AB = /IDE (x3) 0xAC-AF = /MMU"
- moved on the sheet: D1, JP8, JP9, R41, R7, TP121, TP122, TP123, TP124, U3B, U3D

Commit message: Add FDC jumper config, update footprints
- Added JP45 jumper for FDC_PCVAL configuration with three-pole connector
- Added JP33 jumper for SIO_A0_INVERT configuration
- Changed FDC pin 22 (DRV) from GND to +5V
- Connected FDC pin 24 (PCVAL) to new configurable net via JP45
- Updated capacitor footprints from radial to disc types
- Changed crystal resonator from 6.0mm to 10.0mm package
- Added floppy controller datasheets
- Fixed various component value formatting (R220 → 220R)
- Added power and ground symbols for jumper connections
Parts:
- removed U17: 74LS00, Package_DIP:DIP-14_W7.62mm, symbol 74xx:74LS00
- added JP45: FDC_PCVAL, Connector_PinHeader_2.54mm:PinHeader_1x03_P2.54mm_Vertical, symbol Jumper:Jumper_3_Bridged12
- C34: value 2.1uF -> 100nF; footprint Capacitor_THT:C_Radial_D5.0mm_H11.0mm_P2.00mm -> Capacitor_THT:C_Disc_D5.0mm_W2.5mm_P2.50mm
- C37: footprint Capacitor_THT:C_Radial_D5.0mm_H11.0mm_P2.00mm -> Capacitor_THT:C_Disc_D6.0mm_W2.5mm_P5.00mm
- JP33: footprint (none) -> Connector_PinHeader_2.54mm:PinHeader_1x03_P2.54mm_Vertical
- R10, R11, R12, R13, R14, R7, R8, R9: value R220 -> 220R
Connections:
- net +5V: now also FDC_0.22 (DRV), U22.15 (E), JP45.2 (C); no longer FDC_0.24 (PCVAL)
- net +5VSB: now also U0.10, U0.12, U0.13, U0.9
- net GND: now also U22.13 (A1), U22.14 (A0), JP45.3 (B); no longer FDC_0.22 (DRV)
- new net: FDC_0.24 (PCVAL), JP45.1 (A)
- no-connect marks 118 -> 111
Other:
- moved on the sheet: U0D, U22B

Commit message: updates yuo
Parts:
- removed JCBUS_0, JCBUS_1, JCBUS_2, JCBUS_3, JCBUS_4, JCBUS_5: JC100, Carboni_Library:JC100_Bus_16b, symbol Connector_Generic:Conn_02x50_Row_Letter_First
- removed TP121, TP122, TP123, TP124: NC, TestPoint:TestPoint_THTPad_1.5x1.5mm_Drill0.7mm, symbol Connector:TestPoint
- added JCBUS_1, JCBUS_2, JCBUS_3, JCBUS_4, JCBUS_5, JCBUS_6: JC64, Carboni_Library:JC64_Bus_8b, symbol Connector_Generic:Conn_02x32_Row_Letter_First
- added unit 3 of U0
- JP23: value FDC_JP1 -> FDC_DACK
- JP24: value FDC_JP2 -> FDC_TC
Connections:
- net +12V: now also JCBUS_1.b2 (Pin_b2), JCBUS_2.b2 (Pin_b2), JCBUS_3.b2 (Pin_b2), JCBUS_4.b2 (Pin_b2), JCBUS_5.b2 (Pin_b2), JCBUS_6.b2 (Pin_b2)
- net +3.3V: now also JCBUS_1.b4 (Pin_b4), JCBUS_2.b4 (Pin_b4), JCBUS_3.b4 (Pin_b4), JCBUS_4.b4 (Pin_b4), JCBUS_5.b4 (Pin_b4), JCBUS_6.b4 (Pin_b4)
- net +5V: now also JCBUS_1.b1 (Pin_b1), JCBUS_2.b1 (Pin_b1), JCBUS_3.b1 (Pin_b1), JCBUS_4.b1 (Pin_b1), JCBUS_5.b1 (Pin_b1), JCBUS_6.b1 (Pin_b1)
- net +5VSB: now also U0.10, U0.9; no longer U0.10, U0.9
- net -12V: now also JCBUS_1.b3 (Pin_b3), JCBUS_2.b3 (Pin_b3), JCBUS_3.b3 (Pin_b3), JCBUS_4.b3 (Pin_b3), JCBUS_5.b3 (Pin_b3), JCBUS_6.b3 (Pin_b3)
- net A0: now also JCBUS_1.a9 (Pin_a9), JCBUS_2.a9 (Pin_a9), JCBUS_3.a9 (Pin_a9), JCBUS_4.a9 (Pin_a9), JCBUS_5.a9 (Pin_a9), JCBUS_6.a9 (Pin_a9)
- net A1: now also JCBUS_1.a10 (Pin_a10), JCBUS_2.a10 (Pin_a10), JCBUS_3.a10 (Pin_a10), JCBUS_4.a10 (Pin_a10), JCBUS_5.a10 (Pin_a10), JCBUS_6.a10 (Pin_a10)
- net A10: now also JCBUS_1.a19 (Pin_a19), JCBUS_2.a19 (Pin_a19), JCBUS_3.a19 (Pin_a19), JCBUS_4.a19 (Pin_a19), JCBUS_5.a19 (Pin_a19), JCBUS_6.a19 (Pin_a19)
- net A11: now also JCBUS_1.a20 (Pin_a20), JCBUS_2.a20 (Pin_a20), JCBUS_3.a20 (Pin_a20), JCBUS_4.a20 (Pin_a20), JCBUS_5.a20 (Pin_a20), JCBUS_6.a20 (Pin_a20)
- net A12: now also JCBUS_1.a21 (Pin_a21), JCBUS_2.a21 (Pin_a21), JCBUS_3.a21 (Pin_a21), JCBUS_4.a21 (Pin_a21), JCBUS_5.a21 (Pin_a21), JCBUS_6.a21 (Pin_a21)
- net A13: now also JCBUS_1.a22 (Pin_a22), JCBUS_2.a22 (Pin_a22), JCBUS_3.a22 (Pin_a22), JCBUS_4.a22 (Pin_a22), JCBUS_5.a22 (Pin_a22), JCBUS_6.a22 (Pin_a22)
- net A14: now also JCBUS_1.a23 (Pin_a23), JCBUS_2.a23 (Pin_a23), JCBUS_3.a23 (Pin_a23), JCBUS_4.a23 (Pin_a23), JCBUS_5.a23 (Pin_a23), JCBUS_6.a23 (Pin_a23)
- net A15: now also JCBUS_1.a24 (Pin_a24), JCBUS_2.a24 (Pin_a24), JCBUS_3.a24 (Pin_a24), JCBUS_4.a24 (Pin_a24), JCBUS_5.a24 (Pin_a24), JCBUS_6.a24 (Pin_a24)
- net A16: now also JCBUS_1.a25 (Pin_a25), JCBUS_2.a25 (Pin_a25), JCBUS_3.a25 (Pin_a25), JCBUS_4.a25 (Pin_a25), JCBUS_5.a25 (Pin_a25), JCBUS_6.a25 (Pin_a25)
- net A17: now also JCBUS_1.a26 (Pin_a26), JCBUS_2.a26 (Pin_a26), JCBUS_3.a26 (Pin_a26), JCBUS_4.a26 (Pin_a26), JCBUS_5.a26 (Pin_a26), JCBUS_6.a26 (Pin_a26)
- net A18: now also JCBUS_1.a27 (Pin_a27), JCBUS_2.a27 (Pin_a27), JCBUS_3.a27 (Pin_a27), JCBUS_4.a27 (Pin_a27), JCBUS_5.a27 (Pin_a27), JCBUS_6.a27 (Pin_a27)
- net A19: now also JCBUS_1.a28 (Pin_a28), JCBUS_2.a28 (Pin_a28), JCBUS_3.a28 (Pin_a28), JCBUS_4.a28 (Pin_a28), JCBUS_5.a28 (Pin_a28), JCBUS_6.a28 (Pin_a28)
- net A2: now also JCBUS_1.a11 (Pin_a11), JCBUS_2.a11 (Pin_a11), JCBUS_3.a11 (Pin_a11), JCBUS_4.a11 (Pin_a11), JCBUS_5.a11 (Pin_a11), JCBUS_6.a11 (Pin_a11)
- net A20: now also JCBUS_1.a29 (Pin_a29), JCBUS_2.a29 (Pin_a29), JCBUS_3.a29 (Pin_a29), JCBUS_4.a29 (Pin_a29), JCBUS_5.a29 (Pin_a29), JCBUS_6.a29 (Pin_a29)
- net A21: now also JCBUS_1.a30 (Pin_a30), JCBUS_2.a30 (Pin_a30), JCBUS_3.a30 (Pin_a30), JCBUS_4.a30 (Pin_a30), JCBUS_5.a30 (Pin_a30), JCBUS_6.a30 (Pin_a30)
- net A22: now also JCBUS_1.a31 (Pin_a31), JCBUS_2.a31 (Pin_a31), JCBUS_3.a31 (Pin_a31), JCBUS_4.a31 (Pin_a31), JCBUS_5.a31 (Pin_a31), JCBUS_6.a31 (Pin_a31)
- net A23: now also JCBUS_1.a32 (Pin_a32), JCBUS_2.a32 (Pin_a32), JCBUS_3.a32 (Pin_a32), JCBUS_4.a32 (Pin_a32), JCBUS_5.a32 (Pin_a32), JCBUS_6.a32 (Pin_a32)
- net A3: now also JCBUS_1.a12 (Pin_a12), JCBUS_2.a12 (Pin_a12), JCBUS_3.a12 (Pin_a12), JCBUS_4.a12 (Pin_a12), JCBUS_5.a12 (Pin_a12), JCBUS_6.a12 (Pin_a12)
- net A4: now also JCBUS_1.a13 (Pin_a13), JCBUS_2.a13 (Pin_a13), JCBUS_3.a13 (Pin_a13), JCBUS_4.a13 (Pin_a13), JCBUS_5.a13 (Pin_a13), JCBUS_6.a13 (Pin_a13)
- net A5: now also JCBUS_1.a14 (Pin_a14), JCBUS_2.a14 (Pin_a14), JCBUS_3.a14 (Pin_a14), JCBUS_4.a14 (Pin_a14), JCBUS_5.a14 (Pin_a14), JCBUS_6.a14 (Pin_a14)
- net A6: now also JCBUS_1.a15 (Pin_a15), JCBUS_2.a15 (Pin_a15), JCBUS_3.a15 (Pin_a15), JCBUS_4.a15 (Pin_a15), JCBUS_5.a15 (Pin_a15), JCBUS_6.a15 (Pin_a15)
- net A7: now also JCBUS_1.a16 (Pin_a16), JCBUS_2.a16 (Pin_a16), JCBUS_3.a16 (Pin_a16), JCBUS_4.a16 (Pin_a16), JCBUS_5.a16 (Pin_a16), JCBUS_6.a16 (Pin_a16)
- net A8: now also JCBUS_1.a17 (Pin_a17), JCBUS_2.a17 (Pin_a17), JCBUS_3.a17 (Pin_a17), JCBUS_4.a17 (Pin_a17), JCBUS_5.a17 (Pin_a17), JCBUS_6.a17 (Pin_a17)
- net A9: now also JCBUS_1.a18 (Pin_a18), JCBUS_2.a18 (Pin_a18), JCBUS_3.a18 (Pin_a18), JCBUS_4.a18 (Pin_a18), JCBUS_5.a18 (Pin_a18), JCBUS_6.a18 (Pin_a18)
- net BUSACK: now also JCBUS_1.b19 (Pin_b19), JCBUS_2.b19 (Pin_b19), JCBUS_3.b19 (Pin_b19), JCBUS_4.b19 (Pin_b19), JCBUS_5.b19 (Pin_b19), JCBUS_6.b19 (Pin_b19)
- net BUSREQ: now also JCBUS_1.b18 (Pin_b18), JCBUS_2.b18 (Pin_b18), JCBUS_3.b18 (Pin_b18), JCBUS_4.b18 (Pin_b18), JCBUS_5.b18 (Pin_b18), JCBUS_6.b18 (Pin_b18)
- net CLK: now also JCBUS_1.b7 (Pin_b7), JCBUS_2.b7 (Pin_b7), JCBUS_3.b7 (Pin_b7), JCBUS_4.b7 (Pin_b7), JCBUS_5.b7 (Pin_b7), JCBUS_6.b7 (Pin_b7)
- net CLK2: now also JCBUS_1.b5 (Pin_b5), JCBUS_2.b5 (Pin_b5), JCBUS_3.b5 (Pin_b5), JCBUS_4.b5 (Pin_b5), JCBUS_5.b5 (Pin_b5), JCBUS_6.b5 (Pin_b5)
- net D0: now also JCBUS_1.b25 (Pin_b25), JCBUS_2.b25 (Pin_b25), JCBUS_3.b25 (Pin_b25), JCBUS_4.b25 (Pin_b25), JCBUS_5.b25 (Pin_b25), JCBUS_6.b25 (Pin_b25)
- net D1: now also JCBUS_1.b26 (Pin_b26), JCBUS_2.b26 (Pin_b26), JCBUS_3.b26 (Pin_b26), JCBUS_4.b26 (Pin_b26), JCBUS_5.b26 (Pin_b26), JCBUS_6.b26 (Pin_b26)
- net D2: now also JCBUS_1.b27 (Pin_b27), JCBUS_2.b27 (Pin_b27), JCBUS_3.b27 (Pin_b27), JCBUS_4.b27 (Pin_b27), JCBUS_5.b27 (Pin_b27), JCBUS_6.b27 (Pin_b27)
- net D3: now also JCBUS_1.b28 (Pin_b28), JCBUS_2.b28 (Pin_b28), JCBUS_3.b28 (Pin_b28), JCBUS_4.b28 (Pin_b28), JCBUS_5.b28 (Pin_b28), JCBUS_6.b28 (Pin_b28)
- net D4: now also JCBUS_1.b29 (Pin_b29), JCBUS_2.b29 (Pin_b29), JCBUS_3.b29 (Pin_b29), JCBUS_4.b29 (Pin_b29), JCBUS_5.b29 (Pin_b29), JCBUS_6.b29 (Pin_b29)
- net D5: now also JCBUS_1.b30 (Pin_b30), JCBUS_2.b30 (Pin_b30), JCBUS_3.b30 (Pin_b30), JCBUS_4.b30 (Pin_b30), JCBUS_5.b30 (Pin_b30), JCBUS_6.b30 (Pin_b30)
- net D6: now also JCBUS_1.b31 (Pin_b31), JCBUS_2.b31 (Pin_b31), JCBUS_3.b31 (Pin_b31), JCBUS_4.b31 (Pin_b31), JCBUS_5.b31 (Pin_b31), JCBUS_6.b31 (Pin_b31)
- net D7: now also JCBUS_1.b32 (Pin_b32), JCBUS_2.b32 (Pin_b32), JCBUS_3.b32 (Pin_b32), JCBUS_4.b32 (Pin_b32), JCBUS_5.b32 (Pin_b32), JCBUS_6.b32 (Pin_b32)
- net GND: now also JCBUS_1.a1 (Pin_a1), JCBUS_1.a2 (Pin_a2), JCBUS_1.a3 (Pin_a3), JCBUS_1.a4 (Pin_a4), JCBUS_2.a1 (Pin_a1), JCBUS_2.a2 (Pin_a2), JCBUS_2.a3 (Pin_a3), JCBUS_2.a4 (Pin_a4), JCBUS_3.a1 (Pin_a1), JCBUS_3.a2 (Pin_a2), JCBUS_3.a3 (Pin_a3), JCBUS_3.a4 (Pin_a4), JCBUS_4.a1 (Pin_a1), JCBUS_4.a2 (Pin_a2), JCBUS_4.a3 (Pin_a3), JCBUS_4.a4 (Pin_a4), JCBUS_5.a1 (Pin_a1), JCBUS_5.a2 (Pin_a2), JCBUS_5.a3 (Pin_a3), JCBUS_5.a4 (Pin_a4), JCBUS_6.a1 (Pin_a1), JCBUS_6.a2 (Pin_a2), JCBUS_6.a3 (Pin_a3), JCBUS_6.a4 (Pin_a4)
- net HALT: now also JCBUS_1.b17 (Pin_b17), JCBUS_2.b17 (Pin_b17), JCBUS_3.b17 (Pin_b17), JCBUS_4.b17 (Pin_b17), JCBUS_5.b17 (Pin_b17), JCBUS_6.b17 (Pin_b17)
- net INT: now also JCBUS_1.b14 (Pin_b14), JCBUS_2.b14 (Pin_b14), JCBUS_3.b14 (Pin_b14), JCBUS_4.b14 (Pin_b14), JCBUS_5.b14 (Pin_b14), JCBUS_6.b14 (Pin_b14)
- net IORQ: now also DMA_0.10 (~{IORQ}), JCBUS_1.b10 (Pin_b10), JCBUS_2.b10 (Pin_b10), JCBUS_3.b10 (Pin_b10), JCBUS_4.b10 (Pin_b10), JCBUS_5.b10 (Pin_b10), JCBUS_6.b10 (Pin_b10); no longer DMA_0.12 (~{MREQ})
- net IRQ0: now also JCBUS_1.b21 (Pin_b21), JCBUS_2.b21 (Pin_b21), JCBUS_3.b21 (Pin_b21), JCBUS_4.b21 (Pin_b21), JCBUS_5.b21 (Pin_b21), JCBUS_6.b21 (Pin_b21)
- net IRQ1: now also JCBUS_1.b22 (Pin_b22), JCBUS_2.b22 (Pin_b22), JCBUS_3.b22 (Pin_b22), JCBUS_4.b22 (Pin_b22), JCBUS_5.b22 (Pin_b22), JCBUS_6.b22 (Pin_b22)
- net IRQ2: now also JCBUS_1.b23 (Pin_b23), JCBUS_2.b23 (Pin_b23), JCBUS_3.b23 (Pin_b23), JCBUS_4.b23 (Pin_b23), JCBUS_5.b23 (Pin_b23), JCBUS_6.b23 (Pin_b23)
- net IRQ3: now also JCBUS_1.b24 (Pin_b24), JCBUS_2.b24 (Pin_b24), JCBUS_3.b24 (Pin_b24), JCBUS_4.b24 (Pin_b24), JCBUS_5.b24 (Pin_b24), JCBUS_6.b24 (Pin_b24)
- net M1: now also JCBUS_1.b13 (Pin_b13), JCBUS_2.b13 (Pin_b13), JCBUS_3.b13 (Pin_b13), JCBUS_4.b13 (Pin_b13), JCBUS_5.b13 (Pin_b13), JCBUS_6.b13 (Pin_b13)
- net MREQ: now also DMA_0.12 (~{MREQ}), JCBUS_1.b9 (Pin_b9), JCBUS_2.b9 (Pin_b9), JCBUS_3.b9 (Pin_b9), JCBUS_4.b9 (Pin_b9), JCBUS_5.b9 (Pin_b9), JCBUS_6.b9 (Pin_b9); no longer DMA_0.10 (~{IORQ})
- net NMI: now also JCBUS_1.b15 (Pin_b15), JCBUS_2.b15 (Pin_b15), JCBUS_3.b15 (Pin_b15), JCBUS_4.b15 (Pin_b15), JCBUS_5.b15 (Pin_b15), JCBUS_6.b15 (Pin_b15)
- net RD: now also JCBUS_1.b12 (Pin_b12), JCBUS_2.b12 (Pin_b12), JCBUS_3.b12 (Pin_b12), JCBUS_4.b12 (Pin_b12), JCBUS_5.b12 (Pin_b12), JCBUS_6.b12 (Pin_b12)
- net RESET: now also JCBUS_1.b8 (Pin_b8), JCBUS_2.b8 (Pin_b8), JCBUS_3.b8 (Pin_b8), JCBUS_4.b8 (Pin_b8), JCBUS_5.b8 (Pin_b8), JCBUS_6.b8 (Pin_b8)
- net RESET2: now also JCBUS_1.b6 (Pin_b6), JCBUS_2.b6 (Pin_b6), JCBUS_3.b6 (Pin_b6), JCBUS_4.b6 (Pin_b6), JCBUS_5.b6 (Pin_b6), JCBUS_6.b6 (Pin_b6)
- net RFSH: now also JCBUS_1.b20 (Pin_b20), JCBUS_2.b20 (Pin_b20), JCBUS_3.b20 (Pin_b20), JCBUS_4.b20 (Pin_b20), JCBUS_5.b20 (Pin_b20), JCBUS_6.b20 (Pin_b20)
- net RX: now also JCBUS_1.a8 (Pin_a8), JCBUS_2.a8 (Pin_a8), JCBUS_3.a8 (Pin_a8), JCBUS_4.a8 (Pin_a8), JCBUS_5.a8 (Pin_a8), JCBUS_6.a8 (Pin_a8)
- net RX2: now also JCBUS_1.a6 (Pin_a6), JCBUS_2.a6 (Pin_a6), JCBUS_3.a6 (Pin_a6), JCBUS_4.a6 (Pin_a6), JCBUS_5.a6 (Pin_a6), JCBUS_6.a6 (Pin_a6)
- net TX: now also JCBUS_1.a7 (Pin_a7), JCBUS_2.a7 (Pin_a7), JCBUS_3.a7 (Pin_a7), JCBUS_4.a7 (Pin_a7), JCBUS_5.a7 (Pin_a7), JCBUS_6.a7 (Pin_a7)
- net TX2: now also JCBUS_1.a5 (Pin_a5), JCBUS_2.a5 (Pin_a5), JCBUS_3.a5 (Pin_a5), JCBUS_4.a5 (Pin_a5), JCBUS_5.a5 (Pin_a5), JCBUS_6.a5 (Pin_a5)
- net WAIT: now also JCBUS_1.b16 (Pin_b16), JCBUS_2.b16 (Pin_b16), JCBUS_3.b16 (Pin_b16), JCBUS_4.b16 (Pin_b16), JCBUS_5.b16 (Pin_b16), JCBUS_6.b16 (Pin_b16)
- net WR: now also JCBUS_1.b11 (Pin_b11), JCBUS_2.b11 (Pin_b11), JCBUS_3.b11 (Pin_b11), JCBUS_4.b11 (Pin_b11), JCBUS_5.b11 (Pin_b11), JCBUS_6.b11 (Pin_b11)
- no-connect marks 111 -> 87
