File: schem/Model_150/Model_150.kicad_sch (KiCad schematic)
At the start: 378 parts, among them SW1 RESET, SW2 POWER, U0 74LS00, U1 74LS04, U10 MAX232, U11 MAX232, U12 74LS00, U13 74HCT74, U14 74LS32, U15 74LS02, U16 74LS161, U18 74AHCT125, U19 74LS04, U2 DS1233, U20 74HCT138, U21 74LS74, U22 74LS139, U23 74LS32, U24 74HCT273, U25 DS1302+, U26 74AHCT125, U27 82C55A, U28 74LS04, U29 74HCT138, U3 74AHCT125, U30 74LS08, U33 4049UB, U34 74LS76, U36 74LS153, U37 LM555xN, U38 4070, U39 74LS161, U4 74HCT139, U40 74LS00, U41 74LS161, U42 74LS74, U43 4046, U5 74HCT688, U6 74HCT273, U7 74HCT157, U8 74HCT138, U9 74HCT273

Commit message: fssddfsfzfs
Parts:
- removed JP20: CLK_FDC_CLK, symbol Jumper:SolderJumper_2_Open
- removed JP25: CLK_FPU_CLK2, symbol Jumper:SolderJumper_2_Open
- removed JP26: CLK_FPU_CLK, symbol Jumper:SolderJumper_2_Open
- removed JP31: DMA_RDYA, Connector_PinHeader_2.54mm:PinHeader_1x02_P2.54mm_Vertical, symbol Jumper:Jumper_2_Open
- removed JP32: DMA_RDYB, Connector_PinHeader_2.54mm:PinHeader_1x02_P2.54mm_Vertical, symbol Jumper:Jumper_2_Open
- removed JP37: CLK_CTC_TAPE, symbol Jumper:SolderJumper_2_Open
- removed JP38: CLK_555_TAPE, symbol Jumper:SolderJumper_2_Open
- removed JP7: CLK_FDC_RES, symbol Jumper:SolderJumper_2_Open
- removed JP8: CLK_CTC, Connector_PinHeader_2.54mm:PinHeader_1x02_P2.54mm_Vertical, symbol Jumper:Jumper_2_Open
- removed JP9: CLK2_CTC, symbol Jumper:Jumper_2_Bridged
- added JP20: FPU_CLK_CLK2, Connector_PinHeader_2.54mm:PinHeader_1x03_P2.54mm_Vertical, symbol Jumper:Jumper_3_Open
- added JP25: DMA_RDY, Connector_PinHeader_2.54mm:PinHeader_1x03_P2.54mm_Vertical, symbol Jumper:Jumper_3_Open
- added JP37: TAPE_CTC_555, Connector_PinHeader_2.54mm:PinHeader_1x03_P2.54mm_Vertical, symbol Jumper:Jumper_3_Open
- added JP7: FDC_CLK_RES, Connector_PinHeader_2.54mm:PinHeader_1x03_P2.54mm_Vertical, symbol Jumper:Jumper_3_Open
- added JP8: CTC_CLK_CLK2, Connector_PinHeader_2.54mm:PinHeader_1x03_P2.54mm_Vertical, symbol Jumper:Jumper_3_Open
- added TS_1: TAPE_IN, Connector_Audio:Jack_3.5mm_CUI_SJ1-3525N_Horizontal, symbol Connector_Audio:AudioJack2
- added TS_2: TAPE_OUT, Connector_Audio:Jack_3.5mm_CUI_SJ1-3525N_Horizontal, symbol Connector_Audio:AudioJack2
- JP16: value TX1 -> BUS_TX1
- JP17: value RX1 -> BUS_RX1
- JP18: value TX2 -> BUS_TX2
- JP19: value RX2 -> BUS_RX2
- JP9: renamed from JP33; value SIO_A0_INVERT -> SIO_A0_INV
Connections:
- net CLK: now also JP20.1 (A), JP7.1 (A), JP8.3 (B)
- net CLK2: now also JP20.3 (B), JP8.1 (A)
- net CLK_768: now also JP37.1 (A)
- net RDY: now also JP25.2 (C)
- net RDYA: now also JP25.1 (A)
- net RDYB: now also JP25.3 (B)
- net at CTC_0.21 (CLK/TRG2), CTC_0.22 (CLK/TRG1), CTC_0.23 (CLK/TRG0): now also JP8.2 (C)
- net at U19.6: now also JP7.3 (B)
- net at FDC_0.23 (CLK1): now also JP7.2 (C)
- net at JP28.2 (B), U21.3 (C): now also JP20.2 (C)
- net DC: now reaches FDD_0.34 (Pin_34), RN2.2 (R1), U18.2
- net DC: no longer RN2.5 (R4)
- net at FDC_0.38 (~{TR00}), FDD_0.26 (Pin_26): now also RN2.4 (R3); no longer RN2.3 (R2)
- net at U37.3 (Q): now also JP37.3 (B)
- net at U16.2 (CP), U39.2 (CP): now also JP37.2 (C)
- new net: FDC_0.39 (~{IDX}), FDD_0.8 (Pin_8), RN2.3 (R2)
- new net: FDC_0.37 (WP), FDD_0.28 (Pin_28), RN2.5 (R4)
Other:
- note added: "DC"
- note added: "Input: D0 - RTC_DIN D4 - TAPE_IN D5 - TAPE_IN_RAW Output: D0 - TAPE_SPD_L D1 - TAPE_SPD_H D2 - TAPE_MOTOR D3 - TAPE_OUT D4 - RTC_CE D5 - RTC_WE D6 - RTC_SCLK D7 - RTC_DOUT Note: SEL_RTC = SEL_TAPE Note: TAPE_SPD selects baud rate."
- note added: "JP28-30 can divide clock if too fast for FPU."
- note added: "JP8-9 select clock source for CTC: CLK or CLK2 JP10-15 select clock source for SIO (A/B): CTC, CLK, or CLK2"
- note added: "Opt.1) 1x RS-232 on SIO A or B. Opt.2) 2x RS-232 on SIO A and B. Opt.3) 1x RS-232 on SIO A, and 1x KCS-Tape on SIO B."
- note added: "Opt.1) SIO A data, SIO B data. Opt.2) SIO A data, SIO A control. Opt.3) SIO B data, SIO A control."
- note removed: "Input: D0 - RTC_DIN D4 - TAPE_IN D5 - TAPE_IN_RAW Output: D0 - TAPE_SPD_L D1 - TAPE_SPD_H D2 - TAPE_MOTOR D3 - TAPE_OUT D4 - RTC_CE D5 - RTC_WE D6 - RTC_SCLK D7 - RTC_DOUT Note: SEL_RTC = SEL_TAPE"
- note removed: "JP8-9 select clock source for CTC: CLK or CLK2 JP10-15 select clock source for SIO (A&B): CTC, CLK, or CLK2"
- moved on the sheet: FDD_0, JP22
