File: schem/Model_150/Model_150.kicad_pcb (KiCad board)
At the start: 2 copper layers, 300 x 200 mm, 387 parts, among them SW1 RESET, SW2 POWER, U0 74LS00, U1 74LS04, U10 MAX232, U11 MAX232, U12 74LS00, U13 74HCT74, U14 74LS32, U15 74LS02, U16 74LS161, U17 74LS00, U18 74AHCT125, U19 74LS04, U2 DS1233, U20 74HCT138, U21 74LS74, U22 74LS139, U23 74LS32, U24 74HCT273, U25 DS1302+, U26 74AHCT125, U27 82C55A, U28 74LS04, U29 74HCT138, U3 74AHCT125, U30 74LS08, U33 4049UB, U34 74LS76, U37 LM555xN, U38 4070, U39 74LS161, U4 74HCT139, U40 74LS00, U41 74LS161, U42 74LS74, U43 4046, U5 74HCT688, U6 74HCT273, U7 74HCT157, U8 74HCT138, U9 74HCT273

Commit message: Add FDC jumper config, update footprints
- Added JP45 jumper for FDC_PCVAL configuration with three-pole connector
- Added JP33 jumper for SIO_A0_INVERT configuration
- Changed FDC pin 22 (DRV) from GND to +5V
- Connected FDC pin 24 (PCVAL) to new configurable net via JP45
- Updated capacitor footprints from radial to disc types
- Changed crystal resonator from 6.0mm to 10.0mm package
- Added floppy controller datasheets
- Fixed various component value formatting (R220 → 220R)
- Added power and ground symbols for jumper connections
Parts:
- added JP33: SIO_A0_INVERT, Connector_PinHeader_2.54mm:PinHeader_1x03_P2.54mm_Vertical, F.Cu at (244.5, 60.6)
- added JP45: FDC_PCVAL, Connector_PinHeader_2.54mm:PinHeader_1x03_P2.54mm_Vertical, F.Cu at (384.3, 220.2)
- C34: value 2.1uF -> 100nF; footprint Capacitor_THT:C_Radial_D5.0mm_H11.0mm_P2.00mm -> Capacitor_THT:C_Disc_D5.0mm_W2.5mm_P2.50mm
- C37: footprint Capacitor_THT:C_Radial_D5.0mm_H11.0mm_P2.00mm -> Capacitor_THT:C_Disc_D6.0mm_W2.5mm_P5.00mm
- R10, R11, R12, R13, R14, R7, R8, R9: value R220 -> 220R
- XTAL_RES_0: footprint Crystal:Resonator-2Pin_W6.0mm_H3.0mm -> Crystal:Resonator-2Pin_W10.0mm_H5.0mm
Connections:
- FDC_0 pad 22: GND -> +5V
- FDC_0 pad 24: +5V -> Net-(FDC_0-PCVAL)
- U0 pad 10: (no net) -> +5VSB
- U0 pad 12: unconnected-(U0-Pad12) -> +5VSB
- U0 pad 13: unconnected-(U0-Pad13) -> +5VSB
- U0 pad 8: (no net) -> unconnected-(U0-Pad8)
- U0 pad 9: (no net) -> +5VSB
- U22 pad 13: unconnected-(U22B-A1-Pad13) -> GND
- U22 pad 14: unconnected-(U22B-A0-Pad14) -> GND
- U22 pad 15: unconnected-(U22B-E-Pad15) -> +5V

Commit message: updates yuo
Parts:
- removed the ? at (162.3, 190.5)
- removed the ? at (164.8, 193.0)
- removed the ? at (164.8, 190.5)
- removed the ? at (162.3, 193.0)
- removed JCBUS_0: JC100, Carboni_Library:JC100_Bus_16b
- removed the TP1 at (44.5, 193.0)
- removed the TP1 at (44.5, 190.5)
- removed TP121, TP122, TP123, TP124: NC, TestPoint:TestPoint_THTPad_1.5x1.5mm_Drill0.7mm
- removed the TP2 at (41.9, 190.5)
- removed the TP3 at (41.9, 193.0)
- added JCBUS_6: JC64, Carboni_Library:JC64_Bus_8b, F.Cu at (53.3, 61.0)
- JCBUS_1, JCBUS_2, JCBUS_3, JCBUS_4, JCBUS_5: value JC100 -> JC64; footprint Carboni_Library:JC100_Bus_16b -> Carboni_Library:JC64_Bus_8b
- JP23: value FDC_JP1 -> FDC_DACK
- JP24: value FDC_JP2 -> FDC_TC
- moved TP107 174.5 mm to (11.9, 1.27)
- moved TP108 173.5 mm to (11.9, 4.83)
- moved TP109 172.5 mm to (11.9, 8.38)
- moved TP110 171.5 mm to (11.9, 11.9)
- moved TP81 171.0 mm to (4.83, 1.27)
- moved TP111 170.5 mm to (11.9, 15.5)
- moved TP112 169.5 mm to (11.9, 19.0)
- moved TP113 168.6 mm to (11.9, 22.6)
- moved TP96 167.2 mm to (8.38, 1.27)
- moved TP97 166.2 mm to (8.38, 4.83)
- moved TP102 165.2 mm to (8.38, 8.38)
- moved TP103 164.3 mm to (8.38, 11.9)
- moved TP104 163.3 mm to (8.38, 15.5)
- moved TP105 162.3 mm to (8.38, 19.0)
- moved TP74 154.7 mm to (1.27, 1.27)
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Connections:
- DMA_0 pad 10: MREQ -> IORQ
- DMA_0 pad 12: IORQ -> MREQ
- JP33 pad 1: (no net) -> A0
- JP33 pad 2: (no net) -> Net-(JP33-C)
- JP33 pad 3: (no net) -> Net-(JP33-B)
Routing:
- net GND: track 565.4 -> 15.2 mm
- net +5V: track 506.6 -> 0.00 mm
- net +12V: track 506.6 -> 0.00 mm
- net DACK1: track 138.0 -> 0.00 mm
- net DREQ2: track 138.0 -> 0.00 mm
- net DREQ0: track 138.0 -> 0.00 mm
- net DACK3: track 138.0 -> 0.00 mm
- net DACK0: track 138.0 -> 0.00 mm
- net A29: track 138.0 -> 0.00 mm
- net A28: track 138.0 -> 0.00 mm
- net A25: track 138.0 -> 0.00 mm
- net A24: track 138.0 -> 0.00 mm
- net A26: track 138.0 -> 0.00 mm
- net DREQ1: track 138.0 -> 0.00 mm
- net DACK2: track 138.0 -> 0.00 mm
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